File: PCB/Magna/analogIOexpander.kicad_sch (KiCad schematic)
At the start: 2 parts, among them U1501 4052

Commit message: Add final touched to all schematics
Parts:
- renumbered C1501 to C1, U1501 to U9
Other:
- moved on the sheet: C1, U9
