File: PCB/Magna/Magna.kicad_pcb (KiCad board)
At the start: 2 copper layers, 120 x 320 mm, 164 parts, among them J1001 DIN-5_180degree, J1002 DIN-5_180degree, J1003 DIN-5_180degree, J301 Conn_02x15_Odd_Even, J601 Conn_02x10_Counter_Clockwise, J701 Conn_02x06_Odd_Even, J703 Conn_ARM_JTAG_SWD_20, J704 Boot Jumper, J801 USB_A, J802 USB_C_Receptacle_USB2.0, J803 USB_B, U1001 74LVC2G14, U1002 74LVC2G14, U1003 74HC08D, U1004 TLP2361, U201 24.576 MHz, U701 STM32F730V8T6, U801 SRV05-4, U802 USB3300-EZK, U902 XL1509-ADJ, U903 WS3222D, U905 AP2171W, Y701 24MHz

Commit message: Start of layout for Mainboard PCB
Parts:
- removed C803: 220uF, Capacitor_SMD:CP_Elec_4x5.8
- removed C901, C913: 100u/10V, Capacitor_SMD:CP_Elec_6.3x5.8
- removed C908: 22pF/50V, Capacitor_SMD:C_0805_2012Metric_Pad1.18x1.45mm_HandSolder
- removed C910: 4.7uF/25V, Capacitor_SMD:C_0805_2012Metric_Pad1.18x1.45mm_HandSolder
- removed D1005: B5819, Diode_SMD:D_SOD-123
- removed TP903, TP904, TP905, TP906, TP908: TestPoint, TestPoint:TestPoint_Keystone_5005-5009_Compact
- added C401: 22uF/25V, Capacitor_SMD:C_0805_2012Metric_Pad1.18x1.45mm_HandSolder, F.Cu at (15.0, 18.0)
- added C402: 22uF/25V, Capacitor_SMD:C_0805_2012Metric_Pad1.18x1.45mm_HandSolder, F.Cu at (15.0, 21.0)
- added C403: 22uF/25V, Capacitor_SMD:C_0805_2012Metric_Pad1.18x1.45mm_HandSolder, F.Cu at (15.0, 24.0)
- added C601: 22uF/25V, Capacitor_SMD:C_0805_2012Metric_Pad1.18x1.45mm_HandSolder, F.Cu at (-94.2, 75.6)
- added C602: 22uF/25V, Capacitor_SMD:C_0805_2012Metric_Pad1.18x1.45mm_HandSolder, F.Cu at (-94.2, 78.6)
- added C603: 22uF/25V, Capacitor_SMD:C_0805_2012Metric_Pad1.18x1.45mm_HandSolder, F.Cu at (15.0, 79.5)
- added C604: 22uF/25V, Capacitor_SMD:C_0805_2012Metric_Pad1.18x1.45mm_HandSolder, F.Cu at (17.5, 79.5)
- added C605: 22uF/25V, Capacitor_SMD:C_0805_2012Metric_Pad1.18x1.45mm_HandSolder, F.Cu at (12.5, 84.5)
- added C606: 22uF/25V, Capacitor_SMD:C_0805_2012Metric_Pad1.18x1.45mm_HandSolder, F.Cu at (12.5, 79.5)
- added C607: 22uF/25V, Capacitor_SMD:C_0805_2012Metric_Pad1.18x1.45mm_HandSolder, F.Cu at (17.5, 84.5)
- added C609: 22uF/25V, Capacitor_SMD:C_0805_2012Metric_Pad1.18x1.45mm_HandSolder, F.Cu at (-89.4, 81.6)
- added C610: 22uF/25V, Capacitor_SMD:C_0805_2012Metric_Pad1.18x1.45mm_HandSolder, F.Cu at (-89.4, 84.6)
- added C611: 22uF/25V, Capacitor_SMD:C_0805_2012Metric_Pad1.18x1.45mm_HandSolder, F.Cu at (-89.4, 87.7)
- added C612: 22uF/25V, Capacitor_SMD:C_0805_2012Metric_Pad1.18x1.45mm_HandSolder, F.Cu at (-89.4, 90.7)
- added C613: 22uF/25V, Capacitor_SMD:C_0805_2012Metric_Pad1.18x1.45mm_HandSolder, F.Cu at (-84.6, 75.6)
- added C614: 22uF/25V, Capacitor_SMD:C_0805_2012Metric_Pad1.18x1.45mm_HandSolder, F.Cu at (-84.6, 78.6)
- added C615: 22uF/25V, Capacitor_SMD:C_0805_2012Metric_Pad1.18x1.45mm_HandSolder, F.Cu at (-84.6, 81.6)
- added C616: 10p/50V, Capacitor_SMD:C_0603_1608Metric_Pad1.08x0.95mm_HandSolder, F.Cu at (14.0, 61.0)
- added C617: 220nF/16V, Capacitor_SMD:C_0402_1005Metric_Pad0.74x0.62mm_HandSolder, F.Cu at (21.2, 80.8)
- added D501: 1N4148WS, Diode_SMD:D_SOD-123, F.Cu at (107.0, 28.0)
- C1001, C1002: value 10n -> 10nF/50V
- C1003, C1004, C1005, C1006, C705, C706, C707, C708, C709, C710, C711, C713, C715, C801, C802, C804, C805, C914, C917: value 100nF/50V -> 220nF/16V; footprint Capacitor_SMD:C_0805_2012Metric_Pad1.18x1.45mm_HandSolder -> Capacitor_SMD:C_0402_1005Metric_Pad0.74x0.62mm_HandSolder
- C201: footprint Capacitor_SMD:C_0603_1608Metric_Pad1.08x0.95mm_HandSolder -> Capacitor_SMD:C_0805_2012Metric_Pad1.18x1.45mm_HandSolder
- C701, C702, C703, C704: value 2.2uF/6.3V -> 22uF/25V
- C712, C714, C905: value 1uF/50V -> 22uF/25V
- C716, C806, C807, C904, C912: value 4.7uF/25V -> 22uF/25V
- C902: value 10uF/25V -> 22uF/25V; footprint Capacitor_SMD:CP_Elec_4x5.8 -> Capacitor_SMD:C_0805_2012Metric_Pad1.18x1.45mm_HandSolder
- J301: footprint Connector_PinSocket_2.54mm:PinSocket_2x15_P2.54mm_Horizontal -> Connector_PinSocket_2.54mm:PinSocket_2x16_P2.54mm_Horizontal
- R905: value 18k -> 39k; footprint Resistor_SMD:R_0603_1608Metric_Pad0.98x0.95mm_HandSolder -> Resistor_SMD:R_0805_2012Metric_Pad1.20x1.40mm_HandSolder
- R906: value 10k -> 12k
- TP1001, TP1002, TP1003, TP201, TP801, TP802, TP803, TP804, TP805: footprint TestPoint:TestPoint_Keystone_5005-5009_Compact -> TestPoint:TestPoint_Keystone_5000-5004_Miniature
- U1001: footprint Package_SO:SOIC-14_3.9x8.7mm_P1.27mm -> Package_TO_SOT_SMD:SOT-363_SC-70-6_Handsoldering
- U1002: footprint Package_DIP:DIP-8_W7.62mm -> Package_TO_SOT_SMD:SOT-363_SC-70-6_Handsoldering
- moved TP1003 256.6 mm to (-30.0, 7.00)
- moved TP1002 246.0 mm to (-5.65, 7.00)
- moved TP1001 245.4 mm to (-5.65, 2.65)
- moved TP805 237.9 mm to (-23.0, 20.0)
- moved TP804 237.3 mm to (-23.0, 15.7)
- moved TP803 236.7 mm to (-23.0, 11.3)
- moved TP802 234.1 mm to (-18.4, 7.00)
- moved TP801 233.4 mm to (-18.4, 2.65)
- moved D2106 216.1 mm to (-100.0, 122.2)
- moved D2102 216.1 mm to (-100.0, 110.0)
- moved D2103 216.1 mm to (-100.0, 113.0)
- moved D2104 216.1 mm to (-100.0, 116.1)
- moved D2107 216.1 mm to (-100.0, 125.2)
- moved R2102 216.1 mm to (-95.2, 109.9)
- moved R2103 216.1 mm to (-95.2, 112.8)
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Connections:
- net Net-(U902-VIN) renamed /POWER/+5V_ferrited
- J301 pad 29: VDD -> /Audio Daughterboard Connector/VAA_EN
- R1003 pad 1: Net-(D1001-K) -> GND
- R1003 pad 2: GND -> Net-(D1001-K)
- U1003 pad 1: /MCU/MIDI_RX -> +5V
- U1003 pad 10: Net-(R1008-Pad1) -> Net-(R1009-Pad1)
- U1003 pad 11: Net-(R1010-Pad1) -> Net-(R1008-Pad1)
- U1003 pad 2: /MCU/MIDI_RX -> +5V
- U1003 pad 3: Net-(R1009-Pad1) -> Net-(R1010-Pad1)
- U1003 pad 8: +5V -> /MCU/MIDI_RX
- U1003 pad 9: +5V -> /MCU/MIDI_RX
- U701 pad 98: /MCU/VA_en -> /Audio Daughterboard Connector/VAA_EN
Routing:
- net +5V: track 0.00 -> 49.4 mm, vias 0 -> 7
- net GND: track 0.00 -> 44.5 mm, vias 0 -> 28
- net /MCU/MIDI_RX: track 0.00 -> 41.0 mm
- net /MIDI/MIDI_{IN+}: track 0.00 -> 30.8 mm
- net /MIDI/MIDI_{IN-cathode}: track 0.00 -> 22.8 mm
- net Net-(R1009-Pad1): track 0.00 -> 21.9 mm
- net Net-(R1010-Pad1): track 0.00 -> 18.7 mm
- net Net-(R1011-Pad1): track 0.00 -> 17.9 mm
- net /POWER/HS_OVLO: track 0.00 -> 17.3 mm
- net Net-(R1008-Pad1): track 0.00 -> 16.3 mm
- net Net-(D1002-K): track 0.00 -> 15.0 mm
- net Net-(D1001-K): track 0.00 -> 15.0 mm
- net /MCU/MIDI_TX: track 0.00 -> 12.7 mm
- net Net-(D903-K): track 0.00 -> 12.6 mm
- net VBUS_OUT: track 0.00 -> 11.7 mm
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- added copper zone on F.Cu, net +5V
- added copper zone on F.Cu, net /POWER/+5V_ferrited
- added copper zone on F.Cu, net /POWER/VBUS_{fused}
- added copper zone on F.Cu, net GND
- added copper zone on In1.Cu, net GND
- added copper zone on In2.Cu, net GND
Other:
- copper layers 2 -> 4

Commit message: Change DCDC for 3V and more deisgn of PCB
Parts:
- removed C603, C607, C615, C904: 22uF/25V, Capacitor_SMD:C_0805_2012Metric_Pad1.18x1.45mm_HandSolder
- removed D903: SS54, Diode_SMD:D_SMA_Handsoldering
- removed R901: 1k, Resistor_SMD:R_0805_2012Metric_Pad1.20x1.40mm_HandSolder
- removed R904: 1k5, Resistor_SMD:R_0805_2012Metric_Pad1.20x1.40mm_HandSolder
- removed U902: XL1509-ADJ, Package_SO:SOIC-8_3.9x4.9mm_P1.27mm
- added C608: 220nF/16V, Capacitor_SMD:C_0402_1005Metric_Pad0.74x0.62mm_HandSolder, F.Cu at (35.5, 77.6)
- added R601: 10k, Resistor_SMD:R_0805_2012Metric_Pad1.20x1.40mm_HandSolder, F.Cu at (30.0, 82.0)
- added R602: 39k, Resistor_SMD:R_0805_2012Metric_Pad1.20x1.40mm_HandSolder, F.Cu at (37.0, 81.0)
- added R603: 12k, Resistor_SMD:R_0805_2012Metric_Pad1.20x1.40mm_HandSolder, F.Cu at (37.0, 83.0)
- added U601: TPS563201, Package_TO_SOT_SMD:SOT-23-6, F.Cu at (32.0, 79.0)
- L902: value 22µH -> 2.2µH; footprint Skrooter_footprints:MSCD43 -> Inductor_SMD:L_Sunlord_SWPA3012S
- moved C914 171.1 mm to (22.0, 50.4), turned to -90 degrees
- moved U905 167.7 mm to (25.0, 49.0), turned to 180 degrees
- moved FB905 154.8 mm to (29.0, 47.0), turned to 180 degrees
- moved C917 151.7 mm to (28.0, 51.1), turned to -90 degrees
- moved R908 148.8 mm to (28.5, 57.0), turned to 180 degrees
- moved F902 147.5 mm to (14.0, 46.0), turned to -90 degrees
- moved C601 126.6 mm to (30.0, 51.0), turned to -90 degrees
- moved C609 120.1 mm to (30.5, 74.5), turned to -90 degrees
- moved C610 118.3 mm to (28.5, 74.5), turned to -90 degrees
- moved C611 116.6 mm to (26.5, 74.5), turned to -90 degrees
- moved C602 116.5 mm to (19.0, 51.0), turned to -90 degrees
- moved C612 115.0 mm to (24.5, 74.5), turned to -90 degrees
- moved C613 107.1 mm to (22.5, 74.5), turned to -90 degrees
- moved C614 105.2 mm to (20.5, 74.5), turned to -90 degrees
- moved L902 22.1 mm to (33.5, 74.0), turned to 90 degrees
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Connections:
- L902 pad 1: Net-(D903-K) -> /POWER/DCDC_SW
Routing:
- net VBUS_OUT: track 11.7 -> 42.5 mm
- net /POWER/+5V_ferrited: track 0.00 -> 28.7 mm
- net Net-(U601-EN): track 0.00 -> 28.5 mm
- net +5V: track 49.4 -> 29.1 mm, vias 7 -> 29
- net Net-(D903-K): track 12.6 -> 0.00 mm
- net /MCU/~{VBUS_OUT_FLG}: track 0.00 -> 11.7 mm, vias 0 -> 2
- net Net-(U905-IN): track 0.00 -> 10.1 mm
- net Net-(U905-OUT): track 0.00 -> 7.30 mm
- net /MCU/USB_A_PWR_EN: track 0.00 -> 7.07 mm, vias 0 -> 2
- net Net-(U601-VFB): track 0.00 -> 5.30 mm
- net Net-(U601-VBST): track 0.00 -> 2.40 mm
- net VDD: track 2.14 -> 4.14 mm, vias 0 -> 11
- net GND: track 44.5 -> 43.1 mm, vias 28 -> 27
- net /POWER/DCDC_SW: track 0.00 -> 1.00 mm
- added copper zone on B.Cu, net +5V
- added copper zone on F.Cu, net /POWER/DCDC_SW
- added copper zone on B.Cu, net VDD
- added copper zone on F.Cu, net VDD
- removed copper zone on F.Cu, net /POWER/+5V_ferrited

Commit message: Add more traces to the PCB
Parts:
- removed D806: green, Diode_SMD:D_0805_2012Metric_Pad1.15x1.40mm_HandSolder
- removed the J701 at (33.7, 157.5)
- removed J703: Conn_ARM_JTAG_SWD_20, Connector_PinHeader_2.54mm:PinHeader_2x05_P2.54mm_Vertical_SMD
- removed R707: 22R, Resistor_SMD:R_0805_2012Metric_Pad1.20x1.40mm_HandSolder
- removed R807: 470R, Resistor_SMD:R_0805_2012Metric_Pad1.20x1.40mm_HandSolder
- removed TP1001, TP1002, TP1003, TP801, TP802, TP803, TP804, TP805: TestPoint, TestPoint:TestPoint_Keystone_5000-5004_Miniature
- removed U802: USB3300-EZK, Package_DFN_QFN:QFN-32-1EP_5x5mm_P0.5mm_EP3.45x3.45mm
- added C212: 22uF/25V, Capacitor_SMD:C_0805_2012Metric_Pad1.18x1.45mm_HandSolder, F.Cu at (98.4, 152.4)
- added C410: 22uF/25V, Capacitor_SMD:C_0805_2012Metric_Pad1.18x1.45mm_HandSolder, F.Cu at (40.1, 41.7)
- added D406: green, Diode_SMD:D_0805_2012Metric_Pad1.15x1.40mm_HandSolder, F.Cu at (111.3, 69.1)
- added J201: Conn_02x06_Odd_Even, Connector_PinSocket_2.54mm:PinSocket_2x06_P2.54mm_Vertical_SMD, F.Cu at (-64.6, 14.6)
- added J202: Conn_ARM_JTAG_SWD_20, Connector_PinHeader_2.54mm:PinHeader_2x05_P2.54mm_Vertical_SMD, F.Cu at (-53.2, 13.3)
- added R205: 22R, Resistor_SMD:R_0805_2012Metric_Pad1.20x1.40mm_HandSolder, F.Cu at (71.6, 101.1)
- added R225: 0R, Resistor_SMD:R_0805_2012Metric_Pad1.20x1.40mm_HandSolder, F.Cu at (96.4, 118.4)
- added R226: 0R, Resistor_SMD:R_0805_2012Metric_Pad1.20x1.40mm_HandSolder, F.Cu at (93.5, 118.4)
- added R407: 470R, Resistor_SMD:R_0805_2012Metric_Pad1.20x1.40mm_HandSolder, F.Cu at (111.3, 65.0)
- added U402: USB3300-EZK, Package_DFN_QFN:QFN-32-1EP_5x5mm_P0.5mm_EP3.45x3.45mm, F.Cu at (46.7, 41.1)
- added U403: SRV05-4, Package_TO_SOT_SMD:SOT-23-6, F.Cu at (45.5, 25.4)
- J203: renamed from J704; moved to B.Cu
- moved D805 213.6 mm to (106.2, 69.1), turned to 90 degrees
- moved D804 210.4 mm to (103.6, 69.1), turned to 90 degrees
- moved R805 210.0 mm to (106.2, 65.0), turned to -90 degrees
- moved R804 206.8 mm to (103.6, 65.0), turned to -90 degrees
- moved D803 206.5 mm to (101.1, 69.1), turned to 90 degrees
- moved D802 203.3 mm to (98.6, 69.1), turned to 90 degrees
- moved D403 203.2 mm to (39.0, 12.7)
- moved R803 202.8 mm to (101.1, 65.0), turned to -90 degrees
- moved D404 200.3 mm to (33.5, 17.8)
- moved D801 200.2 mm to (96.0, 69.1), turned to 90 degrees
- moved R802 199.6 mm to (98.6, 65.0), turned to -90 degrees
- moved R801 196.4 mm to (96.0, 65.0), turned to -90 degrees
- moved R411 183.0 mm to (24.9, 27.9), turned to -90 degrees
- moved R409 176.4 mm to (24.9, 19.8), turned to -90 degrees
- moved R410 175.3 mm to (24.9, 23.9), turned to -90 degrees
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- renumbered C701 to C201, C702 to C202, C703 to C203, C704 to C204, C705 to C205, C706 to C206, C707 to C207, C708 to C208, C709 to C209, C710 to C210, C711 to C211, C712 to C213, C713 to C214, C714 to C215, C715 to C216, C716 to C217, C717 to C218, C718 to C219, C201 to C220, C801 to C401, C802 to C402, C401 to C403, C804 to C404, C402 to C405, C805 to C406, C403 to C407, C806 to C408, C807 to C409, C1001 to C501, C1002 to C502, C1003 to C503, C1004 to C504, C1005 to C505, C1006 to C506, C606 to C601, C605 to C602, C604 to C603, C617 to C604, C902 to C605, C608 to C606, C906 to C607, C905 to C608, C616 to C612, C612 to C613, C613 to C614, C614 to C615, C602 to C616, C914 to C617, C912 to C618, C917 to C619, C601 to C620, D801 to D401, D802 to D402, D803 to D403, D804 to D404, D805 to D405, D1001 to D501, D1002 to D502, D1003 to D503, D1004 to D504, D501 to D505, D901 to D601, D2102 to D801, D2103 to D802, D2104 to D803, D2106 to D804, D2107 to D805, F901 to F601, F902 to F602, FB701 to FB201, FB901 to FB601, FB905 to FB602, J801 to J401, J802 to J402, J803 to J403, J1001 to J501, J1002 to J502, J1003 to J503, J601 to J701, L902 to L601, R701 to R201, R702 to R202, R705 to R203, R706 to R204, R708 to R206, R201 to R207, R709 to R208, R215 to R209, R216 to R210, R214 to R211, R213 to R212, R212 to R213, R203 to R214, R204 to R215, R205 to R216, R208 to R217, R209 to R218, R210 to R219, R211 to R220, R206 to R221, R207 to R222, R202 to R223, R710 to R224, R801 to R401, R802 to R402, R803 to R403, R804 to R404, R805 to R405, R806 to R406, R808 to R408, R809 to R409, R810 to R410, R811 to R411, R812 to R412, R813 to R413, R814 to R414, R1001 to R501, R1002 to R502, R1003 to R503, R1004 to R504, R1005 to R505, R1006 to R506, R1007 to R507, R1008 to R508, R1009 to R509, R1010 to R510, R1011 to R511, R603 to R602, R602 to R603, R905 to R604, R906 to R605, R907 to R606, R908 to R607, R2102 to R801, R2103 to R802, R2104 to R803, R2106 to R804, R2107 to R805, U701 to U201, U201 to U202, U801 to U401, U1001 to U501, U1002 to U502, U1003 to U503, U1004 to U504, U903 to U602, U905 to U603, Y701 to Y201
Connections:
- J701 pad 1: VDD -> /Human Interface/ADC_3
- J701 pad 10: /Human Interface/register_OE -> /Human Interface/serial_CLR
- J701 pad 12: /Human Interface/input_interrupt -> /Human Interface/serial_CLK
- J701 pad 13: /Human Interface/ADC_5 -> /Human Interface/lsb
- J701 pad 14: /Human Interface/ADC_4 -> /Human Interface/register_CLK
- J701 pad 15: /Human Interface/ADC_3 -> /Human Interface/I2C_SDA
- J701 pad 16: /Human Interface/ADC_2 -> /Human Interface/register_OE
- J701 pad 17: /Human Interface/ADC_1 -> GND
- J701 pad 18: /Human Interface/ADC_0 -> /Human Interface/serial_data
- J701 pad 19: GND -> /Human Interface/I2C_SCL
- J701 pad 2: /Human Interface/msb -> VDDA
- J701 pad 20: VDDA -> VDD
- J701 pad 3: /Human Interface/lsb -> /Human Interface/ADC_4
- J701 pad 4: /Human Interface/I2C_SDA -> /Human Interface/ADC_2
- J701 pad 5: /Human Interface/I2C_SCL -> /Human Interface/ADC_5
- J701 pad 6: /Human Interface/serial_data -> /Human Interface/ADC_1
- J701 pad 7: /Human Interface/serial_CLK -> /Human Interface/input_interrupt
- J701 pad 8: /Human Interface/serial_CLR -> /Human Interface/ADC_0
- J701 pad 9: /Human Interface/register_CLK -> /Human Interface/msb
- R217 pad 1: /MCU/ADC_DATA_0_MCU -> /Audio Daughterboard Connector/ADC_DATA_0
- R217 pad 2: /Audio Daughterboard Connector/ADC_DATA_0 -> /MCU/ADC_DATA_0_MCU
- R218 pad 1: /MCU/ADC_DATA_1_MCU -> /Audio Daughterboard Connector/ADC_DATA_1
- R218 pad 2: /Audio Daughterboard Connector/ADC_DATA_1 -> /MCU/ADC_DATA_1_MCU
- R219 pad 1: /MCU/ADC_DATA_2_MCU -> /Audio Daughterboard Connector/ADC_DATA_2
- R219 pad 2: /Audio Daughterboard Connector/ADC_DATA_2 -> /MCU/ADC_DATA_2_MCU
- R220 pad 1: /MCU/ADC_DATA_3_MCU -> /Audio Daughterboard Connector/ADC_DATA_3
- R220 pad 2: /Audio Daughterboard Connector/ADC_DATA_3 -> /MCU/ADC_DATA_3_MCU
- U201 pad 59: /Human Interface/lsb -> Net-(U201C-PD12)
- U201 pad 60: /Human Interface/msb -> Net-(U201C-PD13)
- U401 pad 1: /USB/USB_C_CONN_N -> /USB/USB_HOST_P
- U401 pad 3: /USB/USB_C_CONN_P -> /USB/USB_HOST_N
- U401 pad 4: /USB/USB_HOST_P -> /USB/USB_HOST_N
- U401 pad 6: /USB/USB_HOST_N -> /USB/USB_HOST_P
Routing:
- net /USB/USB_B_VBUS: track 4.53 -> 116.4 mm, vias 0 -> 3
- net /USB/USB_C_VBUS: track 4.31 -> 110.7 mm, vias 0 -> 5
- net VBUS: track 4.54 -> 99.3 mm, vias 0 -> 7
- net GND: track 43.1 -> 126.1 mm, vias 27 -> 75
- net VBUS_OUT: track 42.5 -> 119.9 mm, vias 0 -> 2
- net VDD: track 4.14 -> 62.3 mm, vias 11 -> 26
- net /Audio Daughterboard Connector/MCLK: track 0.00 -> 55.9 mm
- net Net-(D503-K): track 2.46 -> 56.2 mm, vias 0 -> 2
- net /Audio Daughterboard Connector/DAC_DATA_1: track 0.00 -> 53.3 mm
- net /Audio Daughterboard Connector/DAC_DATA_0: track 0.00 -> 53.3 mm
- net /Audio Daughterboard Connector/BCLK: track 0.00 -> 53.3 mm
- net /Audio Daughterboard Connector/ADC_DATA_3: track 0.00 -> 53.3 mm
- net /Audio Daughterboard Connector/ADC_DATA_2: track 0.00 -> 53.3 mm
- net /Audio Daughterboard Connector/ADC_DATA_0: track 0.00 -> 53.3 mm
- net /Audio Daughterboard Connector/LRCLK: track 0.00 -> 53.3 mm
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- added copper zone on B.Cu, net /USB/USB_B_VBUS
- added copper zone on B.Cu, net /USB/USB_C_VBUS
- added copper zone on B.Cu, net VBUS

Commit message: More routing
Parts:
- removed J201: Conn_02x06_Odd_Even, Connector_PinSocket_2.54mm:PinSocket_2x06_P2.54mm_Vertical_SMD
- removed J202: Conn_ARM_JTAG_SWD_20, Connector_PinHeader_2.54mm:PinHeader_2x05_P2.54mm_Vertical_SMD
- removed TP201: TestPoint, TestPoint:TestPoint_Keystone_5000-5004_Miniature
- added C221: 220nF/16V, Capacitor_SMD:C_0402_1005Metric_Pad0.74x0.62mm_HandSolder, F.Cu at (92.5, 122.2)
- added C411: 22uF/25V, Capacitor_SMD:C_0805_2012Metric_Pad1.18x1.45mm_HandSolder, F.Cu at (74.7, 108.2)
- added C412: 22uF/25V, Capacitor_SMD:C_0805_2012Metric_Pad1.18x1.45mm_HandSolder, F.Cu at (70.1, 108.2)
- added R415: 0R, Resistor_SMD:R_0805_2012Metric_Pad1.20x1.40mm_HandSolder, F.Cu at (103.1, 108.2)
- added R416: 0R, Resistor_SMD:R_0805_2012Metric_Pad1.20x1.40mm_HandSolder, F.Cu at (101.1, 108.2)
- added R417: 0R, Resistor_SMD:R_0805_2012Metric_Pad1.20x1.40mm_HandSolder, F.Cu at (99.1, 108.2)
- added R418: 0R, Resistor_SMD:R_0805_2012Metric_Pad1.20x1.40mm_HandSolder, F.Cu at (97.0, 108.2)
- added R419: 0R, Resistor_SMD:R_0805_2012Metric_Pad1.20x1.40mm_HandSolder, F.Cu at (95.0, 108.2)
- added R420: 0R, Resistor_SMD:R_0805_2012Metric_Pad1.20x1.40mm_HandSolder, F.Cu at (93.0, 108.2)
- added R421: 0R, Resistor_SMD:R_0805_2012Metric_Pad1.20x1.40mm_HandSolder, F.Cu at (90.9, 108.2)
- added R422: 0R, Resistor_SMD:R_0805_2012Metric_Pad1.20x1.40mm_HandSolder, F.Cu at (88.9, 108.2)
- added R423: 0R, Resistor_SMD:R_0805_2012Metric_Pad1.20x1.40mm_HandSolder, F.Cu at (111.3, 108.2)
- added R424: 0R, Resistor_SMD:R_0805_2012Metric_Pad1.20x1.40mm_HandSolder, F.Cu at (109.2, 108.2)
- added R425: 0R, Resistor_SMD:R_0805_2012Metric_Pad1.20x1.40mm_HandSolder, F.Cu at (107.2, 108.2)
- added R426: 0R, Resistor_SMD:R_0805_2012Metric_Pad1.20x1.40mm_HandSolder, F.Cu at (105.2, 108.2)
- added R427: 0R, Resistor_SMD:R_0805_2012Metric_Pad1.20x1.40mm_HandSolder, F.Cu at (113.3, 108.2)
- moved R409 91.1 mm to (68.1, 100.1)
- moved R410 91.1 mm to (68.1, 104.1)
- moved R411 91.1 mm to (68.1, 108.2)
- moved R414 85.5 mm to (38.4, 9.65), turned to -90 degrees
- moved R403 83.9 mm to (72.6, 100.1)
- moved R413 83.6 mm to (36.3, 9.65), turned to -90 degrees
- moved R404 83.6 mm to (72.6, 104.2)
- moved R405 83.6 mm to (72.6, 108.2)
- moved R225 62.5 mm to (158.9, 119.9)
- moved R226 62.5 mm to (156.0, 119.9)
- moved R202 35.3 mm to (79.8, 108.2), turned to -90 degrees
- moved R201 30.1 mm to (81.8, 108.2), turned to -90 degrees
- moved C220 15.2 mm to (88.9, 126.2)
- moved R205 14.5 mm to (84.3, 108.2)
- moved R223 12.5 mm to (88.9, 124.2)
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Connections:
- net Net-(U201A-PE12) renamed /MCU/serial_CLK_MCU
- net Net-(U201A-PE14) renamed /MCU/serial_data_MCU
- net Net-(U201C-PA11) renamed /MCU/USB_HOST_MCU_N
- net Net-(U201C-PA12) renamed /MCU/USB_HOST_MCU_P
- R209 pad 1: /MCU/I2S2_BCLK -> /Audio Daughterboard Connector/BCLK
- R209 pad 2: /Audio Daughterboard Connector/BCLK -> /MCU/I2S2_BCLK
- R210 pad 1: /MCU/I2S3_BCLK -> /Audio Daughterboard Connector/BCLK
- R210 pad 2: /Audio Daughterboard Connector/BCLK -> /MCU/I2S3_BCLK
- R211 pad 1: /MCU/I2S2_LRCLK -> /Audio Daughterboard Connector/LRCLK
- R211 pad 2: /Audio Daughterboard Connector/LRCLK -> /MCU/I2S2_LRCLK
- R212 pad 1: /MCU/I2S3_LRCLK -> /Audio Daughterboard Connector/LRCLK
- R212 pad 2: /Audio Daughterboard Connector/LRCLK -> /MCU/I2S3_LRCLK
- U201 pad 55: /Audio Daughterboard Connector/ADC_FORMAT -> /MCU/MIDI_TX
- U201 pad 56: /Audio Daughterboard Connector/ADC_M/S -> /MCU/MIDI_RX
- U201 pad 61: unconnected-(U201C-PD14-Pad61) -> /Audio Daughterboard Connector/ADC_FORMAT
- U201 pad 62: unconnected-(U201C-PD15-Pad62) -> /Audio Daughterboard Connector/ADC_M/S
- U201 pad 80: /MCU/MIDI_TX -> unconnected-(U201C-PC12-Pad80)
- U201 pad 83: /MCU/MIDI_RX -> unconnected-(U201C-PD2-Pad83)
- U402 pad 11: /MCU/NXT -> /USB/NXT_PHY
- U402 pad 12: /MCU/DIR -> /USB/DIR_PHY
- U402 pad 13: /MCU/STP -> /USB/STP_PHY
- U402 pad 14: /MCU/CLK -> /USB/CLK_PHY
- U402 pad 17: /MCU/DATA7 -> /USB/DATA7_PHY
- U402 pad 18: /MCU/DATA6 -> /USB/DATA6_PHY
- U402 pad 19: /MCU/DATA5 -> /USB/DATA5_PHY
- U402 pad 20: /MCU/DATA4 -> /USB/DATA4_PHY
- U402 pad 21: /MCU/DATA3 -> /USB/DATA3_PHY
- U402 pad 22: /MCU/DATA2 -> /USB/DATA2_PHY
- U402 pad 23: /MCU/DATA1 -> /USB/DATA1_PHY
- U402 pad 24: /MCU/DATA0 -> /USB/DATA0_PHY
- U402 pad 9: /MCU/USB_PHY_RESET -> Net-(U402-RESET)
Routing:
- net /MCU/MIDI_TX: track 5.78 -> 150.1 mm, vias 0 -> 2
- net Net-(U402-RESET): track 0.00 -> 125.6 mm, vias 0 -> 2
- net VDDA: track 11.1 -> 132.9 mm, vias 0 -> 2
- net /USB/USB_HOST_P: track 42.3 -> 147.9 mm
- net /USB/USB_HOST_N: track 42.2 -> 146.4 mm
- net /MCU/MIDI_RX: track 41.0 -> 144.6 mm, vias 0 -> 2
- net /Audio Daughterboard Connector/ADC_IWL: track 0.00 -> 98.3 mm, vias 0 -> 2
- net /USB/USB_B_VBUS: track 116.4 -> 214.6 mm
- net /Audio Daughterboard Connector/ADC_FSAMPEN: track 0.00 -> 93.4 mm, vias 0 -> 2
- net /USB/USB_C_VBUS: track 110.7 -> 201.1 mm, vias 5 -> 7
- net /Audio Daughterboard Connector/VAA_EN: track 0.00 -> 83.2 mm, vias 0 -> 1
- net /MCU/CLK_24MHz: track 7.23 -> 83.5 mm
- net /Audio Daughterboard Connector/ADC_M/S: track 0.00 -> 74.5 mm, vias 0 -> 2
- net /Audio Daughterboard Connector/ADC_FORMAT: track 0.00 -> 74.3 mm, vias 0 -> 2
- net /MCU/ADC_DATA_3_MCU: track 0.00 -> 56.7 mm, vias 0 -> 2
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
Commit message: Add last routing
Parts:
- added J201: Conn_02x06_Odd_Even, Connector_PinSocket_2.54mm:PinSocket_2x06_P2.54mm_Vertical_SMD, F.Cu at (100.6, 178.6)
- added J202: Conn_ARM_JTAG_SWD_20, Connector_PinHeader_2.54mm:PinHeader_2x05_P2.54mm_Vertical_SMD, F.Cu at (47.2, 99.1)
- moved R225 92.6 mm to (75.2, 159.5), turned to -90 degrees
- moved R226 91.8 mm to (73.2, 159.5), turned to 90 degrees
- moved J203 52.9 mm to (114.3, 233.2)
- moved R208 52.9 mm to (111.3, 229.1)
- moved R204 27.5 mm to (77.2, 159.5), turned to -90 degrees
- moved R203 18.0 mm to (79.2, 159.5)
- moved C209 2.69 mm to (77.7, 154.9), turned to 180 degrees
- moved C203 0.51 mm to (82.8, 125.5)
- moved C204 0.51 mm to (82.8, 123.4)
Connections:
- U201 pad 69: unconnected-(U201C-PA10-Pad69) -> /MCU/~{HSW_EN}
- U201 pad 7: /MCU/~{HSW_EN} -> unconnected-(U201C-PC13-Pad7)
Routing:
- net /Human Interface/serial_CLR: track 0.00 -> 272.2 mm, vias 0 -> 2
- net /Human Interface/register_CLK: track 0.00 -> 262.4 mm, vias 0 -> 2
- net /Human Interface/ADC_0: track 0.00 -> 262.0 mm, vias 0 -> 4
- net /Human Interface/ADC_1: track 0.00 -> 239.4 mm, vias 0 -> 4
- net /Human Interface/ADC_2: track 0.00 -> 226.4 mm, vias 0 -> 4
- net VDDA: track 132.9 -> 356.1 mm, vias 2 -> 3
- net /Human Interface/register_OE: track 0.00 -> 215.5 mm, vias 0 -> 2
- net /Human Interface/ADC_4: track 0.00 -> 213.1 mm, vias 0 -> 2
- net /Human Interface/ADC_3: track 10.3 -> 222.7 mm
- net /Human Interface/ADC_5: track 10.3 -> 222.2 mm, vias 0 -> 2
- net /Human Interface/input_interrupt: track 0.00 -> 205.7 mm
- net /Human Interface/serial_CLK: track 0.00 -> 192.6 mm, vias 0 -> 2
- net /Human Interface/I2C_SDA: track 0.00 -> 189.4 mm
- net /Human Interface/I2C_SCL: track 0.00 -> 188.7 mm
- net /Human Interface/serial_data: track 0.00 -> 180.4 mm, vias 0 -> 2
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