File: PCB/Magna/Magna.kicad_pcb (KiCad board)
At the start: 2 copper layers, 13 x 1.4 mm, 497 parts, among them J1001 DIN-5_180degree, J1002 DIN-5_180degree, J1003 DIN-5_180degree, J1201 AudioJack3, J1301 PSG01550, J301 PSG01550, J401 PSG01550, J702 Conn_02x06_Odd_Even, J704 Conn_ARM_JTAG_SWD_20, J705 Boot Jumper, J706 Conn_02x06_Odd_Even, J801 USB_A, J802 USB_C_Receptacle_USB2.0, J803 USB_B, U1001 74HC08D, U1002 6N137, U1101 NE5532, U1201 NE5532, U1202 NE5532, U1203 TDA2822D, U1301 NE5532, U1302 NE5532, U1303 NE5532, U1501 4052, U1601 4052, U1701 4052, U1801 XL9535, U2001 74HC595, U2002 74HC595, U2003 74HC595, U2004 74HC595, U2005 74HC595, U201 24.576 MHz, U202 CY2305SXC-1HT, U203 CY2305SXC-1HT, U301 WM8782SEDS, U401 WM8782SEDS, U501 CS4344, U502 NE5532, U601 CS4344, U602 NE5532, U701 STM32F730V8T6, U801 SRV05-4, U802 USB3300-EZK, U901 TPS61040DBV, U902 XL1509-ADJ, U903 WS3222D, U904 AMS1117-5.0, U905 AP2171W, Y701 24MHz

Commit message: Split schematic to several projects
To allow for several boards to be done a kicad project
is needed for each
Parts:
- removed C1101, C1207, C1208, C1310, C1311: 220uF, Capacitor_SMD:CP_Elec_4x5.8
- removed C1102, C1211, C1213, C1216, C1217, C1303, C1306, C1307, C1501, C1601, C1701, C1801, C1802, C1803, C1804, C1805, C1806, C1807, C1808, C1809, C1810, C1811, C1812, C1813, C1814, C1815, C1816, C1817, C2001, C2002, C2003, C2004, C2005, C303, C305, C306, C308, C403, C405, C406, C408, C501, C503, C506, C601, C603, C606: 100nF/50V, Capacitor_SMD:C_0805_2012Metric_Pad1.18x1.45mm_HandSolder
- removed C1201, C1202, C1209, C1210, C1214, C1215, C1301, C1302, C1314, C1315: 100u/10V, Capacitor_SMD:CP_Elec_6.3x5.8
- removed C1203, C1204, C1304, C1305: 22uF/16V, Capacitor_SMD:CP_Elec_5x5.8
- removed C1205, C1206, C1308, C1309: 100pF/50V, Capacitor_SMD:C_0805_2012Metric_Pad1.18x1.45mm_HandSolder
- removed C1212, C301, C302, C304, C307, C309, C310, C401, C402, C404, C407, C409, C410, C504, C505, C507, C508, C511, C512, C604, C605, C607, C608, C611, C612: 10uF/25V, Capacitor_SMD:CP_Elec_4x5.8
- removed C1312, C1313: 47p/50V, Capacitor_SMD:C_0805_2012Metric_Pad1.18x1.45mm_HandSolder
- removed C201: F/NM, Capacitor_SMD:C_0603_1608Metric_Pad1.08x0.95mm_HandSolder
- removed C502, C602: 1uF/50V, Capacitor_SMD:C_0805_2012Metric_Pad1.18x1.45mm_HandSolder
- removed C509, C510, C609, C610: 10nF/50V, Capacitor_SMD:C_0805_2012Metric_Pad1.18x1.45mm_HandSolder
- removed D2001, D2009, D2017, D2040: Red, Diode_SMD:D_0805_2012Metric_Pad1.15x1.40mm_HandSolder
- removed D2002, D2003, D2004, D2010, D2011, D2012, D2018, D2019, D2020, D2025, D2028, D2031, D2037, D2038: yellow, Diode_SMD:D_0805_2012Metric_Pad1.15x1.40mm_HandSolder
- removed D2005, D2006, D2007, D2008, D2013, D2014, D2015, D2016, D2021, D2022, D2023, D2024, D2029, D2030, D2034, D2035, D2036: green, Diode_SMD:D_0805_2012Metric_Pad1.15x1.40mm_HandSolder
- removed D2026, D2027, D2032, D2033, D2039: White, Diode_SMD:D_0805_2012Metric_Pad1.15x1.40mm_HandSolder
- removed J1201: AudioJack3, Connector_Audio:Jack_3.5mm_CUI_SJ1-3525N_Horizontal
- removed J1301, J301, J401: PSG01550, Skrooter_footprints:psg01550
- removed J705: Boot Jumper, Connector_PinHeader_2.54mm:PinHeader_1x03_P2.54mm_Vertical
- removed J706: Conn_02x06_Odd_Even, Connector_PinSocket_2.54mm:PinSocket_2x06_P2.54mm_Vertical_SMD
- removed JP201, JP202, JP203, JP204, JP205, JP206, JP207, JP208, JP209, JP210: Jumper_2_Open, Jumper:SolderJumper-2_P1.3mm_Open_TrianglePad1.0x1.5mm
- removed JP301, JP302, JP303, JP304, JP401, JP402, JP403, JP404: SolderJumper_3_Bridged12, Jumper:SolderJumper-3_P2.0mm_Open_TrianglePad1.0x1.5mm_NumberLabels
- removed R1101, R1102, R1201, R1202, R1207, R1208, R1301, R1302, R1307, R1308, R1317, R1318, R505, R506, R605, R606: 22k, Resistor_SMD:R_0805_2012Metric_Pad1.20x1.40mm_HandSolder
- removed R1203, R1204, R1303, R1304: 680R, Resistor_SMD:R_0805_2012Metric_Pad1.20x1.40mm_HandSolder
- removed R1205, R1206, R1305, R1306: 1k3, Resistor_SMD:R_0805_2012Metric_Pad1.20x1.40mm_HandSolder
- removed R1209, R1210, R1309, R1310: 100R, Resistor_SMD:R_0805_2012Metric_Pad1.20x1.40mm_HandSolder
- removed R1211, R1212, R1801, R1802, R1803, R1804, R1805, R1810, R1811, R1812, R1813, R1818, R1819, R1820, R1821, R1826, R1827, R1828, R1832, R501, R502, R601, R602: 10k, Resistor_SMD:R_0805_2012Metric_Pad1.20x1.40mm_HandSolder
- removed R1213, R1214: 4R7, Resistor_SMD:R_0805_2012Metric_Pad1.20x1.40mm_HandSolder
- removed R1311, R1312, R1313, R1314: 4k7, Resistor_SMD:R_0805_2012Metric_Pad1.20x1.40mm_HandSolder
- removed R1315, R1316: 68R, Resistor_SMD:R_0805_2012Metric_Pad1.20x1.40mm_HandSolder
- removed R1806, R1807, R1808, R1809, R1814, R1815, R1816, R1817, R1822, R1823, R1824, R1825, R1829, R1830, R1831, R1833: 1k, Resistor_SMD:R_0805_2012Metric_Pad1.20x1.40mm_HandSolder
- removed R2001, R2002, R2003, R2004, R2005, R2006, R2007, R2008, R2009, R2010, R2011, R2012, R2013, R2014, R2015, R2016, R2017, R2018, R2019, R2020, R2021, R2022, R2023, R2024, R2025, R2028, R2029, R2030, R2031, R2034, R2035, R2036, R2037, R2038, R2040: 220R, Resistor_SMD:R_0805_2012Metric_Pad1.20x1.40mm_HandSolder
- removed R201, R202: R/NM, Resistor_SMD:R_0805_2012Metric_Pad1.20x1.40mm_HandSolder
- removed R2026, R2027, R2032, R2033, R2039: 1k5, Resistor_SMD:R_0805_2012Metric_Pad1.20x1.40mm_HandSolder
- removed R301, R302, R401, R402: 5k1, Resistor_SMD:R_0805_2012Metric_Pad1.20x1.40mm_HandSolder
- removed R503, R504, R603, R604: 470R, Resistor_SMD:R_0805_2012Metric_Pad1.20x1.40mm_HandSolder
- removed RV1201, RV1301, RV301, RV401: 10k/PTV112-4420A-B103, Skrooter_footprints:Potentiometer_Bourns_PTV09A-1_Dual_Vertical
- removed RV1401, RV1402, RV1403, RV1404, RV1405, RV1406, RV1407, RV1408, RV1410, RV1411, RV1412, RV1413, RV1414, RV1415, RV1416, RV1417, RV1418, RV1419, RV1420, RV1421, RV1422, RV1423: 10k/PTV09A-4020F-B103, Potentiometer_THT:Potentiometer_Bourns_PTV09A-1_Single_Vertical
- removed RV1409, RV1424: 10k/ PTA6043-2015DPB103, Potentiometer_THT:Potentiometer_Bourns_PTA6043_Single_Slide
- removed SW1801, SW1802, SW1803, SW1804, SW1805, SW1806, SW1807, SW1808, SW1809, SW1810, SW1811, SW1812, SW1813, SW1814, SW1815, SW1816: ~, Button_Switch_SMD:SW_Push_1P1T_XKB_TS-1187A
- removed U1101, U1201, U1202, U1301, U1302, U1303, U502, U602: NE5532, Package_SO:SOIC-8_3.9x4.9mm_P1.27mm
- removed U1203: TDA2822D, Package_SO:SOP-8_3.9x4.9mm_P1.27mm
- removed U1501, U1601, U1701: 4052, Package_SO:SO-16_3.9x9.9mm_P1.27mm
- removed U1801: XL9535, Package_SO:TSSOP-24_4.4x7.8mm_P0.65mm
- removed U2001, U2002, U2003, U2004, U2005: 74HC595, Package_SO:SO-16_3.9x9.9mm_P1.27mm
- removed U201: 24.576 MHz, Oscillator:Oscillator_SMD_Abracon_ASE-4Pin_3.2x2.5mm_HandSoldering
- removed U202, U203: CY2305SXC-1HT, Package_SO:SOIC-8_3.9x4.9mm_P1.27mm
- removed U301, U401: WM8782SEDS, Package_SO:SSOP-20_5.3x7.2mm_P0.65mm
- removed U501, U601: CS4344, Package_SO:MSOP-10_3x3mm_P0.5mm
- added J101: Conn_02x08_Counter_Clockwise, Connector_PinSocket_2.54mm:PinSocket_2x08_P2.54mm_Vertical, F.Cu at (198.1, 83.8)
- added J601: Conn_02x10_Counter_Clockwise, Connector_PinSocket_2.54mm:PinSocket_2x10_P2.54mm_Vertical, F.Cu at (137.2, 114.3)
- added J701: Conn_02x06_Odd_Even, Connector_PinSocket_2.54mm:PinSocket_2x06_P2.54mm_Vertical_SMD, F.Cu at (217.4, 75.5)
- added J703: Conn_ARM_JTAG_SWD_20, Connector_PinHeader_2.54mm:PinHeader_2x05_P2.54mm_Vertical_SMD, F.Cu at (228.8, 74.2)
- added R710: 22R, Resistor_SMD:R_0805_2012Metric_Pad1.20x1.40mm_HandSolder, F.Cu at (224.8, 83.0)
- added TP1001: TestPoint, TestPoint:TestPoint_Keystone_5005-5009_Compact, F.Cu at (234.0, 116.3)
- added TP1002: TestPoint, TestPoint:TestPoint_Keystone_5005-5009_Compact, F.Cu at (234.0, 121.3)
- added TP1003: TestPoint, TestPoint:TestPoint_Keystone_5005-5009_Compact, F.Cu at (234.0, 126.4)
- added TP801: TestPoint, TestPoint:TestPoint_Keystone_5005-5009_Compact, F.Cu at (269.2, 89.0)
- added TP802: TestPoint, TestPoint:TestPoint_Keystone_5005-5009_Compact, F.Cu at (269.2, 94.1)
- added TP803: TestPoint, TestPoint:TestPoint_Keystone_5005-5009_Compact, F.Cu at (269.2, 99.1)
- added TP804: TestPoint, TestPoint:TestPoint_Keystone_5005-5009_Compact, F.Cu at (269.2, 104.2)
- added TP805: TestPoint, TestPoint:TestPoint_Keystone_5005-5009_Compact, F.Cu at (269.2, 109.2)
- added TP901: TestPoint, TestPoint:TestPoint_Keystone_5005-5009_Compact, F.Cu at (248.1, 116.3)
- added TP902: TestPoint, TestPoint:TestPoint_Keystone_5005-5009_Compact, F.Cu at (248.1, 121.3)
- added TP903: TestPoint, TestPoint:TestPoint_Keystone_5005-5009_Compact, F.Cu at (253.1, 116.3)
- added TP904: TestPoint, TestPoint:TestPoint_Keystone_5005-5009_Compact, F.Cu at (253.1, 121.3)
- added TP905: TestPoint, TestPoint:TestPoint_Keystone_5005-5009_Compact, F.Cu at (258.2, 116.3)
- added TP906: TestPoint, TestPoint:TestPoint_Keystone_5005-5009_Compact, F.Cu at (258.2, 121.3)
- added TP907: TestPoint, TestPoint:TestPoint_Keystone_5005-5009_Compact, F.Cu at (263.2, 116.3)
- added TP908: TestPoint, TestPoint:TestPoint_Keystone_5005-5009_Compact, F.Cu at (263.2, 121.3)
- C901: value 10uF/25V -> 100u/10V; footprint Capacitor_SMD:CP_Elec_4x5.8 -> Capacitor_SMD:CP_Elec_6.3x5.8
- C902: value 4.7uF/25V -> 10uF/25V; footprint Capacitor_SMD:C_0805_2012Metric_Pad1.18x1.45mm_HandSolder -> Capacitor_SMD:CP_Elec_4x5.8
- C904: value 1uF/50V -> 4.7uF/25V
- C905: value 10nF/50V -> 1uF/50V
- C906: value 22pF/50V -> 10nF/50V
- C908: value 4.7uF/25V -> 22pF/50V
- C912, C915: value 100nF/50V -> 4.7uF/25V
- C913: value 4.7uF/25V -> 100u/10V; footprint Capacitor_SMD:C_0805_2012Metric_Pad1.18x1.45mm_HandSolder -> Capacitor_SMD:CP_Elec_6.3x5.8
- C914: value 4.7uF/25V -> 100nF/50V
- C917: value 100u/10V -> 100nF/50V; footprint Capacitor_SMD:CP_Elec_6.3x5.8 -> Capacitor_SMD:C_0805_2012Metric_Pad1.18x1.45mm_HandSolder
- C918: value 100u/10V -> 4.7uF/25V; footprint Capacitor_SMD:CP_Elec_6.3x5.8 -> Capacitor_SMD:C_0805_2012Metric_Pad1.18x1.45mm_HandSolder
- J704: value Conn_ARM_JTAG_SWD_20 -> Boot Jumper; footprint Connector_PinHeader_2.54mm:PinHeader_2x05_P2.54mm_Vertical_SMD -> Connector_PinHeader_2.54mm:PinHeader_1x03_P2.54mm_Vertical
- R703, R704, R705, R706: value R_Small -> 22R
- R707: value 47R -> 22R
- R708: value 10k -> 47R
- R709: value 22R -> 10k
- R803, R804, R809, R813, R814: value 4k7 -> 5k1
- R805: value 470R -> 5k1
- R807: value 10k -> 470R
- R808: value 4k7 -> 10k
- R810: value 12k -> 5k1
- R812: value 5k1 -> 12k
- moved J1003 175.6 mm to (144.3, 45.8), turned to 90 degrees
- moved J1002 147.5 mm to (124.3, 45.8), turned to 90 degrees
- moved J1001 119.4 mm to (104.3, 45.8), turned to 90 degrees
- moved J801 74.8 mm to (220.9, 50.8), turned to 180 degrees
- moved C915 53.7 mm to (72.9, 94.8)
- moved C1001 53.7 mm to (49.6, 116.4)
- moved C1002 53.7 mm to (49.6, 119.4)
- moved C701 53.7 mm to (107.0, 82.1)
- moved C704 53.7 mm to (107.0, 91.1)
- moved C705 53.7 mm to (111.5, 82.1)
- moved C708 53.7 mm to (111.5, 91.1)
- moved C709 53.7 mm to (115.9, 82.1)
- moved C712 53.7 mm to (115.9, 91.1)
- moved C713 53.7 mm to (120.4, 82.1)
- moved C716 53.7 mm to (120.4, 91.1)
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Connections:
- net /Human Interface/CLK renamed /MCU/CLK
- C901 pad 1: VBUS -> Net-(U902-VIN)
- C902 pad 1: /POWER/Boost in -> VBUS
- C903 pad 1: Net-(U902-VIN) -> /POWER/Boost in
- C904 pad 1: /POWER/VBUS_{fused} -> Net-(U902-VIN)
- C905 pad 1: Net-(U902-FB) -> /POWER/VBUS_{fused}
- C905 pad 2: VDD -> GND
- C906 pad 1: /POWER/7V -> Net-(U902-FB)
- C906 pad 2: /POWER/Boost Feedback -> VDD
- C907 pad 1: /POWER/HS_OVLO -> /POWER/7V
- C907 pad 2: GND -> /POWER/Boost Feedback
- C908 pad 1: /POWER/7V -> /POWER/HS_OVLO
- C909 pad 1: VDD -> /POWER/7V
- C910 pad 1: Net-(U904-VI) -> VDD
- C911 pad 1: +5V -> Net-(U904-VI)
- C912 pad 1: Net-(U905-IN) -> +5V
- C913 pad 1: Net-(U904-VO) -> VDD
- C914 pad 1: VAA -> Net-(U905-IN)
- C915 pad 1: Net-(U905-OUT) -> Net-(U904-VO)
- C917 pad 1: Net-(U902-VIN) -> Net-(U905-OUT)
- C918 pad 1: VDD -> VAA
- FB901 pad 2: /POWER/Boost in -> Net-(U902-VIN)
- FB902 pad 2: Net-(U902-VIN) -> /POWER/Boost in
- J702 pad 11: /Audio IO/MCLK -> /MCU/MCLK
- J702 pad 12: /Audio IO/MCLK -> VAA
- J704 pad 1: VDD -> GND
- J704 pad 2: /MCU/JTMS_SWDIO -> /MCU/MCU_BOOT0
- J704 pad 3: GND -> VDD
- R703 pad 1: /Audio IO/LRCLK -> /MCU/LRCLK
- R706 pad 1: /MCU/CLK_24MHz -> /Human Interface/serial_data
- R706 pad 2: Net-(U701C-PA8) -> Net-(U701A-PE14)
- R707 pad 1: /MCU/MCU_VREF+ -> /MCU/CLK_24MHz
- R707 pad 2: VDDA -> Net-(U701C-PA8)
- R708 pad 1: VDD -> /MCU/MCU_VREF+
- R708 pad 2: /MCU/MCU_BOOT0 -> VDDA
- R709 pad 1: Net-(C718-Pad1) -> VDD
- R709 pad 2: /MCU/OSC_{OUT} -> /MCU/MCU_BOOT0
- R805 pad 1: /USB/USB_B_VBUS -> Net-(R804-Pad2)
- R805 pad 2: Net-(D805-A) -> GND
- R806 pad 1: VBUS_OUT -> /USB/USB_B_VBUS
- R806 pad 2: Net-(D806-A) -> Net-(D805-A)
- R807 pad 1: VBUS -> VBUS_OUT
- R807 pad 2: Net-(U802-VBUS) -> Net-(D806-A)
- R808 pad 1: /USB/USB_B_VBUS -> VBUS
- R808 pad 2: /MCU/USB_B_VBUS_MCU -> Net-(U802-VBUS)
- R809 pad 1: /MCU/USB_B_VBUS_MCU -> /USB/USB_B_VBUS
- R809 pad 2: Net-(R809-Pad2) -> /MCU/USB_B_VBUS_MCU
- R810 pad 1: Net-(U802-RBIAS) -> /MCU/USB_B_VBUS_MCU
- R810 pad 2: GND -> Net-(R810-Pad2)
- R811 pad 1: /USB/USB_C_CON_CC1 -> Net-(R810-Pad2)
- R812 pad 1: /USB/USB_C_CON_CC2 -> Net-(U802-RBIAS)
- R813 pad 1: Net-(R804-Pad2) -> /USB/USB_C_CON_CC1
- R814 pad 1: Net-(R809-Pad2) -> /USB/USB_C_CON_CC2
- U701 pad 2: /Audio IO/ADCIN1 -> /MCU/AudioAdc1
- U701 pad 41: /Audio IO/DACOUT1 -> /MCU/AudioDac1
- U701 pad 44: /Human Interface/serial_data -> Net-(U701A-PE14)
- U701 pad 5: /Audio IO/ADCIN0 -> /MCU/AudioAdc0
- U701 pad 55: /Audio IO/ADC_FORMAT -> /MCU/ADC_FORMAT
- U701 pad 56: /Audio IO/ADC_M/S -> /MCU/ADC_M/S
- U701 pad 58: /Audio IO/DACOUT0 -> /MCU/AudioDac0
- U701 pad 66: /Audio IO/MCLK -> /MCU/MCLK
- U701 pad 86: /Audio IO/ADC_IWL -> /MCU/ADC_IWL
- U701 pad 88: /Audio IO/ADC_FSAMPEN -> /MCU/ADC_FSAMPEN
Other:
- board outline removed

Commit message: Add board outline for Magna Mainboard
Parts:
- J101: footprint Connector_PinSocket_2.54mm:PinSocket_2x08_P2.54mm_Vertical -> Connector_PinSocket_2.54mm:PinSocket_2x08_P2.54mm_Horizontal
- J601: footprint Connector_PinSocket_2.54mm:PinSocket_2x10_P2.54mm_Vertical -> Connector_PinHeader_2.54mm:PinHeader_2x10_P2.54mm_Vertical
- J702: footprint Connector_PinSocket_2.54mm:PinSocket_2x06_P2.54mm_Vertical_SMD -> Connector_PinSocket_2.54mm:PinSocket_2x06_P2.54mm_Horizontal
- moved TP1002 232.0 mm to (40.1, 248.7)
- moved TP802 232.0 mm to (75.4, 221.5)
- moved TP902 232.0 mm to (54.2, 248.7)
- moved TP906 232.0 mm to (64.3, 248.7)
- moved TP908 232.0 mm to (69.4, 248.7)
- moved TP903 232.0 mm to (59.3, 243.7)
- moved TP904 232.0 mm to (59.3, 248.7)
- moved TP1001 232.0 mm to (40.1, 243.7)
- moved TP1003 232.0 mm to (40.1, 253.8)
- moved TP801 232.0 mm to (75.4, 216.4)
- moved TP803 232.0 mm to (75.4, 226.5)
- moved TP804 232.0 mm to (75.4, 231.6)
- moved TP805 232.0 mm to (75.4, 236.6)
- moved TP901 232.0 mm to (54.2, 243.7)
- moved TP905 232.0 mm to (64.3, 243.7)
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Other:
- board outline added: 120 x 320 mm

Commit message: Update Audio connector pinning (#14)
Parts:
- removed C903, C909, C911, C915, C918: 4.7uF/25V, Capacitor_SMD:C_0805_2012Metric_Pad1.18x1.45mm_HandSolder
- removed C907: 22pF/50V, Capacitor_SMD:C_0805_2012Metric_Pad1.18x1.45mm_HandSolder
- removed C916: 22uF/16V, Capacitor_SMD:CP_Elec_5x5.8
- removed D2101, D2105: Red, Diode_SMD:D_0805_2012Metric_Pad1.15x1.40mm_HandSolder
- removed D902: SS54, Diode_SMD:D_SMA_Handsoldering
- removed FB902, FB903, FB904: FerriteBead, Inductor_SMD:L_0805_2012Metric
- removed J101: Conn_02x08_Counter_Clockwise, Connector_PinSocket_2.54mm:PinSocket_2x08_P2.54mm_Horizontal
- removed J702: Conn_02x06_Odd_Even, Connector_PinSocket_2.54mm:PinSocket_2x06_P2.54mm_Horizontal
- removed L901: 22µH, Skrooter_footprints:MSCD43
- removed R2101: 1k, Resistor_SMD:R_0805_2012Metric_Pad1.20x1.40mm_HandSolder
- removed R2105: 680R, Resistor_SMD:R_0805_2012Metric_Pad1.20x1.40mm_HandSolder
- removed R703, R704: 22R, Resistor_SMD:R_0805_2012Metric_Pad1.20x1.40mm_HandSolder
- removed R902: 470k, Resistor_SMD:R_0805_2012Metric_Pad1.20x1.40mm_HandSolder
- removed R903: 100k, Resistor_SMD:R_0805_2012Metric_Pad1.20x1.40mm_HandSolder
- removed TP901, TP902, TP907: TestPoint, TestPoint:TestPoint_Keystone_5005-5009_Compact
- removed U901: TPS61040DBV, Package_TO_SOT_SMD:SOT-23-5
- removed U904: AMS1117-5.0, Package_TO_SOT_SMD:SOT-223-3_TabPin2
- added C1003: 100nF/50V, Capacitor_SMD:C_0805_2012Metric_Pad1.18x1.45mm_HandSolder, F.Cu at (35.5, 91.7)
- added C1004: 100nF/50V, Capacitor_SMD:C_0805_2012Metric_Pad1.18x1.45mm_HandSolder, F.Cu at (35.5, 94.7)
- added C1005: 100nF/50V, Capacitor_SMD:C_0805_2012Metric_Pad1.18x1.45mm_HandSolder, F.Cu at (35.5, 97.7)
- added C1006: 100nF/50V, Capacitor_SMD:C_0805_2012Metric_Pad1.18x1.45mm_HandSolder, F.Cu at (35.5, 100.7)
- added C201: F/NM, Capacitor_SMD:C_0603_1608Metric_Pad1.08x0.95mm_HandSolder, F.Cu at (36.3, 121.1)
- added D1002: 1N4148WS, Diode_SMD:D_SOD-123, F.Cu at (22.8, 102.0)
- added D1003: Red, Diode_SMD:D_0805_2012Metric_Pad1.15x1.40mm_HandSolder, F.Cu at (40.3, 91.7)
- added D1004: Red, Diode_SMD:D_0805_2012Metric_Pad1.15x1.40mm_HandSolder, F.Cu at (40.3, 94.7)
- added D1005: B5819, Diode_SMD:D_SOD-123, F.Cu at (22.8, 105.4)
- added J301: Conn_02x15_Odd_Even, Connector_PinSocket_2.54mm:PinSocket_2x15_P2.54mm_Horizontal, F.Cu at (6.54, 92.2)
- added R1007: 220R, Resistor_SMD:R_0805_2012Metric_Pad1.20x1.40mm_HandSolder, F.Cu at (30.7, 91.6)
- added R1008: 220R, Resistor_SMD:R_0805_2012Metric_Pad1.20x1.40mm_HandSolder, F.Cu at (30.7, 94.6)
- added R1009: 220R, Resistor_SMD:R_0805_2012Metric_Pad1.20x1.40mm_HandSolder, F.Cu at (30.7, 97.5)
- added R1010: 220R, Resistor_SMD:R_0805_2012Metric_Pad1.20x1.40mm_HandSolder, F.Cu at (30.7, 100.5)
- added R1011: 220R, Resistor_SMD:R_0805_2012Metric_Pad1.20x1.40mm_HandSolder, F.Cu at (30.7, 103.4)
- added R201: R/NM, Resistor_SMD:R_0805_2012Metric_Pad1.20x1.40mm_HandSolder, F.Cu at (22.2, 110.8)
- added R202: R/NM, Resistor_SMD:R_0805_2012Metric_Pad1.20x1.40mm_HandSolder, F.Cu at (22.2, 113.8)
- added R203: 22R, Resistor_SMD:R_0805_2012Metric_Pad1.20x1.40mm_HandSolder, F.Cu at (22.2, 116.7)
- added R204: 22R, Resistor_SMD:R_0805_2012Metric_Pad1.20x1.40mm_HandSolder, F.Cu at (22.2, 119.7)
- added R205: 22R, Resistor_SMD:R_0805_2012Metric_Pad1.20x1.40mm_HandSolder, F.Cu at (22.2, 122.6)
- added R206: 22R, Resistor_SMD:R_0805_2012Metric_Pad1.20x1.40mm_HandSolder, F.Cu at (22.2, 125.6)
- added R207: 22R, Resistor_SMD:R_0805_2012Metric_Pad1.20x1.40mm_HandSolder, F.Cu at (27.0, 110.8)
- added R208: 0R, Resistor_SMD:R_0805_2012Metric_Pad1.20x1.40mm_HandSolder, F.Cu at (27.0, 113.8)
- added R209: 0R, Resistor_SMD:R_0805_2012Metric_Pad1.20x1.40mm_HandSolder, F.Cu at (27.0, 116.7)
- added R210: 0R, Resistor_SMD:R_0805_2012Metric_Pad1.20x1.40mm_HandSolder, F.Cu at (27.0, 119.7)
- added R211: 0R, Resistor_SMD:R_0805_2012Metric_Pad1.20x1.40mm_HandSolder, F.Cu at (27.0, 122.6)
- added R212: 22R, Resistor_SMD:R_0805_2012Metric_Pad1.20x1.40mm_HandSolder, F.Cu at (27.0, 125.6)
- added R213: 0R, Resistor_SMD:R_0805_2012Metric_Pad1.20x1.40mm_HandSolder, F.Cu at (31.7, 110.8)
- added R214: 0R, Resistor_SMD:R_0805_2012Metric_Pad1.20x1.40mm_HandSolder, F.Cu at (31.7, 113.8)
- added R215: 0R, Resistor_SMD:R_0805_2012Metric_Pad1.20x1.40mm_HandSolder, F.Cu at (31.7, 116.7)
- added R216: 0R, Resistor_SMD:R_0805_2012Metric_Pad1.20x1.40mm_HandSolder, F.Cu at (31.7, 119.7)
- added TP201: TestPoint, TestPoint:TestPoint_Keystone_5005-5009_Compact, F.Cu at (36.6, 117.3)
- added U1003: 74HC08D, Package_SO:SOIC-14_3.9x8.7mm_P1.27mm, F.Cu at (24.1, 95.3)
- added U1004: TLP2361, Package_SO:SO-5_4.4x3.6mm_P1.27mm, F.Cu at (38.0, 104.8)
- added U201: 24.576 MHz, Oscillator:Oscillator_SMD_Abracon_ASE-4Pin_3.2x2.5mm_HandSoldering, F.Cu at (37.2, 112.1)
- C1001, C1002: value 100nF/50V -> 10n
- D1001: value B5819 -> 1N4148WS
- R1001: value 470R -> 220R
- R1003, R1004: value 220R -> 470k
- R1005, R1006: value 220R -> 680R
- U1001: value 74HC08D -> 74LVC2G14
- U1002: value 6N137 -> 74LVC2G14
- moved J601 0.73 mm to (16.7, 274.1)
Connections:
- C1001 pad 1: +5V -> Net-(C1001-Pad1)
- C1002 pad 2: VDD -> Net-(C1002-Pad2)
- D1001 pad 1: /MIDI/MIDI_{IN-} -> Net-(D1001-K)
- D1001 pad 2: /MIDI/MIDI_{IN+} -> Net-(D1001-A)
- J1001 pad 4: /MIDI/MIDI_{IN-} -> /MIDI/MIDI_{IN+}
- J1001 pad 5: /MIDI/MIDI_{IN+} -> /MIDI/MIDI_{IN-cathode}
- R1001 pad 1: /MCU/MIDI_RX -> Net-(D1001-K)
- R1001 pad 2: VDD -> Net-(C1001-Pad1)
- R1002 pad 1: /MIDI/MIDI_{IN-cathode} -> Net-(C1002-Pad2)
- R1002 pad 2: /MIDI/MIDI_{IN-} -> Net-(D1002-K)
- R1003 pad 1: Net-(R1003-Pad1) -> Net-(D1001-K)
- R1003 pad 2: /MIDI/MIDI_{THRU+} -> GND
- R1004 pad 1: Net-(R1004-Pad1) -> GND
- R1004 pad 2: /MIDI/MIDI_{THRU-} -> Net-(D1002-K)
- R1005 pad 1: Net-(R1005-Pad1) -> +5V
- R1005 pad 2: /MIDI/MIDI_{OUT+} -> Net-(D1003-A)
- R1006 pad 1: Net-(R1006-Pad1) -> +5V
- R1006 pad 2: /MIDI/MIDI_{OUT-} -> Net-(D1004-A)
- R706 pad 1: /Human Interface/serial_data -> Net-(U701A-PE14)
- R706 pad 2: Net-(U701A-PE14) -> /Human Interface/serial_data
- U1001 pad 1: /MCU/MIDI_RX -> /MCU/MIDI_TX
- U1001 pad 10: Net-(R1003-Pad1) -> (no net)
- U1001 pad 11: Net-(R1005-Pad1) -> (no net)
- U1001 pad 12: +5V -> (no net)
- U1001 pad 13: +5V -> (no net)
- U1001 pad 14: +5V -> (no net)
- U1001 pad 2: /MCU/MIDI_RX -> GND
- U1001 pad 3: Net-(R1004-Pad1) -> Net-(D1001-K)
- U1001 pad 4: Net-(R1006-Pad1) -> Net-(D1003-K)
- U1001 pad 5: /MCU/MIDI_TX -> +5V
- U1001 pad 6: /MCU/MIDI_TX -> Net-(D1001-A)
- U1001 pad 7: GND -> (no net)
- U1001 pad 8: +5V -> (no net)
- U1001 pad 9: +5V -> (no net)
- U1002 pad 1: unconnected-(U1002-NC-Pad1) -> /MCU/MIDI_RX
- U1002 pad 2: /MIDI/MIDI_{IN+} -> GND
- U1002 pad 3: /MIDI/MIDI_{IN-cathode} -> Net-(D1002-K)
- U1002 pad 4: unconnected-(U1002-NC-Pad4) -> Net-(D1004-K)
- U1002 pad 5: GND -> +5V
- U1002 pad 6: /MCU/MIDI_RX -> Net-(D1002-A)
- U1002 pad 7: unconnected-(U1002-EN-Pad7) -> (no net)
- U1002 pad 8: VDD -> (no net)
- U701 pad 1: /MCU/~{HSW_EN} -> /MCU/MCU_MCLK_OUT
- U701 pad 2: /MCU/AudioAdc1 -> /MCU/ADC_DATA_1_MCU
- U701 pad 41: /MCU/AudioDac1 -> /MCU/ADC_DATA_3_MCU
- U701 pad 5: /MCU/AudioAdc0 -> /MCU/ADC_DATA_0_MCU
- U701 pad 54: /MCU/I2S2_SD -> /MCU/DAC_DATA_0_MCU
- U701 pad 55: /MCU/ADC_FORMAT -> /Audio Daughterboard Connector/ADC_FORMAT
- U701 pad 56: /MCU/ADC_M/S -> /Audio Daughterboard Connector/ADC_M/S
- U701 pad 58: /MCU/AudioDac0 -> /MCU/ADC_DATA_2_MCU
- U701 pad 66: /MCU/MCLK -> /MCU/MCLK_24.576MHz
- U701 pad 7: /MCU/USB_PHY_RESET -> /MCU/~{HSW_EN}
- U701 pad 8: unconnected-(U701C-PC14-OSC32_IN-Pad8) -> /MCU/USB_PHY_RESET
- U701 pad 86: /MCU/ADC_IWL -> /Audio Daughterboard Connector/ADC_IWL
- U701 pad 87: /MCU/I2S3_SD -> /MCU/DAC_DATA_1_MCU
- U701 pad 88: /MCU/ADC_FSAMPEN -> /Audio Daughterboard Connector/ADC_FSAMPEN

Commit message: Mainboard layout (#19)
Also adds mounting holes to IO daughterboard
Parts:
- removed C803: 220uF, Capacitor_SMD:CP_Elec_4x5.8
- removed C901, C913: 100u/10V, Capacitor_SMD:CP_Elec_6.3x5.8
- removed C904, C910: 4.7uF/25V, Capacitor_SMD:C_0805_2012Metric_Pad1.18x1.45mm_HandSolder
- removed C908: 22pF/50V, Capacitor_SMD:C_0805_2012Metric_Pad1.18x1.45mm_HandSolder
- removed D1005: B5819, Diode_SMD:D_SOD-123
- removed D806: green, Diode_SMD:D_0805_2012Metric_Pad1.15x1.40mm_HandSolder
- removed D903: SS54, Diode_SMD:D_SMA_Handsoldering
- removed J601: Conn_02x10_Counter_Clockwise, Connector_PinHeader_2.54mm:PinHeader_2x10_P2.54mm_Vertical
- removed J703: Conn_ARM_JTAG_SWD_20, Connector_PinHeader_2.54mm:PinHeader_2x05_P2.54mm_Vertical_SMD
- removed J704: Boot Jumper, Connector_PinHeader_2.54mm:PinHeader_1x03_P2.54mm_Vertical
- removed the R207 at (27.0, 110.8)
- removed the R213 at (31.7, 110.8)
- removed the R214 at (31.7, 113.8)
- removed the R215 at (31.7, 116.7)
- removed the R216 at (31.7, 119.7)
- removed R707: 22R, Resistor_SMD:R_0805_2012Metric_Pad1.20x1.40mm_HandSolder
- removed R709: 10k, Resistor_SMD:R_0805_2012Metric_Pad1.20x1.40mm_HandSolder
- removed R807: 470R, Resistor_SMD:R_0805_2012Metric_Pad1.20x1.40mm_HandSolder
- removed R901: 1k, Resistor_SMD:R_0805_2012Metric_Pad1.20x1.40mm_HandSolder
- removed R904: 1k5, Resistor_SMD:R_0805_2012Metric_Pad1.20x1.40mm_HandSolder
- removed TP1001, TP1002, TP1003, TP801, TP802, TP803, TP804, TP805, TP903, TP904, TP905, TP906, TP908: TestPoint, TestPoint:TestPoint_Keystone_5005-5009_Compact
- removed U802: USB3300-EZK, Package_DFN_QFN:QFN-32-1EP_5x5mm_P0.5mm_EP3.45x3.45mm
- removed U902: XL1509-ADJ, Package_SO:SOIC-8_3.9x4.9mm_P1.27mm
- added C212: 22uF/25V, Capacitor_SMD:C_0805_2012Metric_Pad1.18x1.45mm_HandSolder, F.Cu at (194.5, 104.6)
- added C221: 220nF/16V, Capacitor_SMD:C_0402_1005Metric_Pad0.74x0.62mm_HandSolder, F.Cu at (188.6, 74.4)
- added C403: 22uF/25V, Capacitor_SMD:C_0805_2012Metric_Pad1.18x1.45mm_HandSolder, F.Cu at (138.3, 18.0)
- added C405: 22uF/25V, Capacitor_SMD:C_0805_2012Metric_Pad1.18x1.45mm_HandSolder, F.Cu at (138.3, 21.0)
- added C407: 22uF/25V, Capacitor_SMD:C_0805_2012Metric_Pad1.18x1.45mm_HandSolder, F.Cu at (138.3, 24.0)
- added C410: 22uF/25V, Capacitor_SMD:C_0805_2012Metric_Pad1.18x1.45mm_HandSolder, F.Cu at (158.6, 39.5)
- added C411: 22uF/25V, Capacitor_SMD:C_0805_2012Metric_Pad1.18x1.45mm_HandSolder, F.Cu at (154.5, 60.5)
- added C412: 22uF/25V, Capacitor_SMD:C_0805_2012Metric_Pad1.18x1.45mm_HandSolder, F.Cu at (150.5, 56.4)
- added C601: 22uF/25V, Capacitor_SMD:C_0805_2012Metric_Pad1.18x1.45mm_HandSolder, F.Cu at (142.5, 77.7)
- added C602: 22uF/25V, Capacitor_SMD:C_0805_2012Metric_Pad1.18x1.45mm_HandSolder, F.Cu at (142.5, 75.7)
- added C603: 22uF/25V, Capacitor_SMD:C_0805_2012Metric_Pad1.18x1.45mm_HandSolder, F.Cu at (142.5, 79.8)
- added C604: 220nF/16V, Capacitor_SMD:C_0402_1005Metric_Pad0.74x0.62mm_HandSolder, F.Cu at (142.0, 81.3)
- added C606: 220nF/16V, Capacitor_SMD:C_0402_1005Metric_Pad0.74x0.62mm_HandSolder, F.Cu at (143.9, 87.5)
- added C609: 22uF/25V, Capacitor_SMD:C_0805_2012Metric_Pad1.18x1.45mm_HandSolder, F.Cu at (147.0, 82.5)
- added C610: 22uF/25V, Capacitor_SMD:C_0805_2012Metric_Pad1.18x1.45mm_HandSolder, F.Cu at (147.0, 80.5)
- added C611: 22uF/25V, Capacitor_SMD:C_0805_2012Metric_Pad1.18x1.45mm_HandSolder, F.Cu at (147.0, 78.5)
- added C612: 10p/50V, Capacitor_SMD:C_0603_1608Metric_Pad1.08x0.95mm_HandSolder, F.Cu at (138.0, 61.0)
- added C613: 22uF/25V, Capacitor_SMD:C_0805_2012Metric_Pad1.18x1.45mm_HandSolder, F.Cu at (147.0, 76.5)
- added C614: 22uF/25V, Capacitor_SMD:C_0805_2012Metric_Pad1.18x1.45mm_HandSolder, F.Cu at (147.0, 74.5)
- added C615: 22uF/25V, Capacitor_SMD:C_0805_2012Metric_Pad1.18x1.45mm_HandSolder, F.Cu at (147.0, 72.5)
- added C616: 22uF/25V, Capacitor_SMD:C_0805_2012Metric_Pad1.18x1.45mm_HandSolder, F.Cu at (143.0, 51.0)
- added C620: 22uF/25V, Capacitor_SMD:C_0805_2012Metric_Pad1.18x1.45mm_HandSolder, F.Cu at (145.5, 42.5)
- added D406: green, Diode_SMD:D_0805_2012Metric_Pad1.15x1.40mm_HandSolder, F.Cu at (230.7, 69.1)
- added D505: 1N4148WS, Diode_SMD:D_SOD-123, F.Cu at (226.2, 28.0)
- added H101: MountingHole_Pad, MountingHole:MountingHole_3.2mm_M3_Pad_Via, F.Cu at (124.2, 135.8)
- added H102: MountingHole_Pad, MountingHole:MountingHole_3.2mm_M3_Pad_Via, F.Cu at (236.8, 135.8)
- added H103: MountingHole_Pad, MountingHole:MountingHole_3.2mm_M3_Pad_Via, F.Cu at (124.2, 3.25)
- added H104: MountingHole_Pad, MountingHole:MountingHole_3.2mm_M3_Pad_Via, F.Cu at (236.8, 3.25)
- added H105: MountingHole_Pad, MountingHole:MountingHole_3.2mm_M3_Pad_Via, F.Cu at (131.0, 25.0)
- added H106: MountingHole_Pad, MountingHole:MountingHole_3.2mm_M3_Pad_Via, F.Cu at (226.0, 127.0)
- added H107: MountingHole_Pad, MountingHole:MountingHole_3.2mm_M3_Pad_Via, F.Cu at (232.0, 32.0)
- added H108: MountingHole_Pad, MountingHole:MountingHole_3.2mm_M3_Pad_Via, F.Cu at (160.0, 107.0)
- added J201: Conn_02x06_Odd_Even, Connector_PinSocket_2.54mm:PinSocket_2x06_P2.54mm_Vertical_SMD, F.Cu at (231.2, 92.0)
- added J202: Conn_ARM_JTAG_SWD_20, Connector_PinHeader_2.54mm:PinHeader_2x05_P2.54mm_Vertical_SMD, F.Cu at (162.7, 68.6)
- added J203: Boot Jumper, Connector_PinHeader_2.54mm:PinHeader_1x03_P2.54mm_Vertical, F.Cu at (232.2, 114.9)
- added R205: 22R, Resistor_SMD:R_0805_2012Metric_Pad1.20x1.40mm_HandSolder, F.Cu at (182.5, 60.5)
- added R208: 10k, Resistor_SMD:R_0805_2012Metric_Pad1.20x1.40mm_HandSolder, F.Cu at (232.3, 123.7)
- added R222: 22R, Resistor_SMD:R_0805_2012Metric_Pad1.20x1.40mm_HandSolder, F.Cu at (150.5, 92.5)
- added R225: 0R, Resistor_SMD:R_0805_2012Metric_Pad1.20x1.40mm_HandSolder, F.Cu at (169.3, 111.8)
- added R226: 0R, Resistor_SMD:R_0805_2012Metric_Pad1.20x1.40mm_HandSolder, F.Cu at (171.3, 111.8)
- added R407: 470R, Resistor_SMD:R_0805_2012Metric_Pad1.20x1.40mm_HandSolder, F.Cu at (230.7, 65.0)
- added R415: 0R, Resistor_SMD:R_0805_2012Metric_Pad1.20x1.40mm_HandSolder, F.Cu at (193.1, 60.5)
- added R416: 0R, Resistor_SMD:R_0805_2012Metric_Pad1.20x1.40mm_HandSolder, F.Cu at (195.2, 60.5)
- added R417: 0R, Resistor_SMD:R_0805_2012Metric_Pad1.20x1.40mm_HandSolder, F.Cu at (197.2, 60.5)
- added R418: 0R, Resistor_SMD:R_0805_2012Metric_Pad1.20x1.40mm_HandSolder, F.Cu at (199.2, 60.5)
- added R419: 0R, Resistor_SMD:R_0805_2012Metric_Pad1.20x1.40mm_HandSolder, F.Cu at (201.3, 60.5)
- added R420: 0R, Resistor_SMD:R_0805_2012Metric_Pad1.20x1.40mm_HandSolder, F.Cu at (203.3, 60.5)
- added R421: 0R, Resistor_SMD:R_0805_2012Metric_Pad1.20x1.40mm_HandSolder, F.Cu at (205.3, 60.5)
- added R422: 0R, Resistor_SMD:R_0805_2012Metric_Pad1.20x1.40mm_HandSolder, F.Cu at (207.4, 60.5)
- added R423: 0R, Resistor_SMD:R_0805_2012Metric_Pad1.20x1.40mm_HandSolder, F.Cu at (185.0, 60.5)
- added R424: 0R, Resistor_SMD:R_0805_2012Metric_Pad1.20x1.40mm_HandSolder, F.Cu at (187.0, 60.5)
- added R425: 0R, Resistor_SMD:R_0805_2012Metric_Pad1.20x1.40mm_HandSolder, F.Cu at (189.1, 60.5)
- added R426: 0R, Resistor_SMD:R_0805_2012Metric_Pad1.20x1.40mm_HandSolder, F.Cu at (191.1, 60.5)
- added R427: 0R, Resistor_SMD:R_0805_2012Metric_Pad1.20x1.40mm_HandSolder, F.Cu at (209.4, 60.5)
- added R601: 10k, Resistor_SMD:R_0805_2012Metric_Pad1.20x1.40mm_HandSolder, F.Cu at (139.5, 81.5)
- added R602: 12k, Resistor_SMD:R_0805_2012Metric_Pad1.20x1.40mm_HandSolder, F.Cu at (136.7, 83.0)
- added R603: 39k, Resistor_SMD:R_0805_2012Metric_Pad1.20x1.40mm_HandSolder, F.Cu at (136.7, 85.0)
- added TP401: TestPoint, TestPoint:TestPoint_Keystone_5000-5004_Miniature, F.Cu at (168.2, 10.7)
- added TP402: TestPoint, TestPoint:TestPoint_Keystone_5000-5004_Miniature, F.Cu at (176.4, 39.6)
- added TP405: TestPoint, TestPoint:TestPoint_Keystone_5000-5004_Miniature, F.Cu at (154.0, 27.9)
- added TP501: TestPoint, TestPoint:TestPoint_Keystone_5000-5004_Miniature, F.Cu at (221.3, 49.5)
- added TP502: TestPoint, TestPoint:TestPoint_Keystone_5000-5004_Miniature, F.Cu at (217.5, 49.5)
- added TP503: TestPoint, TestPoint:TestPoint_Keystone_5000-5004_Miniature, F.Cu at (213.7, 49.5)
- added TP602: TestPoint, TestPoint:TestPoint_Keystone_5000-5004_Miniature, F.Cu at (150.5, 70.0)
- added TP603: TestPoint, TestPoint:TestPoint_Keystone_5000-5004_Miniature, F.Cu at (127.0, 78.0)
- added TP604: TestPoint, TestPoint:TestPoint_Keystone_5000-5004_Miniature, F.Cu at (137.3, 27.9)
- added TP605: TestPoint, TestPoint:TestPoint_Keystone_5000-5004_Miniature, F.Cu at (140.8, 27.9)
- added U402: USB3300-EZK, Package_DFN_QFN:QFN-32-1EP_5x5mm_P0.5mm_EP3.45x3.45mm, F.Cu at (165.2, 37.6)
- added U403: SRV05-4, Package_TO_SOT_SMD:SOT-23-6, F.Cu at (166.4, 22.4)
- added U601: TPS563201, Package_TO_SOT_SMD:SOT-23-6, F.Cu at (142.5, 84.0)
- C201: renamed from C701; value 2.2uF/6.3V -> 22uF/25V
- C202: renamed from C702; value 2.2uF/6.3V -> 22uF/25V
- C203: renamed from C703; value 2.2uF/6.3V -> 22uF/25V
- C204: renamed from C704; value 2.2uF/6.3V -> 22uF/25V
- C205: renamed from C705; value 100nF/50V -> 220nF/16V; footprint Capacitor_SMD:C_0805_2012Metric_Pad1.18x1.45mm_HandSolder -> Capacitor_SMD:C_0402_1005Metric_Pad0.74x0.62mm_HandSolder
- C206: renamed from C706; value 100nF/50V -> 220nF/16V; footprint Capacitor_SMD:C_0805_2012Metric_Pad1.18x1.45mm_HandSolder -> Capacitor_SMD:C_0402_1005Metric_Pad0.74x0.62mm_HandSolder
- C207: renamed from C707; value 100nF/50V -> 220nF/16V; footprint Capacitor_SMD:C_0805_2012Metric_Pad1.18x1.45mm_HandSolder -> Capacitor_SMD:C_0402_1005Metric_Pad0.74x0.62mm_HandSolder
- C208: renamed from C708; value 100nF/50V -> 220nF/16V; footprint Capacitor_SMD:C_0805_2012Metric_Pad1.18x1.45mm_HandSolder -> Capacitor_SMD:C_0402_1005Metric_Pad0.74x0.62mm_HandSolder
- C209: renamed from C709; value 100nF/50V -> 220nF/16V; footprint Capacitor_SMD:C_0805_2012Metric_Pad1.18x1.45mm_HandSolder -> Capacitor_SMD:C_0402_1005Metric_Pad0.74x0.62mm_HandSolder
- C210: renamed from C710; value 100nF/50V -> 220nF/16V; footprint Capacitor_SMD:C_0805_2012Metric_Pad1.18x1.45mm_HandSolder -> Capacitor_SMD:C_0402_1005Metric_Pad0.74x0.62mm_HandSolder
- C211: renamed from C711; value 100nF/50V -> 220nF/16V; footprint Capacitor_SMD:C_0805_2012Metric_Pad1.18x1.45mm_HandSolder -> Capacitor_SMD:C_0402_1005Metric_Pad0.74x0.62mm_HandSolder
- C213: renamed from C712; value 1uF/50V -> 22uF/25V
- C214: renamed from C713; value 100nF/50V -> 220nF/16V; footprint Capacitor_SMD:C_0805_2012Metric_Pad1.18x1.45mm_HandSolder -> Capacitor_SMD:C_0402_1005Metric_Pad0.74x0.62mm_HandSolder
- C215: renamed from C714; value 1uF/50V -> 22uF/25V
- C216: renamed from C715; value 100nF/50V -> 220nF/16V; footprint Capacitor_SMD:C_0805_2012Metric_Pad1.18x1.45mm_HandSolder -> Capacitor_SMD:C_0402_1005Metric_Pad0.74x0.62mm_HandSolder
- C217: renamed from C716; value 4.7uF/25V -> 22uF/25V
- C220: renamed from C201; footprint Capacitor_SMD:C_0603_1608Metric_Pad1.08x0.95mm_HandSolder -> Capacitor_SMD:C_0805_2012Metric_Pad1.18x1.45mm_HandSolder
- C401: renamed from C801; value 100nF/50V -> 220nF/16V; footprint Capacitor_SMD:C_0805_2012Metric_Pad1.18x1.45mm_HandSolder -> Capacitor_SMD:C_0402_1005Metric_Pad0.74x0.62mm_HandSolder
- C402: renamed from C802; value 100nF/50V -> 220nF/16V; footprint Capacitor_SMD:C_0805_2012Metric_Pad1.18x1.45mm_HandSolder -> Capacitor_SMD:C_0402_1005Metric_Pad0.74x0.62mm_HandSolder
- C404: renamed from C804; value 100nF/50V -> 220nF/16V; footprint Capacitor_SMD:C_0805_2012Metric_Pad1.18x1.45mm_HandSolder -> Capacitor_SMD:C_0402_1005Metric_Pad0.74x0.62mm_HandSolder
- C406: renamed from C805; value 100nF/50V -> 220nF/16V; footprint Capacitor_SMD:C_0805_2012Metric_Pad1.18x1.45mm_HandSolder -> Capacitor_SMD:C_0402_1005Metric_Pad0.74x0.62mm_HandSolder
- C408: renamed from C806; value 4.7uF/25V -> 22uF/25V
- C409: renamed from C807; value 4.7uF/25V -> 22uF/25V
- C501: renamed from C1001; value 10n -> 10nF/50V
- C502: renamed from C1002; value 10n -> 10nF/50V
- C503: renamed from C1003; value 100nF/50V -> 220nF/16V; footprint Capacitor_SMD:C_0805_2012Metric_Pad1.18x1.45mm_HandSolder -> Capacitor_SMD:C_0402_1005Metric_Pad0.74x0.62mm_HandSolder
- C504: renamed from C1004; value 100nF/50V -> 220nF/16V; footprint Capacitor_SMD:C_0805_2012Metric_Pad1.18x1.45mm_HandSolder -> Capacitor_SMD:C_0402_1005Metric_Pad0.74x0.62mm_HandSolder
- C505: renamed from C1005; value 100nF/50V -> 220nF/16V; footprint Capacitor_SMD:C_0805_2012Metric_Pad1.18x1.45mm_HandSolder -> Capacitor_SMD:C_0402_1005Metric_Pad0.74x0.62mm_HandSolder
- C506: renamed from C1006; value 100nF/50V -> 220nF/16V; footprint Capacitor_SMD:C_0805_2012Metric_Pad1.18x1.45mm_HandSolder -> Capacitor_SMD:C_0402_1005Metric_Pad0.74x0.62mm_HandSolder
- C605: renamed from C902; value 10uF/25V -> 22uF/25V; footprint Capacitor_SMD:CP_Elec_4x5.8 -> Capacitor_SMD:C_0805_2012Metric_Pad1.18x1.45mm_HandSolder
- C608: renamed from C905; value 1uF/50V -> 22uF/25V
- C617: renamed from C914; value 100nF/50V -> 220nF/16V; footprint Capacitor_SMD:C_0805_2012Metric_Pad1.18x1.45mm_HandSolder -> Capacitor_SMD:C_0402_1005Metric_Pad0.74x0.62mm_HandSolder
- C618: renamed from C912; value 4.7uF/25V -> 22uF/25V
- C619: renamed from C917; value 100nF/50V -> 220nF/16V; footprint Capacitor_SMD:C_0805_2012Metric_Pad1.18x1.45mm_HandSolder -> Capacitor_SMD:C_0402_1005Metric_Pad0.74x0.62mm_HandSolder
- J301: footprint Connector_PinSocket_2.54mm:PinSocket_2x15_P2.54mm_Horizontal -> Connector_PinSocket_2.54mm:PinSocket_2x16_P2.54mm_Horizontal
- J701: value Conn_02x06_Odd_Even -> Conn_02x10_Counter_Clockwise; footprint Connector_PinSocket_2.54mm:PinSocket_2x06_P2.54mm_Vertical_SMD -> Connector_PinHeader_2.54mm:PinHeader_2x10_P2.54mm_Horizontal
- L601: renamed from L902; value 22µH -> 2.2µH; footprint Skrooter_footprints:MSCD43 -> Inductor_SMD:L_Sunlord_SWPA3012S
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- renumbered C717 to C218, C718 to C219, C906 to C607, D801 to D401, D802 to D402, D803 to D403, D804 to D404, D805 to D405, D1001 to D501, D1002 to D502, D1003 to D503, D1004 to D504, D901 to D601, D2102 to D801, D2103 to D802, D2104 to D803, D2106 to D804, D2107 to D805, F901 to F601, F902 to F602, FB701 to FB201, FB901 to FB601, FB905 to FB602, J801 to J401, J802 to J402, J803 to J403, J1001 to J501, J1002 to J502, J1003 to J503, R701 to R201, R702 to R202, R705 to R203, R706 to R204, R708 to R206, R201 to R207, R212 to R213, R203 to R214, R204 to R215, R205 to R216, R208 to R217, R209 to R218, R210 to R219, R211 to R220, R206 to R221, R202 to R223, R710 to R224, R801 to R401, R802 to R402, R803 to R403, R804 to R404, R805 to R405, R806 to R406, R808 to R408, R809 to R409, R810 to R410, R811 to R411, R812 to R412, R813 to R413, R814 to R414, R1001 to R501, R1002 to R502, R1003 to R503, R1004 to R504, R1005 to R505, R1006 to R506, R1007 to R507, R1008 to R508, R1009 to R509, R1010 to R510, R1011 to R511, R907 to R606, R908 to R607, R2102 to R801, R2103 to R802, R2104 to R803, R2106 to R804, R2107 to R805, U701 to U201, U201 to U202, U801 to U401, U1003 to U503, U1004 to U504, U903 to U602, U905 to U603, Y701 to Y201
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Connections:
- net Net-(U701A-PE12) renamed /MCU/serial_CLK_MCU
- net Net-(U701A-PE14) renamed /MCU/serial_data_MCU
- net Net-(U701C-PA11) renamed /MCU/USB_HOST_MCU_N
- net Net-(U701C-PA12) renamed /MCU/USB_HOST_MCU_P
- D501 pad 1: Net-(D1001-K) -> Net-(D501-K)
- FB601 pad 2: Net-(U902-VIN) -> /POWER/+5V_ferrited
- J301 pad 29: VDD -> /Audio Daughterboard Connector/VAA_EN
- J701 pad 1: VDD -> /Human Interface/ADC_3
- J701 pad 10: GND -> /Human Interface/serial_CLR
- J701 pad 11: VDD -> GND
- J701 pad 12: GND -> /Human Interface/serial_CLK
- J701 pad 2: /MCU/QUADSPI_DATA_2 -> VDDA
- J701 pad 3: /MCU/QUADSPI_DATA_0 -> /Human Interface/ADC_4
- J701 pad 4: /MCU/QUADSPI_DATA_3 -> /Human Interface/ADC_2
- J701 pad 5: /MCU/QUADSPI_DATA_1 -> /Human Interface/ADC_5
- J701 pad 6: /MCU/QUADSPI_CLK -> /Human Interface/ADC_1
- J701 pad 7: /MCU/QUADSPI_NCS -> /Human Interface/input_interrupt
- J701 pad 8: GND -> /Human Interface/ADC_0
- J701 pad 9: VDD -> /Human Interface/msb
- L601 pad 1: Net-(D903-K) -> /POWER/DCDC_SW
- R217 pad 1: /MCU/ADC_DATA_0_MCU -> /Audio Daughterboard Connector/ADC_DATA_0
- R217 pad 2: /Audio Daughterboard Connector/ADC_DATA_0 -> /MCU/ADC_DATA_0_MCU
- R218 pad 1: /MCU/ADC_DATA_1_MCU -> /Audio Daughterboard Connector/ADC_DATA_1
- R218 pad 2: /Audio Daughterboard Connector/ADC_DATA_1 -> /MCU/ADC_DATA_1_MCU
- R219 pad 1: /MCU/ADC_DATA_2_MCU -> /Audio Daughterboard Connector/ADC_DATA_2
- R219 pad 2: /Audio Daughterboard Connector/ADC_DATA_2 -> /MCU/ADC_DATA_2_MCU
- R220 pad 1: /MCU/ADC_DATA_3_MCU -> /Audio Daughterboard Connector/ADC_DATA_3
- R220 pad 2: /Audio Daughterboard Connector/ADC_DATA_3 -> /MCU/ADC_DATA_3_MCU
- R501 pad 1: Net-(D1001-K) -> Net-(D501-K)
- R503 pad 1: Net-(D1001-K) -> GND
- R503 pad 2: GND -> Net-(D501-K)
- R508 pad 1: Net-(R1008-Pad1) -> Net-(R508-Pad1)
- R509 pad 1: Net-(R1009-Pad1) -> Net-(R509-Pad1)
- R510 pad 1: Net-(R1010-Pad1) -> Net-(R510-Pad1)
- U201 pad 28: /MCU/I2S3_LRCLK -> unconnected-(U201C-PA4-Pad28)
- U201 pad 31: unconnected-(U701C-PA7-Pad31) -> /Human Interface/register_OE
- U201 pad 53: /Human Interface/register_OE -> unconnected-(U201C-PB14-Pad53)
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Routing:
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- added copper zone on B.Cu, net +5V
- added copper zone on F.Cu, net +5V
- added copper zone on F.Cu, net /POWER/DCDC_SW
- added copper zone on F.Cu, net /POWER/VBUS_{fused}
- added copper zone on B.Cu, net /USB/USB_B_VBUS
- added copper zone on B.Cu, net /USB/USB_C_VBUS
- added copper zone on F.Cu, net GND
- added copper zone on In1.Cu, net GND
- added copper zone on In2.Cu, net GND
- added copper zone on B.Cu, net SHIELD
- added copper zone on F.Cu, net SHIELD
- added copper zone on In1.Cu, net SHIELD
- added copper zone on In2.Cu, net SHIELD
- added copper zone on B.Cu, net VBUS
- added copper zone on B.Cu, net VDD
- added copper zone on F.Cu, net VDD
Other:
- board size 120 x 320 mm -> 119 x 139 mm
- copper layers 2 -> 4
- board text added: "JLCJLCJLCJLC"

Commit message: Add final edit to Mainboard design (#20)
Routing:
- net Net-(D503-K): track 48.6 -> 47.0 mm, vias 3 -> 2
- net Net-(D504-K): track 27.4 -> 25.9 mm, vias 1 -> 0
- net /USB/DATA4_PHY: track 61.4 -> 60.8 mm
- net /MCU/~{VBUS_OUT_FLG}: vias 3 -> 2
