File: PCB/Magna/MCU.kicad_sch (KiCad schematic)
At the start: 55 parts, among them J201 Conn_02x06_Odd_Even, J202 Conn_ARM_JTAG_SWD_20, J203 Boot Jumper, U201 STM32F730V8T6, U202 24.576 MHz, Y201 24MHz

Commit message: Making the routing way nicer
Connections:
- net ADC_M/S: now also U201.65 (PC8); no longer U201.62 (PD15)
- net DAC_DATA_1_MCU: now also U201.80 (PC12); no longer U201.87 (PD6)
- net USB_A_PWR_EN: now also U201.83 (PD2); no longer U201.97 (PE0)
Changed lines of the file:
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@@
   (junction (at 264.16 144.78) (diameter 0) (color 0 0 0 0)
+  )
+  (junction (at 179.07 116.84) (diameter 0) (color 0 0 0 0)
   )
   (junction (at 280.67 50.8) (diameter 0) (color 0 0 0 0)
@@
   (no_connect (at 132.08 81.28))
   (no_connect (at 132.08 83.82))
-  (no_connect (at 132.08 96.52))
+  (no_connect (at 93.98 167.64))
   (no_connect (at 132.08 104.14))
-  (no_connect (at 132.08 114.3))
+  (no_connect (at 132.08 147.32))
+  (no_connect (at 132.08 124.46))
   (no_connect (at 132.08 119.38))
   (no_connect (at 132.08 99.06))
@@
   (no_connect (at 132.08 134.62))
   (no_connect (at 132.08 109.22))
-  (no_connect (at 132.08 86.36))
   (bus_entry (at 48.26 76.2) (size 2.54 2.54)
     (stroke (width 0) (type default))
@@
     (stroke (width 0) (type default))
   )
-  (bus_entry (at 176.53 129.54) (size -2.54 2.54)
-    (stroke (width 0) (type default))
-  )
   (bus_entry (at 185.42 139.7) (size 2.54 2.54)
     (stroke (width 0) (type default))
@@
     (stroke (width 0) (type default))
   )
-  (bus_entry (at 176.53 124.46) (size -2.54 2.54)
+  (bus_entry (at 179.07 124.46) (size -2.54 2.54)
     (stroke (width 0) (type default))
   )
@@
     (stroke (width 0) (type default))
   )
+  (bus_entry (at 176.53 86.36) (size 2.54 2.54)
+    (stroke (width 0) (type default))
+  )
   (bus_entry (at 367.03 173.99) (size -2.54 2.54)
     (stroke (width 0) (type default))
@@
     (stroke (width 0) (type default))
   )
-  (bus_entry (at 176.53 127) (size -2.54 2.54)
-    (stroke (width 0) (type default))
-  )
-  (bus_entry (at 176.53 119.38) (size -2.54 2.54)
+  (bus_entry (at 179.07 127) (size -2.54 2.54)
+    (stroke (width 0) (type default))
+  )
+  (bus_entry (at 179.07 119.38) (size -2.54 2.54)
     (stroke (width 0) (type default))
   )
@@
     (stroke (width 0) (type default))
   )
-  (bus (pts (xy 176.53 116.84) (xy 176.53 119.38))
-    (stroke (width 0) (type default))
-  )
-  (wire (pts (xy 132.08 127) (xy 173.99 127))
+  (bus (pts (xy 179.07 116.84) (xy 179.07 119.38))
+    (stroke (width 0) (type default))
+  )
+  (wire (pts (xy 132.08 127) (xy 176.53 127))
     (stroke (width 0) (type default))
   )
@@
     (stroke (width 0) (type default))
   )
+  (bus (pts (xy 179.07 88.9) (xy 179.07 116.84))
+    (stroke (width 0) (type default))
+  )
   (wire (pts (xy 52.07 193.04) (xy 93.98 193.04))
     (stroke (width 0) (type default))
@@
     (stroke (width 0) (type default))
   )
-  (wire (pts (xy 161.29 147.32) (xy 161.29 132.08))
-    (stroke (width 0) (type default))
-  )
   (wire (pts (xy 132.08 132.08) (xy 147.32 132.08))
     (stroke (width 0) (type default))
@@
     (stroke (width 0) (type default))
   )
-  (wire (pts (xy 38.1 167.64) (xy 93.98 167.64))
+  (wire (pts (xy 160.02 114.3) (xy 132.08 114.3))
     (stroke (width 0) (type default))
   )
@@
     (stroke (width 0) (type default))
   )
-  (bus (pts (xy 176.53 119.38) (xy 176.53 124.46))
+  (bus (pts (xy 179.07 119.38) (xy 179.07 124.46))
     (stroke (width 0) (type default))
   )
@@
     (stroke (width 0) (type default))
   )
-  (bus (pts (xy 176.53 116.84) (xy 186.69 116.84))
+  (bus (pts (xy 179.07 116.84) (xy 189.23 116.84))
     (stroke (width 0) (type default))
   )
@@
     (stroke (width 0) (type default))
   )
-  (wire (pts (xy 132.08 121.92) (xy 173.99 121.92))
+  (wire (pts (xy 132.08 121.92) (xy 176.53 121.92))
     (stroke (width 0) (type default))
   )
@@
     (stroke (width 0) (type default))
   )
-  (wire (pts (xy 157.48 129.54) (xy 173.99 129.54))
+  (wire (pts (xy 157.48 129.54) (xy 176.53 129.54))
     (stroke (width 0) (type default))
   )
@@
     (stroke (width 0) (type default))
   )
-  (wire (pts (xy 132.08 147.32) (xy 161.29 147.32))
+  (wire (pts (xy 132.08 86.36) (xy 176.53 86.36))
     (stroke (width 0) (type default))
   )
@@
     (stroke (width 0) (type default))
   )
-  (wire (pts (xy 132.08 124.46) (xy 154.94 124.46))
+  (wire (pts (xy 132.08 96.52) (xy 154.94 96.52))
     (stroke (width 0) (type default))
   )
@@
     (stroke (width 0) (type default))
   )
-  (bus (pts (xy 176.53 124.46) (xy 176.53 127))
-    (stroke (width 0) (type default))
-  )
-  (bus (pts (xy 176.53 127) (xy 176.53 129.54))
+  (bus (pts (xy 179.07 124.46) (xy 179.07 127))
     (stroke (width 0) (type default))
   )
@@
     (stroke (width 0) (type default))
   )
-  (wire (pts (xy 161.29 132.08) (xy 173.99 132.08))
-    (stroke (width 0) (type default))
-  )
   (wire (pts (xy 57.15 99.06) (xy 81.28 99.06))
     (stroke (width 0) (type default))
@@
     (effects (font (size 1.27 1.27)) (justify left bottom))
   )
-  (label "DAC_DATA_1_MCU" (at 154.94 124.46 180) (fields_autoplaced)
+  (label "DAC_DATA_1_MCU" (at 154.94 96.52 180) (fields_autoplaced)
     (effects (font (size 1.27 1.27)) (justify right bottom))
   )
@@
     (effects (font (size 1.27 1.27)) (justify right bottom))
   )
-  (label "ADC_M{slash}S" (at 154.94 147.32 180) (fields_autoplaced)
+  (label "ADC_M{slash}S" (at 154.94 86.36 180) (fields_autoplaced)
     (effects (font (size 1.27 1.27)) (justify right bottom))
   )
@@
     (effects (font (size 1.27 1.27)) (justify left))
   )
-  (hierarchical_label "{ADC_CONFIG}" (shape output) (at 186.69 116.84 0) (fields_autoplaced)
+  (hierarchical_label "{ADC_CONFIG}" (shape output) (at 189.23 116.84 0) (fields_autoplaced)
     (effects (font (size 1.27 1.27)) (justify left))
   )
@@
     (effects (font (size 1.27 1.27)) (justify right))
   )
-  (hierarchical_label "USB_A_PWR_EN" (shape output) (at 38.1 167.64 180) (fields_autoplaced)
-    (effects (font (size 1.27 1.27)) (justify right))
+  (hierarchical_label "USB_A_PWR_EN" (shape output) (at 160.02 114.3 0) (fields_autoplaced)
+    (effects (font (size 1.27 1.27)) (justify left))
   )
   (hierarchical_label "USB_HOST_N" (shape bidirectional) (at 30.48 93.98 180) (fields_autoplaced)

Commit message: Finish PCB design and added mounting holes
Parts:
- removed R209, R210, R211, R212: 0R, Resistor_SMD:R_0805_2012Metric_Pad1.20x1.40mm_HandSolder, symbol Device:R_Small
Connections:
- net I2S2_BCLK is gone; now on net BCLK_MCU: U201.84 (PD3)
- net I2S2_LRCLK is gone; now on net I2C_SCA: U201.96 (PB9)
- net I2S3_BCLK is gone; now on net BCLK_MCU: U201.78 (PC10)
- net ADC_FSAMPEN: now also U201.93 (PB7); no longer U201.88 (PD7)
- net ADC_IWL: now also U201.92 (PB6); no longer U201.86 (PD5)
- net GND: now also J201.1 (Pin_1), J201.5 (Pin_5), J201.9 (Pin_9); no longer J201.10 (Pin_10), J201.2 (Pin_2), J201.6 (Pin_6)
- net I2C_SCA: no longer U201.93 (PB7)
- net I2C_SCL: now also U201.95 (PB8); no longer U201.92 (PB6)
- net JTDI: no longer U201.77 (PA15)
- net LRCLK_MCU: now also U201.77 (PA15), U201.90 (PB4)
- net QUADSPI_CLK: now also J201.10 (Pin_10); no longer J201.1 (Pin_1)
- net QUADSPI_DATA_0: now also J201.8 (Pin_8); no longer J201.3 (Pin_3)
- net QUADSPI_DATA_1: now also J201.6 (Pin_6); no longer J201.5 (Pin_5)
- net QUADSPI_DATA_2: now also J201.4 (Pin_4); no longer J201.7 (Pin_7)
- net QUADSPI_DATA_3: now also J201.2 (Pin_2); no longer J201.9 (Pin_9)
- net QUADSPI_NCS: now also J201.12 (Pin_12); no longer J201.11 (Pin_11)
- net VDD: now also J201.11 (Pin_11), J201.3 (Pin_3), J201.7 (Pin_7); no longer J201.12 (Pin_12), J201.4 (Pin_4), J201.8 (Pin_8)
- net input_interrupt: now also U201.87 (PD6); no longer U201.95 (PB8)
- net register_OE: now also U201.31 (PA7); no longer U201.53 (PB14)
- net I2S3_LRCLK: no longer names the net of U201.28 (PA4)
