File: PCB/Magna/audio_daughterboard_connector.kicad_sch (KiCad schematic)
At the start: 1 part, among them J301 Conn_02x15_Odd_Even

Commit message: Update Mainboard PCB
* Added better power ORing
* Added DRC for length matching
* Changed out components for cheaper production
* Removed some optional circuits from BOM for first prototype
Parts:
- J301: now left out of the parts list
Changed lines of the file:
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@@
 		(unit 1)
 		(exclude_from_sim no)
-		(in_bom yes)
+		(in_bom no)
 		(on_board yes)
 		(dnp no)
@@
 			(at 160.02 93.98 0)
 			(effects
+				(font
+					(size 1.27 1.27)
+				)
+				(hide yes)
+			)
+		)
+		(property "Sim.Type" ""
+			(at 160.02 93.98 0)
+			(effects
