File: PCB/Magna/io_daughterboard/io_daughterboard.kicad_pcb (KiCad board)
At the start: 2 copper layers, 240 x 320 mm, 209 parts, among them J101 Conn_02x10_Counter_Clockwise, U201 74HC595, U202 74HC595, U203 74HC595, U204 74HC595, U205 74HC595, U301 XL9535, U501 4052, U601 4052, U701 4052

Commit message: Add a lot on the IO PCB
Also some schematic changes to accomodate issues found
when routing
Parts:
- removed TP201, TP202, TP203, TP204, TP205, TP206, TP301, TP302, TP303, TP304, TP401, TP402, TP403, TP404, TP405, TP406, TP407, TP408, TP409: TestPoint, TestPoint:TestPoint_Keystone_5005-5009_Compact
- added C101: 100nF/50V, Capacitor_SMD:C_0805_2012Metric_Pad1.18x1.45mm_HandSolder, F.Cu at (52.5, 45.0)
- added C102: 100nF/50V, Capacitor_SMD:C_0805_2012Metric_Pad1.18x1.45mm_HandSolder, F.Cu at (120.0, 30.0)
- added C103: 100nF/50V, Capacitor_SMD:C_0805_2012Metric_Pad1.18x1.45mm_HandSolder, F.Cu at (182.5, 173.5)
- added C104: 1uF/50V, Capacitor_SMD:C_0805_2012Metric_Pad1.18x1.45mm_HandSolder, F.Cu at (120.0, 300.0)
- added C105: 1uF/50V, Capacitor_SMD:C_0805_2012Metric_Pad1.18x1.45mm_HandSolder, F.Cu at (120.0, 270.0)
- added R101: 22R, Resistor_SMD:R_0805_2012Metric_Pad1.20x1.40mm_HandSolder, F.Cu at (50.0, 48.0)
- added R102: 22R, Resistor_SMD:R_0805_2012Metric_Pad1.20x1.40mm_HandSolder, F.Cu at (55.0, 48.0)
- added R103: 22R, Resistor_SMD:R_0805_2012Metric_Pad1.20x1.40mm_HandSolder, F.Cu at (117.5, 35.0)
- added R104: 22R, Resistor_SMD:R_0805_2012Metric_Pad1.20x1.40mm_HandSolder, F.Cu at (122.5, 35.0)
- added R105: 22R, Resistor_SMD:R_0805_2012Metric_Pad1.20x1.40mm_HandSolder, F.Cu at (185.0, 170.0)
- added R106: 22R, Resistor_SMD:R_0805_2012Metric_Pad1.20x1.40mm_HandSolder, F.Cu at (180.0, 170.0)
- added U101: NE5532, Package_SO:SOIC-8_3.9x4.9mm_P1.27mm, F.Cu at (52.5, 40.0)
- added U102: NE5532, Package_SO:SOIC-8_3.9x4.9mm_P1.27mm, F.Cu at (120.0, 25.0)
- added U103: NE5532, Package_SO:SOIC-8_3.9x4.9mm_P1.27mm, F.Cu at (182.5, 177.5)
- moved R233 362.6 mm to (276.9, 178.3)
- moved R234 362.6 mm to (276.9, 181.3)
- moved R301 358.5 mm to (272.2, 139.7)
- moved R302 358.5 mm to (272.2, 142.7)
- moved R303 358.5 mm to (272.2, 145.6)
- moved R304 358.5 mm to (272.2, 148.6)
- moved R305 358.5 mm to (272.2, 151.5)
- moved R306 358.5 mm to (272.2, 154.4)
- moved R307 358.5 mm to (272.2, 157.4)
- moved R308 358.5 mm to (276.9, 139.7)
- moved R309 358.5 mm to (276.9, 142.7)
- moved R310 358.5 mm to (276.9, 145.6)
- moved R311 358.5 mm to (276.9, 148.6)
- moved R312 358.5 mm to (276.9, 151.5)
- moved R313 358.5 mm to (276.9, 154.4)
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Connections:
- D225 pad 1: /LEDs/CH1_CUE_Status -> Net-(D225-K)
- D225 pad 2: Net-(D225-A) -> VDD
- D226 pad 1: /LEDs/COL1_Sel_Status -> Net-(D226-K)
- D226 pad 2: Net-(D226-A) -> VDD
- D227 pad 1: /LEDs/COL3_Sel_Status -> Net-(D227-K)
- D227 pad 2: Net-(D227-A) -> VDD
- D228 pad 1: /LEDs/Effect_On_Status -> Net-(D228-K)
- D228 pad 2: Net-(D228-A) -> VDD
- D229 pad 1: /LEDs/Effect_CH1_Assign -> Net-(D229-K)
- D229 pad 2: Net-(D229-A) -> VDD
- D230 pad 1: /LEDs/MIDI_IN_INDICATOR -> Net-(D230-K)
- D230 pad 2: Net-(D230-A) -> VDD
- D231 pad 1: /LEDs/CH2_CUE_Status -> Net-(D231-K)
- D231 pad 2: Net-(D231-A) -> VDD
- D232 pad 1: /LEDs/COL2_Sel_Status -> Net-(D232-K)
- D232 pad 2: Net-(D232-A) -> VDD
- D233 pad 1: /LEDs/COL4_Sel_Status -> Net-(D233-K)
- D233 pad 2: Net-(D233-A) -> VDD
- D234 pad 1: /LEDs/Effect_CH2_Assign -> Net-(D234-K)
- D234 pad 2: Net-(D234-A) -> VDD
- D235 pad 1: /LEDs/SPARE_LED1 -> Net-(D235-K)
- D235 pad 2: Net-(D235-A) -> VDD
- D236 pad 1: /LEDs/SPARE_LED4 -> Net-(D236-K)
- D236 pad 2: Net-(D236-A) -> VDD
- D237 pad 1: /LEDs/EFFECT_CUE_STATUS -> Net-(D237-K)
- D237 pad 2: Net-(D237-A) -> VDD
- D238 pad 1: /LEDs/SPARE_LED5 -> Net-(D238-K)
- D238 pad 2: Net-(D238-A) -> VDD
- D239 pad 1: /LEDs/SPARE_LED2 -> Net-(D239-K)
- D239 pad 2: Net-(D239-A) -> VDD
- D240 pad 1: /LEDs/SPARE_LED3 -> Net-(D240-K)
- D240 pad 2: Net-(D240-A) -> VDD
- J101 pad 10: GND -> /register_OE
- J101 pad 11: /register_OE -> GND
- J101 pad 12: /register_CLK -> /serial_CLK
- J101 pad 13: /serial_CLR -> /Potentiometers/lsb
- J101 pad 14: /serial_CLK -> /serial_CLR
- J101 pad 15: /serial_data -> /Buttons/I2C_SDA
- J101 pad 16: /Buttons/I2C_SCL -> /register_CLK
- J101 pad 17: /Buttons/I2C_SDA -> GND
- J101 pad 18: /Potentiometers/lsb -> /serial_data
- J101 pad 19: /Potentiometers/msb -> /Buttons/I2C_SCL
- J101 pad 2: GND -> /ADC_3_CONN
- J101 pad 3: /Potentiometers/ADC_0 -> /ADC_4_CONN
- J101 pad 4: /Potentiometers/ADC_1 -> /ADC_2_CONN
- J101 pad 5: /Potentiometers/ADC_2 -> /ADC_5_CONN
- J101 pad 6: /Potentiometers/ADC_3 -> /ADC_1_CONN
- J101 pad 7: /Potentiometers/ADC_4 -> /Buttons/button_interrupt
- J101 pad 8: /Potentiometers/ADC_5 -> /ADC_0_CONN
- J101 pad 9: /Buttons/button_interrupt -> /Potentiometers/msb
- R225 pad 1: Net-(D225-A) -> Net-(D225-K)
- R225 pad 2: VDD -> /LEDs/CH1_CUE_Status
- R226 pad 1: Net-(D226-A) -> Net-(D226-K)
- R226 pad 2: VDD -> /LEDs/COL1_Sel_Status
- R227 pad 1: Net-(D227-A) -> Net-(D227-K)
- R227 pad 2: VDD -> /LEDs/COL3_Sel_Status
- R228 pad 1: Net-(D228-A) -> Net-(D228-K)
- R228 pad 2: VDD -> /LEDs/Effect_On_Status
- R229 pad 1: Net-(D229-A) -> /LEDs/Effect_CH1_Assign
- R229 pad 2: VDD -> Net-(D229-K)
- R230 pad 1: Net-(D230-A) -> Net-(D230-K)
- R230 pad 2: VDD -> /LEDs/MIDI_IN_INDICATOR
- R231 pad 1: Net-(D231-A) -> Net-(D231-K)
- R231 pad 2: VDD -> /LEDs/CH2_CUE_Status
- R232 pad 1: Net-(D232-A) -> Net-(D232-K)
- R232 pad 2: VDD -> /LEDs/COL2_Sel_Status
- R233 pad 1: Net-(D233-A) -> Net-(D233-K)
- R233 pad 2: VDD -> /LEDs/COL4_Sel_Status
- R234 pad 1: Net-(D234-A) -> Net-(D234-K)
- R234 pad 2: VDD -> /LEDs/Effect_CH2_Assign
- R235 pad 1: Net-(D235-A) -> Net-(D235-K)
- R235 pad 2: VDD -> /LEDs/SPARE_LED1
- R236 pad 1: Net-(D236-A) -> Net-(D236-K)
- R236 pad 2: VDD -> /LEDs/SPARE_LED4
- R237 pad 1: Net-(D237-A) -> Net-(D237-K)
- R237 pad 2: VDD -> /LEDs/EFFECT_CUE_STATUS
- R238 pad 1: Net-(D238-A) -> Net-(D238-K)
- R238 pad 2: VDD -> /LEDs/SPARE_LED5
- R239 pad 1: Net-(D239-A) -> Net-(D239-K)
- R239 pad 2: VDD -> /LEDs/SPARE_LED2
- R240 pad 1: Net-(D240-A) -> Net-(D240-K)
- R240 pad 2: VDD -> /LEDs/SPARE_LED3
- U201 pad 1: /LEDs/CH1_0db -> /LEDs/CH1_20db
- U201 pad 10: /serial_CLR -> /serial_data
- U201 pad 11: /serial_CLK -> /serial_CLR
- U201 pad 14: /serial_data -> Net-(U201-SER)
- U201 pad 15: /LEDs/CH1_clip -> /LEDs/CH1_25db
- U201 pad 2: /LEDs/CH1_3db -> /LEDs/CH1_12db
- U201 pad 3: /LEDs/CH1_6db -> /LEDs/CH1_9db
- U201 pad 4: /LEDs/CH1_9db -> /LEDs/CH1_6db
- U201 pad 5: /LEDs/CH1_12db -> /LEDs/CH1_3db
- U201 pad 6: /LEDs/CH1_20db -> /LEDs/CH1_0db
- U201 pad 7: /LEDs/CH1_25db -> /LEDs/CH1_clip
- U202 pad 10: /serial_CLR -> /serial_data
- U202 pad 11: /serial_CLK -> /serial_CLR
- U202 pad 14: Net-(U201-QH') -> Net-(U202-SER)
- U202 pad 9: Net-(U202-QH') -> Net-(U201-SER)
- U203 pad 1: /LEDs/Master_0db -> /LEDs/Master_20db
- U203 pad 10: /serial_CLR -> /serial_data
- U203 pad 11: /serial_CLK -> /serial_CLR
- U203 pad 14: Net-(U202-QH') -> Net-(U203-SER)
- U203 pad 15: /LEDs/Master_clip -> /LEDs/Master_25db
- U203 pad 2: /LEDs/Master_3db -> /LEDs/Master_12db
- U203 pad 3: /LEDs/Master_6db -> /LEDs/Master_9db
- U203 pad 4: /LEDs/Master_9db -> /LEDs/Master_6db
- U203 pad 5: /LEDs/Master_12db -> /LEDs/Master_3db
- U203 pad 6: /LEDs/Master_20db -> /LEDs/Master_0db
- U203 pad 7: /LEDs/Master_25db -> /LEDs/Master_clip
- U203 pad 9: Net-(U203-QH') -> Net-(U202-SER)
- U204 pad 10: /serial_CLR -> /serial_data
- U204 pad 11: /serial_CLK -> /serial_CLR
- U204 pad 14: Net-(U203-QH') -> Net-(U201-QH')
- U204 pad 6: /LEDs/SPARE_LED1 -> /LEDs/Effect_CH1_Assign
- U204 pad 7: /LEDs/SPARE_LED2 -> /LEDs/Effect_CH2_Assign
- U204 pad 9: Net-(U204-QH') -> unconnected-(U204-QH'-Pad9)
- U205 pad 1: /LEDs/Effect_CH1_Assign -> /LEDs/EFFECT_CUE_STATUS
- U205 pad 10: /serial_CLR -> /serial_data
- U205 pad 11: /serial_CLK -> /serial_CLR
- U205 pad 14: Net-(U204-QH') -> /serial_CLK
- U205 pad 2: /LEDs/Effect_CH2_Assign -> /LEDs/MIDI_IN_INDICATOR
- U205 pad 3: /LEDs/EFFECT_CUE_STATUS -> /LEDs/SPARE_LED1
- U205 pad 4: /LEDs/MIDI_IN_INDICATOR -> /LEDs/SPARE_LED2
- U205 pad 9: unconnected-(U205-QH'-Pad9) -> Net-(U203-SER)
- U501 pad 10: /Potentiometers/lsb -> /Potentiometers/msb
- U501 pad 12: /Potentiometers/CH1_HI -> /Potentiometers/CH1_LOW-MID
- U501 pad 13: /Potentiometers/ADC_0 -> /Potentiometers/ADC_2
- U501 pad 15: /Potentiometers/CH1_LOW-MID -> /Potentiometers/CH1_HI
- U501 pad 2: /Potentiometers/CH2_LOW-MID -> /Potentiometers/CH2_MID
- U501 pad 3: /Potentiometers/ADC_1 -> /Potentiometers/ADC_3
- U501 pad 4: /Potentiometers/CH2_LOW -> /Potentiometers/CH2_LOW-MID
- U501 pad 5: /Potentiometers/CH2_MID -> /Potentiometers/CH2_LOW
- U501 pad 9: /Potentiometers/msb -> /Potentiometers/lsb
- U601 pad 1: /Potentiometers/SPARE3 -> /Potentiometers/CH1_COLOUR
- U601 pad 10: /Potentiometers/lsb -> /Potentiometers/analogueIOexpander1/sel1
- U601 pad 12: /Potentiometers/CUE_MIX -> /Potentiometers/SPARE3
- U601 pad 13: /Potentiometers/ADC_2 -> /Potentiometers/analogueIOexpander1/MCU_ADC_X
- U601 pad 14: /Potentiometers/COLOUR_PARAM -> /Potentiometers/SPARE4
- U601 pad 15: /Potentiometers/SPARE1 -> /Potentiometers/COLOUR_PARAM
- U601 pad 3: /Potentiometers/ADC_3 -> /Potentiometers/analogueIOexpander1/MCU_ADC_Y
- U601 pad 5: /Potentiometers/SPARE4 -> /Potentiometers/SPARE1
- U601 pad 9: /Potentiometers/msb -> /Potentiometers/analogueIOexpander1/sel0
- U701 pad 10: /Potentiometers/lsb -> /Potentiometers/msb
- U701 pad 12: /Potentiometers/CH1_COLOUR -> /Potentiometers/CUE_MIX
- U701 pad 14: /Potentiometers/CH1_VOL -> /Potentiometers/EFFECT_WET_DRY
- U701 pad 15: /Potentiometers/CH2_COLOUR -> /Potentiometers/EFFECT_PARAM_2
- U701 pad 2: /Potentiometers/EFFECT_WET_DRY -> /Potentiometers/SPARE5
- U701 pad 4: /Potentiometers/SPARE5 -> /Potentiometers/CH2_COLOUR
- U701 pad 5: /Potentiometers/EFFECT_PARAM_2 -> /Potentiometers/CH1_VOL
- U701 pad 9: /Potentiometers/msb -> /Potentiometers/lsb
Routing:
- net VDDA: track 0.00 -> 1572.2 mm, vias 0 -> 3
- net /Potentiometers/lsb: track 0.00 -> 855.8 mm, vias 0 -> 9
- net /Potentiometers/msb: track 0.00 -> 837.1 mm, vias 0 -> 9
- net /ADC_3_CONN: track 0.00 -> 514.5 mm, vias 0 -> 4
- net /ADC_2_CONN: track 0.00 -> 499.5 mm, vias 0 -> 4
- net /ADC_1_CONN: track 0.00 -> 404.2 mm, vias 0 -> 2
- net /ADC_0_CONN: track 0.00 -> 389.7 mm, vias 0 -> 2
- net Net-(D230-K): track 0.00 -> 373.7 mm, vias 0 -> 2
- net /Potentiometers/CH2_VOL: track 0.00 -> 347.5 mm, vias 0 -> 2
- net Net-(D228-K): track 0.00 -> 344.8 mm, vias 0 -> 2
- net Net-(R309-Pad2): track 0.00 -> 338.2 mm
- net /Potentiometers/CUE_MIX: track 0.00 -> 314.4 mm
- net VDD: track 159.2 -> 443.9 mm
- net Net-(D237-K): track 0.00 -> 275.0 mm, vias 0 -> 2
- net Net-(R335-Pad2): track 0.00 -> 264.4 mm
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Other:
- board text added: "-12Db"
- board text added: "-20Db"
- board text added: "-25Db"
- board text added: "-3Db"
- board text added: "-6Db"
- board text added: "-9Db"
- board text added: "0Db"
- board text added: "1"
- board text added: "2"
- board text added: "3"
- board text added: "4"
- board text added: "CH1 COLOUR FX"
- board text added: "CH1 CUE"
- board text added: "CH1 SFX"
- board text added: "CH1 VOL"
- board text added: "CH2 COLOUR FX"
- board text added: "CH2 CUE"
- board text added: "CH2 VOL"
- board text added: "CLIP"
- board text added: "COLOUR FX PARAM"
- board text added: "COLOUR SELECT FX"
- board text added: "CUE MIX"
- board text added: "GAIN"
- board text added: "HI"
- board text added: "LO-MID"
- board text added: "LOW"
- board text added: "MID"
- board text added: "SFX CUE"
- board text added: "SFX ON"
- board text added: "SFX PARAM"
- board text added: "SFX WET/DRY"

Commit message: Route most of io daughterboard
Parts:
- moved C305 636.7 mm to (242.0, 300.0)
- moved C303 630.5 mm to (237.0, 288.0)
- moved C304 580.7 mm to (166.2, 352.0)
- moved C307 580.7 mm to (171.0, 343.0)
- moved C308 580.7 mm to (171.0, 346.0)
- moved C309 580.7 mm to (171.0, 349.0)
- moved C310 580.7 mm to (171.0, 352.0)
- moved C311 580.7 mm to (171.0, 355.0)
- moved C312 580.7 mm to (171.0, 358.1)
- moved C313 580.7 mm to (175.8, 343.0)
- moved C314 580.7 mm to (175.8, 346.0)
- moved C315 580.7 mm to (175.8, 349.0)
- moved C317 580.7 mm to (175.8, 355.0)
- moved C306 569.0 mm to (157.8, 347.0)
- moved C301 554.9 mm to (167.5, 246.0), turned to -90 degrees
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Connections:
- C201 pad 2: GND -> unconnected-(C201-Pad2)
- D201 pad 1: Net-(D201-K) -> unconnected-(D201-K-Pad1)
- D201 pad 2: VDD -> Net-(D201-A)
- D202 pad 1: Net-(D202-K) -> GND
- D202 pad 2: VDD -> Net-(D202-A)
- D203 pad 1: Net-(D203-K) -> GND
- D203 pad 2: VDD -> Net-(D203-A)
- D204 pad 1: Net-(D204-K) -> GND
- D204 pad 2: VDD -> Net-(D204-A)
- D205 pad 1: Net-(D205-K) -> GND
- D205 pad 2: VDD -> Net-(D205-A)
- D206 pad 1: Net-(D206-K) -> GND
- D206 pad 2: VDD -> Net-(D206-A)
- D207 pad 1: Net-(D207-K) -> GND
- D207 pad 2: VDD -> Net-(D207-A)
- D208 pad 1: Net-(D208-K) -> GND
- D208 pad 2: VDD -> Net-(D208-A)
- D209 pad 1: Net-(D209-K) -> GND
- D209 pad 2: VDD -> Net-(D209-A)
- D210 pad 1: Net-(D210-K) -> GND
- D210 pad 2: VDD -> Net-(D210-A)
- D211 pad 1: Net-(D211-K) -> GND
- D211 pad 2: VDD -> Net-(D211-A)
- D212 pad 1: Net-(D212-K) -> GND
- D212 pad 2: VDD -> Net-(D212-A)
- D213 pad 1: Net-(D213-K) -> GND
- D213 pad 2: VDD -> Net-(D213-A)
- D214 pad 1: Net-(D214-K) -> GND
- D214 pad 2: VDD -> Net-(D214-A)
- D215 pad 1: Net-(D215-K) -> GND
- D215 pad 2: VDD -> Net-(D215-A)
- D216 pad 1: Net-(D216-K) -> GND
- D216 pad 2: VDD -> Net-(D216-A)
- D217 pad 1: Net-(D217-K) -> GND
- D217 pad 2: VDD -> Net-(D217-A)
- D218 pad 1: Net-(D218-K) -> GND
- D218 pad 2: VDD -> Net-(D218-A)
- D219 pad 1: Net-(D219-K) -> GND
- D219 pad 2: VDD -> Net-(D219-A)
- D220 pad 1: Net-(D220-K) -> GND
- D220 pad 2: VDD -> Net-(D220-A)
- D221 pad 1: Net-(D221-K) -> GND
- D221 pad 2: VDD -> Net-(D221-A)
- D222 pad 1: Net-(D222-K) -> GND
- D222 pad 2: VDD -> Net-(D222-A)
- D223 pad 1: Net-(D223-K) -> GND
- D223 pad 2: VDD -> Net-(D223-A)
- D224 pad 1: Net-(D224-K) -> GND
- D224 pad 2: VDD -> Net-(D224-A)
- D225 pad 1: Net-(D225-K) -> GND
- D225 pad 2: VDD -> Net-(D225-A)
- D226 pad 1: Net-(D226-K) -> GND
- D226 pad 2: VDD -> Net-(D226-A)
- D227 pad 1: Net-(D227-K) -> GND
- D227 pad 2: VDD -> Net-(D227-A)
- D228 pad 1: Net-(D228-K) -> GND
- D228 pad 2: VDD -> Net-(D228-A)
- D229 pad 1: Net-(D229-K) -> GND
- D229 pad 2: VDD -> Net-(D229-A)
- D230 pad 1: Net-(D230-K) -> GND
- D230 pad 2: VDD -> Net-(D230-A)
- D231 pad 1: Net-(D231-K) -> GND
- D231 pad 2: VDD -> Net-(D231-A)
- D232 pad 1: Net-(D232-K) -> GND
- D232 pad 2: VDD -> Net-(D232-A)
- D233 pad 1: Net-(D233-K) -> GND
- D233 pad 2: VDD -> Net-(D233-A)
- D234 pad 1: Net-(D234-K) -> GND
- D234 pad 2: VDD -> Net-(D234-A)
- D235 pad 1: Net-(D235-K) -> GND
- D235 pad 2: VDD -> Net-(D235-A)
- D236 pad 1: Net-(D236-K) -> GND
- D236 pad 2: VDD -> Net-(D236-A)
- D237 pad 1: Net-(D237-K) -> GND
- D237 pad 2: VDD -> Net-(D237-A)
- D238 pad 1: Net-(D238-K) -> GND
- D238 pad 2: VDD -> Net-(D238-A)
- D239 pad 1: Net-(D239-K) -> GND
- D239 pad 2: VDD -> Net-(D239-A)
- D240 pad 1: Net-(D240-K) -> GND
- D240 pad 2: VDD -> Net-(D240-A)
- J101 pad 1: VDDA -> /ADC_3_CONN
- J101 pad 10: /register_OE -> /Potentiometers/msb
- J101 pad 11: GND -> /serial_data
- J101 pad 12: /serial_CLK -> GND
- J101 pad 13: /Potentiometers/lsb -> /register_CLK
- J101 pad 14: /serial_CLR -> /Potentiometers/lsb
- J101 pad 15: /Buttons/I2C_SDA -> /serial_CLR
- J101 pad 16: /register_CLK -> /Buttons/I2C_SCL
- J101 pad 17: GND -> /serial_CLK
- J101 pad 18: /serial_data -> GND
- J101 pad 19: /Buttons/I2C_SCL -> VDD
- J101 pad 2: /ADC_3_CONN -> VDDA
- J101 pad 20: VDD -> /Buttons/I2C_SDA
- J101 pad 3: /ADC_4_CONN -> /ADC_2_CONN
- J101 pad 4: /ADC_2_CONN -> /ADC_4_CONN
- J101 pad 5: /ADC_5_CONN -> /ADC_1_CONN
- J101 pad 6: /ADC_1_CONN -> /ADC_5_CONN
- J101 pad 7: /Buttons/button_interrupt -> /ADC_0_CONN
- J101 pad 8: /ADC_0_CONN -> /Buttons/button_interrupt
- J101 pad 9: /Potentiometers/msb -> /register_OE
- R201 pad 1: Net-(D201-K) -> /LEDs/CH1_clip
- R201 pad 2: /LEDs/CH1_clip -> Net-(D201-A)
- R202 pad 1: Net-(D202-K) -> Net-(D202-A)
- R203 pad 1: Net-(D203-K) -> Net-(D203-A)
- R204 pad 1: Net-(D204-K) -> Net-(D204-A)
- R205 pad 1: Net-(D205-K) -> Net-(D205-A)
- R206 pad 1: Net-(D206-K) -> Net-(D206-A)
- R207 pad 1: Net-(D207-K) -> Net-(D207-A)
- R208 pad 1: Net-(D208-K) -> Net-(D208-A)
- R209 pad 1: Net-(D209-K) -> Net-(D209-A)
- R210 pad 1: Net-(D210-K) -> Net-(D210-A)
- R211 pad 1: Net-(D211-K) -> Net-(D211-A)
- R212 pad 1: Net-(D212-K) -> Net-(D212-A)
- R213 pad 1: Net-(D213-K) -> Net-(D213-A)
- R214 pad 1: Net-(D214-K) -> Net-(D214-A)
- R215 pad 1: Net-(D215-K) -> Net-(D215-A)
- R216 pad 1: Net-(D216-K) -> Net-(D216-A)
- R217 pad 1: Net-(D217-K) -> Net-(D217-A)
- R218 pad 1: Net-(D218-K) -> Net-(D218-A)
- R219 pad 1: Net-(D219-K) -> Net-(D219-A)
- R220 pad 1: Net-(D220-K) -> Net-(D220-A)
- R221 pad 1: Net-(D221-K) -> Net-(D221-A)
- R222 pad 1: Net-(D222-K) -> Net-(D222-A)
- R223 pad 1: Net-(D223-K) -> Net-(D223-A)
- R224 pad 1: Net-(D224-K) -> Net-(D224-A)
- R225 pad 1: Net-(D225-K) -> Net-(D225-A)
- R226 pad 1: Net-(D226-K) -> Net-(D226-A)
- R227 pad 1: Net-(D227-K) -> Net-(D227-A)
- R228 pad 1: Net-(D228-K) -> Net-(D228-A)
- R229 pad 1: /LEDs/Effect_CH1_Assign -> Net-(D229-A)
- R229 pad 2: Net-(D229-K) -> /LEDs/Effect_CH1_Assign
- R230 pad 1: Net-(D230-K) -> /LEDs/MIDI_IN_INDICATOR
- R230 pad 2: /LEDs/MIDI_IN_INDICATOR -> Net-(D230-A)
- R231 pad 1: Net-(D231-K) -> Net-(D231-A)
- R232 pad 1: Net-(D232-K) -> Net-(D232-A)
- R233 pad 1: Net-(D233-K) -> Net-(D233-A)
- R234 pad 1: Net-(D234-K) -> Net-(D234-A)
- R235 pad 1: Net-(D235-K) -> Net-(D235-A)
- R236 pad 1: Net-(D236-K) -> Net-(D236-A)
- R237 pad 1: Net-(D237-K) -> Net-(D237-A)
- R238 pad 1: Net-(D238-K) -> Net-(D238-A)
- R239 pad 1: Net-(D239-K) -> Net-(D239-A)
- R240 pad 1: Net-(D240-K) -> Net-(D240-A)
- U201 pad 10: /serial_data -> /serial_CLR
- U201 pad 11: /serial_CLR -> /serial_CLK
- U202 pad 10: /serial_data -> /serial_CLR
- U202 pad 11: /serial_CLR -> /serial_CLK
- U202 pad 9: Net-(U201-SER) -> Net-(U202-QH')
- U203 pad 10: /serial_data -> /serial_CLR
- U203 pad 11: /serial_CLR -> /serial_CLK
- U203 pad 14: Net-(U203-SER) -> Net-(U202-QH')
- U203 pad 9: Net-(U202-SER) -> Net-(U201-SER)
- U204 pad 10: /serial_data -> /serial_CLR
- U204 pad 11: /serial_CLR -> /serial_CLK
- U204 pad 15: /LEDs/CH1_CUE_Status -> /LEDs/Effect_CH1_Assign
- U204 pad 2: /LEDs/COL1_Sel_Status -> /LEDs/CH1_CUE_Status
- U204 pad 3: /LEDs/COL2_Sel_Status -> /LEDs/COL1_Sel_Status
- U204 pad 4: /LEDs/COL3_Sel_Status -> /LEDs/COL2_Sel_Status
- U204 pad 5: /LEDs/COL4_Sel_Status -> /LEDs/COL3_Sel_Status
- U204 pad 6: /LEDs/Effect_CH1_Assign -> /LEDs/COL4_Sel_Status
- U205 pad 1: /LEDs/EFFECT_CUE_STATUS -> /LEDs/Effect_On_Status
- U205 pad 10: /serial_data -> /serial_CLR
- U205 pad 11: /serial_CLR -> /serial_CLK
- U205 pad 14: /serial_CLK -> /serial_data
- U205 pad 15: /LEDs/Effect_On_Status -> /LEDs/MIDI_IN_INDICATOR
- U205 pad 2: /LEDs/MIDI_IN_INDICATOR -> /LEDs/EFFECT_CUE_STATUS
- U205 pad 3: /LEDs/SPARE_LED1 -> /LEDs/SPARE_LED5
- U205 pad 4: /LEDs/SPARE_LED2 -> /LEDs/SPARE_LED4
- U205 pad 6: /LEDs/SPARE_LED4 -> /LEDs/SPARE_LED2
- U205 pad 7: /LEDs/SPARE_LED5 -> /LEDs/SPARE_LED1
- U205 pad 9: Net-(U203-SER) -> Net-(U202-SER)
- U301 pad 10: /Buttons/EFFECT_ASSIGN_CH2 -> /Buttons/CUE_EFFECT_SEL
- U301 pad 11: /Buttons/SPARE_2 -> /Buttons/SPARE_1
- U301 pad 13: /Buttons/COLOUR_SEL_1 -> /Buttons/EFFECT_ASSIGN_CH1
- U301 pad 14: /Buttons/COLOUR_SEL_2 -> /Buttons/EFFECT_ASSIGN_CH2
- U301 pad 15: /Buttons/COLOUR_SEL_3 -> /Buttons/CUE_CH2_SEL
- U301 pad 16: /Buttons/COLOUR_SEL_4 -> unconnected-(U301-P13-Pad16)
- U301 pad 17: /Buttons/SPARE_3 -> unconnected-(U301-P14-Pad17)
- U301 pad 18: /Buttons/SPARE_4 -> /Buttons/COLOUR_SEL_2
- U301 pad 19: /Buttons/SPARE_5 -> /Buttons/COLOUR_SEL_3
- U301 pad 20: /Buttons/SPARE_6 -> /Buttons/COLOUR_SEL_4
- U301 pad 4: /Buttons/CUE_CH1_SEL -> /Buttons/EFFECT ON
- U301 pad 5: /Buttons/CUE_CH2_SEL -> /Buttons/SPARE_3
- U301 pad 6: /Buttons/CUE_EFFECT_SEL -> /Buttons/SPARE_4
- U301 pad 7: /Buttons/SPARE_1 -> /Buttons/SPARE_5
- U301 pad 8: /Buttons/EFFECT ON -> /Buttons/SPARE_6
- U301 pad 9: /Buttons/EFFECT_ASSIGN_CH1 -> /Buttons/SPARE_2
- U501 pad 1: /Potentiometers/CH2_HI -> /Potentiometers/EFFECT_PARAM_2
- U501 pad 11: /Potentiometers/CH1_LOW -> /Potentiometers/CH2_MID
- U501 pad 12: /Potentiometers/CH1_LOW-MID -> /Potentiometers/CH2_LOW-MID
- U501 pad 14: /Potentiometers/CH1_MID -> /Potentiometers/CH2_LOW
- U501 pad 15: /Potentiometers/CH1_HI -> /Potentiometers/CH2_COLOUR
- U501 pad 2: /Potentiometers/CH2_MID -> /Potentiometers/EFFECT_PARAM_1
- U501 pad 4: /Potentiometers/CH2_LOW-MID -> /Potentiometers/SPARE5
- U501 pad 5: /Potentiometers/CH2_LOW -> /Potentiometers/CH2_GAIN
- U601 pad 1: /Potentiometers/CH1_COLOUR -> /Potentiometers/CH1_HI
- U601 pad 10: /Potentiometers/analogueIOexpander1/sel1 -> /Potentiometers/msb
- U601 pad 11: /Potentiometers/SPARE2 -> /Potentiometers/CH1_COLOUR
- U601 pad 12: /Potentiometers/SPARE3 -> /Potentiometers/CH1_LOW
- U601 pad 13: /Potentiometers/analogueIOexpander1/MCU_ADC_X -> /Potentiometers/ADC_0
- U601 pad 14: /Potentiometers/SPARE4 -> /Potentiometers/CH1_LOW-MID
- U601 pad 15: /Potentiometers/COLOUR_PARAM -> /Potentiometers/CH1_MID
- U601 pad 2: /Potentiometers/CH1_GAIN -> /Potentiometers/CH2_HI
- U601 pad 3: /Potentiometers/analogueIOexpander1/MCU_ADC_Y -> /Potentiometers/ADC_1
- U601 pad 4: /Potentiometers/CH2_GAIN -> /Potentiometers/CH1_GAIN
- U601 pad 9: /Potentiometers/analogueIOexpander1/sel0 -> /Potentiometers/lsb
- U701 pad 1: /Potentiometers/EFFECT_PARAM_1 -> /Potentiometers/analogueIOexpander2/IN_Y0
- U701 pad 15: /Potentiometers/EFFECT_PARAM_2 -> /Potentiometers/analogueIOexpander2/IN_X2
- U701 pad 2: /Potentiometers/SPARE5 -> /Potentiometers/analogueIOexpander2/IN_Y2
- U701 pad 4: /Potentiometers/CH2_COLOUR -> /Potentiometers/analogueIOexpander2/IN_Y3
Routing:
- net VDDA: track 1572.2 -> 1062.6 mm, vias 3 -> 0
- net Net-(D230-K): track 373.7 -> 0.00 mm, vias 2 -> 0
- net /Potentiometers/CH2_VOL: track 347.5 -> 0.00 mm, vias 2 -> 0
- net Net-(D228-K): track 344.8 -> 0.00 mm, vias 2 -> 0
- net /Potentiometers/CUE_MIX: track 314.4 -> 0.00 mm
- net Net-(D235-A): track 0.00 -> 309.1 mm
- net Net-(D239-A): track 0.00 -> 298.1 mm
- net Net-(R309-Pad2): track 338.2 -> 41.1 mm
- net Net-(D240-A): track 0.00 -> 287.5 mm
- net Net-(D236-A): track 0.00 -> 276.4 mm
- net Net-(D237-K): track 275.0 -> 0.00 mm, vias 2 -> 0
- net Net-(D238-A): track 0.00 -> 267.4 mm
- net VDD: track 443.9 -> 186.6 mm, vias 0 -> 11
- net /register_OE: track 0.00 -> 254.8 mm
- net /register_CLK: track 0.00 -> 247.8 mm
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Other:
- board text added: "locked"
- board text removed: "CH2 CUE"

Commit message: Add more routing to IO Daugherboard
Parts:
- removed C103: 100nF/50V, Capacitor_SMD:C_0805_2012Metric_Pad1.18x1.45mm_HandSolder
- removed C104, C105: 1uF/50V, Capacitor_SMD:C_0805_2012Metric_Pad1.18x1.45mm_HandSolder
- removed R101, R102, R103, R104, R105, R106: 22R, Resistor_SMD:R_0805_2012Metric_Pad1.20x1.40mm_HandSolder
- removed U101, U102, U103: NE5532, Package_SO:SOIC-8_3.9x4.9mm_P1.27mm
- added C502: 100nF/50V, Capacitor_SMD:C_0805_2012Metric_Pad1.18x1.45mm_HandSolder, F.Cu at (33.0, 276.0)
- added C602: 100nF/50V, Capacitor_SMD:C_0805_2012Metric_Pad1.18x1.45mm_HandSolder, F.Cu at (53.0, 36.0)
- added C702: 100nF/50V, Capacitor_SMD:C_0805_2012Metric_Pad1.18x1.45mm_HandSolder, F.Cu at (189.0, 36.0)
- added R501: 22R, Resistor_SMD:R_0805_2012Metric_Pad1.20x1.40mm_HandSolder, F.Cu at (49.0, 279.5)
- added R502: 22R, Resistor_SMD:R_0805_2012Metric_Pad1.20x1.40mm_HandSolder, F.Cu at (49.0, 274.0)
- added R601: 22R, Resistor_SMD:R_0805_2012Metric_Pad1.20x1.40mm_HandSolder, F.Cu at (50.0, 50.0)
- added R602: 22R, Resistor_SMD:R_0805_2012Metric_Pad1.20x1.40mm_HandSolder, F.Cu at (55.0, 50.0)
- added R701: 22R, Resistor_SMD:R_0805_2012Metric_Pad1.20x1.40mm_HandSolder, F.Cu at (185.5, 50.0)
- added R702: 22R, Resistor_SMD:R_0805_2012Metric_Pad1.20x1.40mm_HandSolder, F.Cu at (190.0, 50.0)
- added TP201: TestPoint, TestPoint:TestPoint_Keystone_5000-5004_Miniature, B.Cu at (107.0, 275.0)
- added TP202: TestPoint, TestPoint:TestPoint_Keystone_5000-5004_Miniature, B.Cu at (111.0, 275.0)
- added TP203: TestPoint, TestPoint:TestPoint_Keystone_5000-5004_Miniature, B.Cu at (105.0, 272.0)
- added TP204: TestPoint, TestPoint:TestPoint_Keystone_5000-5004_Miniature, B.Cu at (109.0, 272.0)
- added TP205: TestPoint, TestPoint:TestPoint_Keystone_5000-5004_Miniature, B.Cu at (113.0, 272.0)
- added TP206: TestPoint, TestPoint:TestPoint_Keystone_5000-5004_Miniature, B.Cu at (115.0, 275.0)
- added TP301: TestPoint, TestPoint:TestPoint_Keystone_5000-5004_Miniature, B.Cu at (134.0, 270.0)
- added TP302: TestPoint, TestPoint:TestPoint_Keystone_5000-5004_Miniature, B.Cu at (132.0, 267.0)
- added TP303: TestPoint, TestPoint:TestPoint_Keystone_5000-5004_Miniature, B.Cu at (134.0, 276.0)
- added TP304: TestPoint, TestPoint:TestPoint_Keystone_5000-5004_Miniature, B.Cu at (132.0, 273.0)
- added TP401: TestPoint, TestPoint:TestPoint_Keystone_5000-5004_Miniature, B.Cu at (18.0, 281.0)
- added TP402: TestPoint, TestPoint:TestPoint_Keystone_5000-5004_Miniature, B.Cu at (16.0, 278.0)
- added TP403: TestPoint, TestPoint:TestPoint_Keystone_5000-5004_Miniature, B.Cu at (14.0, 281.0)
- added TP404: TestPoint, TestPoint:TestPoint_Keystone_5000-5004_Miniature, B.Cu at (12.0, 278.0)
- added TP405: TestPoint, TestPoint:TestPoint_Keystone_5000-5004_Miniature, B.Cu at (10.0, 281.0)
- added TP406: TestPoint, TestPoint:TestPoint_Keystone_5000-5004_Miniature, B.Cu at (8.00, 278.0)
- added TP407: TestPoint, TestPoint:TestPoint_Keystone_5000-5004_Miniature, B.Cu at (6.00, 281.0)
- added TP408: TestPoint, TestPoint:TestPoint_Keystone_5000-5004_Miniature, B.Cu at (2.00, 281.0)
- added TP409: TestPoint, TestPoint:TestPoint_Keystone_5000-5004_Miniature, B.Cu at (4.00, 278.0)
- added U502: 4052, Package_SO:SO-16_3.9x9.9mm_P1.27mm, F.Cu at (56.5, 277.0)
- added U602: 4052, Package_SO:SO-16_3.9x9.9mm_P1.27mm, F.Cu at (52.5, 57.5)
- added U702: 4052, Package_SO:SO-16_3.9x9.9mm_P1.27mm, F.Cu at (187.5, 57.5)
- C101, C102: value 100nF/50V -> 1uF/50V
- U501, U601, U701: value 4052 -> NE5532; footprint Package_SO:SO-16_3.9x9.9mm_P1.27mm -> Package_SO:SOIC-8_3.9x4.9mm_P1.27mm
- moved U701 331.5 mm to (188.0, 40.0)
- moved C701 317.0 mm to (185.0, 65.0), turned to 0 degrees
- moved U501 265.0 mm to (39.0, 277.0), turned to 90 degrees
- moved C101 263.8 mm to (120.0, 300.0)
- moved C501 244.0 mm to (66.0, 278.0), turned to 90 degrees
- moved C102 236.0 mm to (120.0, 271.0)
- moved C302 143.2 mm to (177.0, 234.0), turned to 180 degrees
- moved C316 139.5 mm to (171.0, 226.0)
- moved C312 130.1 mm to (172.5, 228.0), turned to 180 degrees
- moved C304 120.4 mm to (175.5, 232.0), turned to 180 degrees
- moved C311 117.4 mm to (180.0, 238.0), turned to 180 degrees
- moved C308 116.0 mm to (174.0, 230.0), turned to 180 degrees
- moved C306 113.0 mm to (178.5, 236.0), turned to 180 degrees
- moved C307 103.5 mm to (181.5, 240.0), turned to 180 degrees
- moved C310 90.5 mm to (180.0, 262.0), turned to 180 degrees
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Connections:
- C102 pad 1: VDDA -> VDD
- C201 pad 2: unconnected-(C201-Pad2) -> GND
- D201 pad 1: unconnected-(D201-K-Pad1) -> GND
- J101 pad 1: /ADC_3_CONN -> /Potentiometers/ADC_3
- J101 pad 10: /Potentiometers/msb -> /serial_CLR
- J101 pad 11: /serial_data -> GND
- J101 pad 12: GND -> /serial_CLK
- J101 pad 13: /register_CLK -> /Potentiometers/lsb
- J101 pad 14: /Potentiometers/lsb -> /register_CLK
- J101 pad 15: /serial_CLR -> /Buttons/I2C_SDA
- J101 pad 16: /Buttons/I2C_SCL -> /register_OE
- J101 pad 17: /serial_CLK -> GND
- J101 pad 18: GND -> /serial_data
- J101 pad 19: VDD -> /Buttons/I2C_SCL
- J101 pad 20: /Buttons/I2C_SDA -> VDD
- J101 pad 3: /ADC_2_CONN -> /Potentiometers/ADC_4
- J101 pad 4: /ADC_4_CONN -> /Potentiometers/ADC_2
- J101 pad 5: /ADC_1_CONN -> /Potentiometers/ADC_5
- J101 pad 6: /ADC_5_CONN -> /Potentiometers/ADC_1
- J101 pad 7: /ADC_0_CONN -> /Buttons/button_interrupt
- J101 pad 8: /Buttons/button_interrupt -> /Potentiometers/ADC_0
- J101 pad 9: /register_OE -> /Potentiometers/msb
- R201 pad 1: /LEDs/CH1_clip -> Net-(D201-A)
- R201 pad 2: Net-(D201-A) -> /LEDs/CH1_clip
- R229 pad 1: Net-(D229-A) -> /LEDs/Effect_CH1_Assign
- R229 pad 2: /LEDs/Effect_CH1_Assign -> Net-(D229-A)
- U201 pad 1: /LEDs/CH1_20db -> /LEDs/Effect_On_Status
- U201 pad 14: Net-(U201-SER) -> /serial_data
- U201 pad 15: /LEDs/CH1_25db -> /LEDs/MIDI_IN_INDICATOR
- U201 pad 2: /LEDs/CH1_12db -> /LEDs/EFFECT_CUE_STATUS
- U201 pad 3: /LEDs/CH1_9db -> /LEDs/SPARE_LED5
- U201 pad 4: /LEDs/CH1_6db -> /LEDs/SPARE_LED4
- U201 pad 5: /LEDs/CH1_3db -> /LEDs/SPARE_LED3
- U201 pad 6: /LEDs/CH1_0db -> /LEDs/SPARE_LED2
- U201 pad 7: /LEDs/CH1_clip -> /LEDs/SPARE_LED1
- U202 pad 14: Net-(U202-SER) -> Net-(U201-QH')
- U203 pad 9: Net-(U201-SER) -> Net-(U203-QH')
- U204 pad 1: /LEDs/CH2_CUE_Status -> /LEDs/CH1_20db
- U204 pad 14: Net-(U201-QH') -> Net-(U203-QH')
- U204 pad 15: /LEDs/Effect_CH1_Assign -> /LEDs/CH1_25db
- U204 pad 2: /LEDs/CH1_CUE_Status -> /LEDs/CH1_12db
- U204 pad 3: /LEDs/COL1_Sel_Status -> /LEDs/CH1_9db
- U204 pad 4: /LEDs/COL2_Sel_Status -> /LEDs/CH1_6db
- U204 pad 5: /LEDs/COL3_Sel_Status -> /LEDs/CH1_3db
- U204 pad 6: /LEDs/COL4_Sel_Status -> /LEDs/CH1_0db
- U204 pad 7: /LEDs/Effect_CH2_Assign -> /LEDs/CH1_clip
- U204 pad 9: unconnected-(U204-QH'-Pad9) -> Net-(U204-QH')
- U205 pad 1: /LEDs/Effect_On_Status -> /LEDs/Effect_CH2_Assign
- U205 pad 14: /serial_data -> Net-(U204-QH')
- U205 pad 15: /LEDs/MIDI_IN_INDICATOR -> /LEDs/Effect_CH1_Assign
- U205 pad 2: /LEDs/EFFECT_CUE_STATUS -> /LEDs/CH2_CUE_Status
- U205 pad 3: /LEDs/SPARE_LED5 -> /LEDs/CH1_CUE_Status
- U205 pad 4: /LEDs/SPARE_LED4 -> /LEDs/COL1_Sel_Status
- U205 pad 5: /LEDs/SPARE_LED3 -> /LEDs/COL2_Sel_Status
- U205 pad 6: /LEDs/SPARE_LED2 -> /LEDs/COL3_Sel_Status
- U205 pad 7: /LEDs/SPARE_LED1 -> /LEDs/COL4_Sel_Status
- U205 pad 9: Net-(U202-SER) -> unconnected-(U205-QH'-Pad9)
- U301 pad 16: unconnected-(U301-P13-Pad16) -> /Buttons/CUE_CH1_SEL
- U301 pad 17: unconnected-(U301-P14-Pad17) -> /Buttons/COLOUR_SEL_1
- U501 pad 1: /Potentiometers/EFFECT_PARAM_2 -> /Potentiometers/ADC_0
- U501 pad 2: /Potentiometers/EFFECT_PARAM_1 -> /Potentiometers/ADC_0
- U501 pad 3: /Potentiometers/ADC_3 -> Net-(U501A-+)
- U501 pad 4: /Potentiometers/SPARE5 -> GND
- U501 pad 5: /Potentiometers/CH2_GAIN -> Net-(U501B-+)
- U501 pad 6: GND -> /Potentiometers/ADC_1
- U501 pad 7: GND -> /Potentiometers/ADC_1
- U501 pad 8: GND -> VDDA
- U601 pad 1: /Potentiometers/CH1_HI -> /Potentiometers/ADC_2
- U601 pad 2: /Potentiometers/CH2_HI -> /Potentiometers/ADC_2
- U601 pad 3: /Potentiometers/ADC_1 -> Net-(U601A-+)
- U601 pad 4: /Potentiometers/CH1_GAIN -> GND
- U601 pad 5: /Potentiometers/SPARE1 -> Net-(U601B-+)
- U601 pad 6: GND -> /Potentiometers/ADC_3
- U601 pad 7: GND -> /Potentiometers/ADC_3
- U601 pad 8: GND -> VDDA
- U701 pad 1: /Potentiometers/analogueIOexpander2/IN_Y0 -> /Potentiometers/ADC_4
- U701 pad 2: /Potentiometers/analogueIOexpander2/IN_Y2 -> /Potentiometers/ADC_4
- U701 pad 3: /Potentiometers/ADC_5 -> Net-(U701A-+)
- U701 pad 4: /Potentiometers/analogueIOexpander2/IN_Y3 -> GND
- U701 pad 5: /Potentiometers/CH1_VOL -> Net-(U701B-+)
- U701 pad 6: GND -> /Potentiometers/ADC_5
- U701 pad 7: GND -> /Potentiometers/ADC_5
- U701 pad 8: GND -> VDDA
Routing:
- net /Potentiometers/ADC_5: track 0.00 -> 659.6 mm, vias 0 -> 4
- net /Potentiometers/ADC_4: track 0.00 -> 627.7 mm, vias 0 -> 2
- net /ADC_3_CONN: track 603.4 -> 0.00 mm, vias 4 -> 0
- net /ADC_2_CONN: track 592.6 -> 0.00 mm, vias 2 -> 0
- net VDDA: track 1062.6 -> 1632.4 mm, vias 0 -> 5
- net /Potentiometers/ADC_3: track 10.1 -> 453.0 mm
- net /ADC_1_CONN: track 409.5 -> 0.00 mm
- net /Potentiometers/ADC_2: track 8.66 -> 417.3 mm
- net /ADC_0_CONN: track 383.1 -> 0.00 mm
- net /Potentiometers/EFFECT_WET_DRY: track 0.00 -> 317.4 mm, vias 0 -> 4
- net VDD: track 186.6 -> 503.0 mm, vias 11 -> 26
- net /Buttons/CUE_CH1_SEL: track 0.00 -> 211.2 mm, vias 0 -> 4
- net /Buttons/COLOUR_SEL_4: track 8.65 -> 218.7 mm, vias 0 -> 4
- net /Buttons/COLOUR_SEL_1: track 2.41 -> 211.5 mm, vias 0 -> 4
- net /Buttons/COLOUR_SEL_3: track 7.52 -> 215.1 mm, vias 0 -> 4
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Other:
- board text added: "Button Test Pins"

Commit message: Fix DRC erros and warnings
Parts:
- moved C204 167.9 mm to (109.0, 186.5), turned to -90 degrees
- moved C205 128.6 mm to (108.0, 238.0), turned to 180 degrees
- moved C201 70.7 mm to (133.0, 253.0), turned to 0 degrees
- moved C202 17.5 mm to (144.0, 186.5)
- moved C203 17.5 mm to (126.5, 186.5)
Routing:
- net VDDA: track 1632.4 -> 1780.3 mm, vias 5 -> 4
- net GND: track 231.5 -> 244.9 mm, vias 95 -> 100
- net VDD: track 503.0 -> 512.6 mm
- net /Potentiometers/msb: track 800.3 -> 802.7 mm
- net /Potentiometers/lsb: track 817.7 -> 820.2 mm
- net /Buttons/I2C_SCL: track 77.6 -> 79.6 mm
Other:
- board text added: "ADC_0"
- board text added: "ADC_1"
- board text added: "ADC_2"
- board text added: "ADC_3"
- board text added: "ADC_4"
- board text added: "ADC_5"
- board text added: "GND"
- board text added: "INT"
- board text added: "LSB"
- board text added: "MSB"
- board text added: "REG_CK"
- board text added: "REG_OE"
- board text added: "SCL"
- board text added: "SDA"
- board text added: "SER_CK"
- board text added: "SER_CLR"
- board text added: "SER_DATA"

Commit message: Fix DRC issues from rounded tracks
Routing:
- net /Potentiometers/lsb: track 820.2 -> 826.6 mm
- net /Potentiometers/msb: track 802.7 -> 808.3 mm
- net /Potentiometers/ADC_4: track 627.7 -> 632.9 mm
- net /serial_CLR: track 189.3 -> 184.3 mm
- net /Potentiometers/CH1_COLOUR: track 148.3 -> 153.3 mm
- net VDDA: track 1780.3 -> 1775.7 mm
- net /Potentiometers/CH1_LOW: track 109.4 -> 113.2 mm
- net Net-(D233-A): track 112.4 -> 115.6 mm
- net /Potentiometers/CH1_HI: track 73.1 -> 75.0 mm
- net /Buttons/EFFECT ON: track 119.5 -> 117.7 mm
- net Net-(D238-A): track 267.4 -> 269.2 mm
- net /Potentiometers/ADC_5: track 659.6 -> 661.3 mm
- net /Potentiometers/CH1_LOW-MID: track 81.7 -> 83.2 mm
- net /Potentiometers/CH2_HI: track 147.2 -> 148.7 mm
- net Net-(D236-A): track 276.4 -> 277.6 mm
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
Commit message: Make rounded lines look nicer for the analogue part
Routing:
- net /Potentiometers/lsb: track 826.6 -> 833.7 mm
- net /Potentiometers/msb: track 808.3 -> 814.7 mm
- net /Potentiometers/COLOUR_PARAM: track 147.2 -> 150.1 mm
- net /Potentiometers/CH1_VOL: track 40.5 -> 43.3 mm
- net /Buttons/button_interrupt: track 106.4 -> 108.7 mm
- net /Potentiometers/ADC_0: track 152.3 -> 154.0 mm
- net /Potentiometers/ADC_1: track 167.1 -> 168.8 mm
- net /Potentiometers/SPARE5: track 65.4 -> 66.6 mm
- net /Potentiometers/SPARE2: track 261.2 -> 260.0 mm
- net Net-(U501B-+): track 8.42 -> 7.31 mm
- net /Potentiometers/EFFECT_PARAM_1: track 126.6 -> 127.6 mm
- net VDDA: track 1775.7 -> 1774.7 mm
- net /Potentiometers/CH2_HI: track 148.7 -> 149.6 mm
- net Net-(U501A-+): track 10.3 -> 11.1 mm
- net /Potentiometers/ADC_3: track 453.4 -> 454.1 mm
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Other:
- board text removed: "COLOUR FX PARAM"

Commit message: Make rounded traces look better for digital signals
Parts:
- moved D230 15.0 mm to (210.0, 306.0)
Routing:
- net Net-(D230-A): track 122.8 -> 109.6 mm
- net Net-(D228-A): track 185.5 -> 174.8 mm
- net Net-(D236-A): track 277.6 -> 282.1 mm
- net Net-(D239-A): track 298.1 -> 302.3 mm
- net Net-(D240-A): track 287.5 -> 291.4 mm
- net Net-(D231-A): track 100.0 -> 103.8 mm
- net Net-(D235-A): track 309.1 -> 312.4 mm
- net Net-(D238-A): track 269.2 -> 272.2 mm
- net VDDA: track 1774.7 -> 1777.1 mm
- net Net-(D233-A): track 115.6 -> 118.0 mm
- net Net-(D225-A): track 78.0 -> 80.3 mm
- net VDD: track 513.0 -> 511.0 mm, vias 26 -> 25
- net Net-(U204-QH'): track 70.8 -> 72.7 mm
- net /serial_CLR: track 184.3 -> 182.5 mm
- net /LEDs/Effect_CH2_Assign: track 154.2 -> 156.0 mm
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Other:
- board text added: "MIDI ACTIVE"
