File: PCB/Magna/io_daughterboard/io_daughterboard.kicad_pcb (KiCad board)
At the start: 2 copper layers, 240 x 320 mm, 223 parts, among them J101 Conn_02x10_Counter_Clockwise, U201 74HC595, U202 74HC595, U203 74HC595, U204 74HC595, U205 74HC595, U301 XL9535, U501 NE5532, U502 4052, U601 NE5532, U602 4052, U701 NE5532, U702 4052

Commit message: Make IO daughterboard production ready
Parts:
- added REF**: JLC_toolinghole, JLC:JLC_toolinghole, F.Cu at (7.50, 7.50)
- added REF**: JLC_toolinghole, JLC:JLC_toolinghole, F.Cu at (235.0, 315.0)
Other:
- board text added: "JLCJLCJLCJLC"
Changed lines of the file:
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@@
     )
   )
+  (footprint "JLC:JLC_toolinghole" (layer "F.Cu")
+    (at 7.5 7.5)
+    (attr through_hole)
+    (fp_text reference "REF**" (at 0 -1.905 unlocked) (layer "F.SilkS")
+        (effects (font (size 1 1) (thickness 0.15)))
+    )
+    (fp_text value "JLC_toolinghole" (at 0 1.524 unlocked) (layer "F.Fab")
+        (effects (font (size 1 1) (thickness 0.15)))
+    )
+    (pad "" np_thru_hole circle (at 0 0) (size 1.3 1.3) (drill 1.152) (layers "*.Mask"))
+  )
   (footprint "Diode_SMD:D_0805_2012Metric_Pad1.15x1.40mm_HandSolder" (layer "F.Cu")
     (at 141.025 57.5)
@@
     )
   )
+  (footprint "JLC:JLC_toolinghole" (layer "F.Cu")
+    (at 235 315)
+    (attr through_hole)
+    (fp_text reference "REF**" (at 0 -1.905 unlocked) (layer "F.SilkS")
+        (effects (font (size 1 1) (thickness 0.15)))
+    )
+    (fp_text value "JLC_toolinghole" (at 0 1.524 unlocked) (layer "F.Fab")
+        (effects (font (size 1 1) (thickness 0.15)))
+    )
+    (pad "" np_thru_hole circle (at 0 0) (size 1.3 1.3) (drill 1.152) (layers "*.Mask"))
+  )
   (footprint "Capacitor_SMD:C_0805_2012Metric_Pad1.18x1.45mm_HandSolder" (layer "F.Cu")
     (at 174 270 180)
@@
     (effects (font (size 3 3) (thickness 0.5) bold))
   )
+  (gr_text "JLCJLCJLCJLC" (at 82.5 252.27 90) (layer "F.SilkS")
+    (effects (font (size 1.5 1.5) (thickness 0.3) bold))
+  )
   (gr_text "SFX ON" (at 210 267.5) (layer "F.SilkS")
