File: PCB/Magna/io_daughterboard/LEDs.kicad_sch (KiCad schematic)
At the start: 96 parts, among them U2001 74HC595, U2002 74HC595, U2003 74HC595, U2004 74HC595, U2005 74HC595

Commit message: Update schematics to Kicad 9
Parts:
- renumbered C2001 to C201, C2002 to C202, C2003 to C203, C2004 to C204, C2005 to C205, D2001 to D201, D2002 to D202, D2003 to D203, D2004 to D204, D2005 to D205, D2006 to D206, D2007 to D207, D2008 to D208, D2009 to D209, D2010 to D210, D2011 to D211, D2012 to D212, D2013 to D213, D2014 to D214, D2015 to D215, D2016 to D216, D2017 to D217, D2018 to D218, D2019 to D219, D2020 to D220, D2021 to D221, D2022 to D222, D2023 to D223, D2024 to D224, D2025 to D225, D2026 to D226, D2027 to D227, D2028 to D228, D2029 to D229, D2030 to D230, D2031 to D231, D2032 to D232, D2033 to D233, D2034 to D234, D2035 to D235, D2036 to D236, D2037 to D237, D2038 to D238, D2039 to D239, D2040 to D240, R2001 to R201, R2002 to R202, R2003 to R203, R2004 to R204, R2005 to R205, R2006 to R206, R2007 to R207, R2008 to R208, R2009 to R209, R2010 to R210, R2011 to R211, R2012 to R212, R2013 to R213, R2014 to R214, R2015 to R215, R2016 to R216, R2017 to R217, R2018 to R218, R2019 to R219, R2020 to R220, R2021 to R221, R2022 to R222, R2023 to R223, R2024 to R224, R2025 to R225, R2026 to R226, R2027 to R227, R2028 to R228, R2029 to R229, R2030 to R230, R2031 to R231, R2032 to R232, R2033 to R233, R2034 to R234, R2035 to R235, R2036 to R236, R2037 to R237, R2038 to R238, R2039 to R239, R2040 to R240, TP2001 to TP201, TP2002 to TP202, TP2003 to TP203, TP2004 to TP204, TP2005 to TP205, TP2006 to TP206, U2005 to U201, U2002 to U202, U2003 to U203, U2001 to U204, U2004 to U205
