File: PCB/Magna/audio_daughterboard/Audio_daughterboard.kicad_pcb (KiCad board)
At the start: 2 copper layers, 90 x 320 mm, 240 parts, among them J201 PSG01550, J301 PSG01550, J601 AudioJack3, J701 PSG01550, U101 24.576 MHz, U102 CY2305SXC-1HT, U103 CY2305SXC-1HT, U201 WM8782SEDS, U301 WM8782SEDS, U401 CS4344, U402 NE5532, U501 CS4344, U502 NE5532, U601 NE5532, U602 NE5532, U603 TDA2822D, U701 NE5532, U702 NE5532, U703 NE5532, U801 NE5532, U901 TPS61040DBV, U902 AMS1117-5.0

Commit message: Add inital layout for Audio Daughterboard
Parts:
- moved TP701 250.7 mm to (46.5, 280.6), turned to 180 degrees
- moved C701 245.3 mm to (54.3, 279.0), turned to 180 degrees
- moved R401 245.2 mm to (6.38, 186.0), turned to 180 degrees
- moved R402 241.6 mm to (6.38, 183.1), turned to 180 degrees
- moved TP702 240.7 mm to (46.5, 275.5), turned to 180 degrees
- moved RV601 238.2 mm to (32.0, 312.2), turned to 90 degrees
- moved R403 238.0 mm to (6.38, 180.1), turned to 180 degrees
- moved C401 237.8 mm to (11.2, 186.0), turned to 180 degrees
- moved R404 234.6 mm to (6.38, 177.2), turned to 180 degrees
- moved C402 234.0 mm to (11.2, 183.0), turned to 180 degrees
- moved R405 231.2 mm to (6.38, 174.2), turned to 180 degrees
- moved J601 231.1 mm to (11.0, 315.0)
- moved TP703 230.8 mm to (46.5, 270.4), turned to 180 degrees
- moved C403 230.2 mm to (11.2, 179.9), turned to 180 degrees
- moved C702 229.1 mm to (54.3, 270.9), turned to 180 degrees
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
Commit message: Update schematics to Kicad 9
Parts:
- removed C101: F/NM, Capacitor_SMD:C_0603_1608Metric_Pad1.08x0.95mm_HandSolder
- removed C403: 100nF/50V, Capacitor_SMD:C_0805_2012Metric_Pad1.18x1.45mm_HandSolder
- removed C404, C405, C407, C408, C411, C412, C508, C511, C512: 10uF/25V, Capacitor_SMD:CP_Elec_4x5.8
- removed C409, C410, C509: 10nF/50V, Capacitor_SMD:C_0805_2012Metric_Pad1.18x1.45mm_HandSolder
- removed C701, C702: 100u/10V, Capacitor_SMD:CP_Elec_6.3x5.8
- removed C704, C705: 22uF/16V, Capacitor_SMD:CP_Elec_5x5.8
- removed C708, C709: 100pF/50V, Capacitor_SMD:C_0805_2012Metric_Pad1.18x1.45mm_HandSolder
- removed C710, C711: 220uF, Capacitor_SMD:CP_Elec_4x5.8
- removed the D901 at (55.9, 96.8)
- removed JP101, JP102, JP103, JP104, JP105, JP106, JP107, JP108, JP109, JP110: Jumper_2_Open, Jumper:SolderJumper-2_P1.3mm_Open_TrianglePad1.0x1.5mm
- removed JP201, JP202, JP203, JP204, JP301, JP302, JP303, JP304: SolderJumper_3_Bridged12, Jumper:SolderJumper-3_P2.0mm_Open_TrianglePad1.0x1.5mm_NumberLabels
- removed R101, R102: R/NM, Resistor_SMD:R_0805_2012Metric_Pad1.20x1.40mm_HandSolder
- removed R201, R202, R301, R302: 5k1, Resistor_SMD:R_0805_2012Metric_Pad1.20x1.40mm_HandSolder
- removed R401, R402, R501, R502: 10k, Resistor_SMD:R_0805_2012Metric_Pad1.20x1.40mm_HandSolder
- removed R403, R404, R503, R504: 470R, Resistor_SMD:R_0805_2012Metric_Pad1.20x1.40mm_HandSolder
- removed R405, R406, R505, R506, R701, R702: 22k, Resistor_SMD:R_0805_2012Metric_Pad1.20x1.40mm_HandSolder
- removed R703, R704: 680R, Resistor_SMD:R_0805_2012Metric_Pad1.20x1.40mm_HandSolder
- removed R705, R706: 1k3, Resistor_SMD:R_0805_2012Metric_Pad1.20x1.40mm_HandSolder
- removed RV201, RV301, RV701: 10k/PTV112-4420A-B103, Skrooter_footprints:Potentiometer_Bourns_PTV09A-1_Dual_Vertical
- removed TP401, TP402, TP404, TP405, TP501, TP502, TP504, TP505: TestPoint, TestPoint:TestPoint_Keystone_5005-5009_Compact
- removed the U101 at (9.39, 88.5)
- removed U401: CS4344, Package_SO:MSOP-10_3x3mm_P0.5mm
- removed U402, U502: NE5532, Package_SO:SOIC-8_3.9x4.9mm_P1.27mm
- added C1006: 100nF, Capacitor_SMD:C_0805_2012Metric_Pad1.18x1.45mm_HandSolder, F.Cu at (65.1, 65.6)
- added C1007: 100nF, Capacitor_SMD:C_0805_2012Metric_Pad1.18x1.45mm_HandSolder, F.Cu at (65.1, 68.6)
- added C1010: 100nF, Capacitor_SMD:C_0805_2012Metric_Pad1.18x1.45mm_HandSolder, F.Cu at (65.1, 71.6)
- added C1012: 100nF, Capacitor_SMD:C_0805_2012Metric_Pad1.18x1.45mm_HandSolder, F.Cu at (65.1, 74.7)
- added C1013: 100nF, Capacitor_SMD:C_0805_2012Metric_Pad1.18x1.45mm_HandSolder, F.Cu at (65.1, 77.7)
- added C1106: 100nF, Capacitor_SMD:C_0805_2012Metric_Pad1.18x1.45mm_HandSolder, F.Cu at (68.8, 24.4)
- added C1107: 100nF, Capacitor_SMD:C_0805_2012Metric_Pad1.18x1.45mm_HandSolder, F.Cu at (68.8, 27.4)
- added C1110: 100nF, Capacitor_SMD:C_0805_2012Metric_Pad1.18x1.45mm_HandSolder, F.Cu at (68.8, 30.4)
- added C1112: 100nF, Capacitor_SMD:C_0805_2012Metric_Pad1.18x1.45mm_HandSolder, F.Cu at (68.8, 33.4)
- added C1113: 100nF, Capacitor_SMD:C_0805_2012Metric_Pad1.18x1.45mm_HandSolder, F.Cu at (68.8, 36.4)
- added C1206: 100nF, Capacitor_SMD:C_0805_2012Metric_Pad1.18x1.45mm_HandSolder, F.Cu at (6.96, 45.7)
- added C1207: 100nF, Capacitor_SMD:C_0805_2012Metric_Pad1.18x1.45mm_HandSolder, F.Cu at (6.96, 48.7)
- added C1210: 100nF, Capacitor_SMD:C_0805_2012Metric_Pad1.18x1.45mm_HandSolder, F.Cu at (6.96, 51.7)
- added C1212: 100nF, Capacitor_SMD:C_0805_2012Metric_Pad1.18x1.45mm_HandSolder, F.Cu at (6.96, 54.7)
- added C1213: 100nF, Capacitor_SMD:C_0805_2012Metric_Pad1.18x1.45mm_HandSolder, F.Cu at (6.96, 57.7)
- added C1306: 100nF, Capacitor_SMD:C_0805_2012Metric_Pad1.18x1.45mm_HandSolder, F.Cu at (6.96, 62.9)
- added C1307: 100nF, Capacitor_SMD:C_0805_2012Metric_Pad1.18x1.45mm_HandSolder, F.Cu at (6.96, 65.9)
- added C1310: 100nF, Capacitor_SMD:C_0805_2012Metric_Pad1.18x1.45mm_HandSolder, F.Cu at (6.96, 68.9)
- added C1312: 100nF, Capacitor_SMD:C_0805_2012Metric_Pad1.18x1.45mm_HandSolder, F.Cu at (6.96, 71.9)
- added C1313: 100nF, Capacitor_SMD:C_0805_2012Metric_Pad1.18x1.45mm_HandSolder, F.Cu at (6.96, 74.9)
- added C413: 100nF/50V, Capacitor_SMD:C_0805_2012Metric_Pad1.18x1.45mm_HandSolder, F.Cu at (71.5, 1.00)
- added C414: 1uF/50V, Capacitor_SMD:C_0805_2012Metric_Pad1.18x1.45mm_HandSolder, F.Cu at (71.5, 4.01)
- added C415: 100nF/50V, Capacitor_SMD:C_0805_2012Metric_Pad1.18x1.45mm_HandSolder, F.Cu at (71.5, 7.03)
- added C416: 1uF/50V, Capacitor_SMD:C_0805_2012Metric_Pad1.18x1.45mm_HandSolder, F.Cu at (71.5, 10.0)
- added C417: 10uF/25V, Capacitor_SMD:CP_Elec_4x5.8, F.Cu at (65.2, 2.42)
- added C418: 10uF/25V, Capacitor_SMD:CP_Elec_4x5.8, F.Cu at (65.2, 8.28)
- added C420: 10uF/25V, Capacitor_SMD:CP_Elec_4x5.8, F.Cu at (65.2, 14.1)
- added C514: 100nF/50V, Capacitor_SMD:C_0805_2012Metric_Pad1.18x1.45mm_HandSolder, F.Cu at (60.1, 60.6)
- added C520: 10uF/25V, Capacitor_SMD:CP_Elec_4x5.8, F.Cu at (66.3, 55.7)
- added C902: 4.7uF, Capacitor_SMD:C_0805_2012Metric_Pad1.18x1.45mm_HandSolder, F.Cu at (43.9, 42.6)
- added C906: 4.7uF, Capacitor_SMD:C_0805_2012Metric_Pad1.18x1.45mm_HandSolder, F.Cu at (43.9, 45.6)
- added C908: 22uF, Capacitor_SMD:CP_Elec_5x5.8, F.Cu at (37.0, 44.5)
- added C909: 4.7uF, Capacitor_SMD:C_0805_2012Metric_Pad1.18x1.45mm_HandSolder, F.Cu at (43.9, 48.6)
- added C915: 4.7uF, Capacitor_SMD:C_0805_2012Metric_Pad1.18x1.45mm_HandSolder, F.Cu at (43.9, 51.6)
- added C916: 22uF, Capacitor_SMD:CP_Elec_5x5.8, F.Cu at (37.0, 51.3)
- added C917: 4.7uF, Capacitor_SMD:C_0805_2012Metric_Pad1.18x1.45mm_HandSolder, F.Cu at (43.9, 54.6)
- added C918: 4.7uF, Capacitor_SMD:C_0805_2012Metric_Pad1.18x1.45mm_HandSolder, F.Cu at (43.9, 57.6)
- added D902: Red, Diode_SMD:D_0805_2012Metric_Pad1.15x1.40mm_HandSolder, F.Cu at (48.7, 52.7)
- added D904: Red, Diode_SMD:D_0805_2012Metric_Pad1.15x1.40mm_HandSolder, F.Cu at (48.7, 55.7)
- added D905: Red, Diode_SMD:D_0805_2012Metric_Pad1.15x1.40mm_HandSolder, F.Cu at (48.7, 58.8)
- added FB903: FerriteBead, Inductor_SMD:L_0805_2012Metric, F.Cu at (53.4, 55.3)
- added FB905: FerriteBead, Inductor_SMD:L_0805_2012Metric, F.Cu at (53.4, 58.0)
- added J101: Conn_02x15_Odd_Even, Connector_PinHeader_2.54mm:PinHeader_2x16_P2.54mm_Horizontal, F.Cu at (1.79, 1.79)
- added R906: 470, Resistor_SMD:R_0805_2012Metric_Pad1.20x1.40mm_HandSolder, F.Cu at (38.9, 56.2)
- added R912: 470, Resistor_SMD:R_0805_2012Metric_Pad1.20x1.40mm_HandSolder, F.Cu at (38.9, 59.2)
- added R913: 680, Resistor_SMD:R_0805_2012Metric_Pad1.20x1.40mm_HandSolder, F.Cu at (38.9, 62.1)
- added TP1001: TestPoint, TestPoint:TestPoint_Keystone_5005-5009_Compact, F.Cu at (60.2, 66.6)
- added TP1002: TestPoint, TestPoint:TestPoint_Keystone_5005-5009_Compact, F.Cu at (60.2, 71.7)
- added TP1003: TestPoint, TestPoint:TestPoint_Keystone_5005-5009_Compact, F.Cu at (60.2, 76.7)
- added TP102: TestPoint, TestPoint:TestPoint_Keystone_5005-5009_Compact, F.Cu at (17.9, 7.08)
- added TP109: TestPoint, TestPoint:TestPoint_Keystone_5005-5009_Compact, F.Cu at (23.0, 7.08)
- added TP1101: TestPoint, TestPoint:TestPoint_Keystone_5005-5009_Compact, F.Cu at (63.8, 25.4)
- added TP1102: TestPoint, TestPoint:TestPoint_Keystone_5005-5009_Compact, F.Cu at (63.8, 30.5)
- added TP1103: TestPoint, TestPoint:TestPoint_Keystone_5005-5009_Compact, F.Cu at (63.8, 35.5)
- added TP111: TestPoint, TestPoint:TestPoint_Keystone_5005-5009_Compact, F.Cu at (23.0, 17.2)
- added TP112: TestPoint, TestPoint:TestPoint_Keystone_5005-5009_Compact, F.Cu at (23.0, 22.2)
- added TP113: TestPoint, TestPoint:TestPoint_Keystone_5005-5009_Compact, F.Cu at (23.0, 27.3)
- added TP116: TestPoint, TestPoint:TestPoint_Keystone_5005-5009_Compact, F.Cu at (28.0, 2.02)
- added TP117: TestPoint, TestPoint:TestPoint_Keystone_5005-5009_Compact, F.Cu at (28.0, 7.08)
- added TP118: TestPoint, TestPoint:TestPoint_Keystone_5005-5009_Compact, F.Cu at (28.0, 12.1)
- added TP119: TestPoint, TestPoint:TestPoint_Keystone_5005-5009_Compact, F.Cu at (28.0, 17.2)
- added TP120: TestPoint, TestPoint:TestPoint_Keystone_5005-5009_Compact, F.Cu at (28.0, 22.2)
- added TP1201: TestPoint, TestPoint:TestPoint_Keystone_5005-5009_Compact, F.Cu at (2.02, 46.7)
- added TP1202: TestPoint, TestPoint:TestPoint_Keystone_5005-5009_Compact, F.Cu at (2.02, 51.8)
- added TP1203: TestPoint, TestPoint:TestPoint_Keystone_5005-5009_Compact, F.Cu at (2.02, 56.8)
- added TP1301: TestPoint, TestPoint:TestPoint_Keystone_5005-5009_Compact, F.Cu at (2.02, 63.9)
- added TP1302: TestPoint, TestPoint:TestPoint_Keystone_5005-5009_Compact, F.Cu at (2.02, 68.9)
- added TP1303: TestPoint, TestPoint:TestPoint_Keystone_5005-5009_Compact, F.Cu at (2.02, 74.0)
- added TP904: TestPoint, TestPoint:TestPoint_Keystone_5005-5009_Compact, F.Cu at (48.8, 43.6)
- added TP906: TestPoint, TestPoint:TestPoint_Keystone_5005-5009_Compact, F.Cu at (48.8, 48.6)
- added U1005: LM1971M, Package_SO:SOIC-8_3.9x4.9mm_P1.27mm, F.Cu at (71.7, 67.5)
- added U1105: LM1971M, Package_SO:SOIC-8_3.9x4.9mm_P1.27mm, F.Cu at (75.4, 26.2)
- added U1205: LM1971M, Package_SO:SOIC-8_3.9x4.9mm_P1.27mm, F.Cu at (13.6, 47.6)
- added U1305: LM1971M, Package_SO:SOIC-8_3.9x4.9mm_P1.27mm, F.Cu at (13.6, 64.7)
- added U1306: STM32F030C8Tx, Package_QFP:LQFP-48_7x7mm_P0.5mm, F.Cu at (38.2, 73.3)
- added U403: PCM1789, Package_SO:TSSOP-24_4.4x7.8mm_P0.65mm, F.Cu at (73.8, 16.2)
- added U903: TLV76701DRVx, Package_SON:WSON-6-1EP_2x2mm_P0.65mm_EP1x1.6mm_ThermalVias, F.Cu at (34.6, 60.2)
- added U904: TLV76701DRVx, Package_SON:WSON-6-1EP_2x2mm_P0.65mm_EP1x1.6mm_ThermalVias, F.Cu at (34.6, 63.9)
- C306, C501: value 100nF/50V -> 10uF/25V; footprint Capacitor_SMD:C_0805_2012Metric_Pad1.18x1.45mm_HandSolder -> Capacitor_SMD:CP_Elec_4x5.8
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- renumbered C208 to C205, C210 to C206, C205 to C207, C206 to C208, C207 to C209, C209 to C210, D903 to D901, D902 to D903, FB903 to FB904, R904 to R901, R903 to R907, TP102 to TP108, TP108 to TP114, TP109 to TP115, TP904 to TP905, U102 to U101, U103 to U102, U703 to U702, U702 to U703
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Connections:
- net Net-(U201-COM) renamed /AudioAdc0/VMID
- C201 pad 1: Net-(C201-Pad1) -> /AudioAdc0/Input Filtering1/signal_out
- C201 pad 2: Net-(J201-IN1) -> Net-(C201-Pad2)
- C202 pad 1: Net-(C202-Pad1) -> /AudioAdc0/Input Filtering/signal_out
- C202 pad 2: Net-(J201-IN2) -> Net-(C202-Pad2)
- C205 pad 1: VAA -> +3.3VA
- C206 pad 1: VAA -> +3.3VA
- C301 pad 1: Net-(C301-Pad1) -> /AudioAdc1/Input Filtering1/signal_out
- C301 pad 2: Net-(J301-IN1) -> Net-(C301-Pad2)
- C302 pad 1: Net-(C302-Pad1) -> /AudioAdc1/Input Filtering/signal_out
- C302 pad 2: Net-(J301-IN2) -> Net-(C302-Pad2)
- C305 pad 1: Net-(U301-COM) -> +3.3VA
- C306 pad 1: Net-(U301-VREFP) -> +3.3VA
- C307 pad 1: Net-(U301-COM) -> /AudioAdc1/VMID
- C308 pad 1: VAA -> Net-(U301-VREFP)
- C309 pad 1: Net-(U301-VREFP) -> /AudioAdc1/VMID
- C310 pad 1: VAA -> Net-(U301-VREFP)
- C401 pad 1: VAA -> +5VA
- C402 pad 1: VAA -> +5VA
- C501 pad 1: VAA -> VDD
- C502 pad 1: VAA -> VDD
- C503 pad 1: Net-(U501-VQ) -> VDD
- C504 pad 1: Net-(U501-VQ) -> /AudioDac1/VCOM
- C505 pad 1: Net-(U501-FILT+) -> /AudioDac1/VCOM
- C506 pad 1: VAA -> +5VA
- C507 pad 1: Net-(U501-AOUTL) -> +5VA
- C507 pad 2: Net-(C507-Pad2) -> GND
- C510 pad 1: Net-(C510-Pad1) -> +5VA
- C904 pad 1: /AudioPower/7V -> /AudioPower/16V
- C905 pad 1: /AudioPower/7V -> /AudioPower/16V
- C907 pad 1: Net-(U902-VI) -> Net-(U903-EN)
- C911 pad 1: Net-(U902-VO) -> Net-(U903-OUT)
- C912 pad 1: Net-(U902-VO) -> Net-(U903-OUT)
- FB902 pad 1: /AudioPower/7V -> /AudioPower/16V
- FB902 pad 2: Net-(U902-VI) -> Net-(U903-EN)
- FB904 pad 1: Net-(U902-VO) -> Net-(U903-OUT)
- J201 pad 1: Net-(J201-IN1) -> /AudioAdc0/Input Filtering1/signal in
- J201 pad 2: Net-(J201-IN2) -> /AudioAdc0/Input Filtering/signal in
- J301 pad 1: Net-(J301-IN1) -> /AudioAdc1/Input Filtering1/signal in
- J301 pad 2: Net-(J301-IN2) -> /AudioAdc1/Input Filtering/signal in
- L901 pad 2: /AudioPower/Boost Sw -> /AudioPower/Boost_SW
- R707 pad 2: VAA_BIAS_L -> unconnected-(R707-Pad2)
- R904 pad 1: /AudioPower/7V -> /AudioPower/16V
- R907 pad 1: /AudioPower/7V -> /AudioPower/16V
- TP101 pad 1: /ADCIN0 -> /DAC_DATA_1
- TP103 pad 1: /ADCIN1 -> /ADC_DATA_3
- TP104 pad 1: /LRCLK -> /ADC_DATA_2
- TP105 pad 1: Net-(JP101-B) -> /ADC_DATA_1
- TP106 pad 1: /DACOUT0 -> /ADC_DATA_0
- TP107 pad 1: /DACOUT1 -> /LRCLK
- TP110 pad 1: /ADC0_BCLK -> /MCLK
- TP114 pad 1: /MCLK -> Net-(U101-CLKOUT)
- TP201 pad 1: Net-(J201-IN1) -> /AudioAdc0/Input Filtering1/signal in
- TP202 pad 1: Net-(J201-IN2) -> /AudioAdc0/Input Filtering/signal in
- TP301 pad 1: Net-(J301-IN1) -> /AudioAdc1/Input Filtering1/signal in
- TP302 pad 1: Net-(J301-IN2) -> /AudioAdc1/Input Filtering/signal in
- TP901 pad 1: /AudioPower/Boost Sw -> /AudioPower/Boost_SW
- TP902 pad 1: /AudioPower/7V -> /AudioPower/16V
- U101 pad 1: Net-(JP101-B) -> /MCLK
- U101 pad 2: /ADC1_MCLK -> Net-(JP117-A)
- U101 pad 3: /ADC0_MCLK -> Net-(JP118-A)
- U101 pad 5: /DAC0_MCLK -> Net-(JP116-A)
- U101 pad 7: /DAC1_MCLK -> Net-(JP115-A)
- U101 pad 8: /MCLK -> Net-(U101-CLKOUT)
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
Commit message: Do most of the component placement for audio board
Just a general layout, things will probably change
as the routing begins.
Parts:
- removed the C205 at (36.4, 176.9)
- removed the C305 at (47.8, 27.1)
- removed the C505 at (60.1, 51.6)
- removed the C510 at (66.3, 49.8)
- removed the C703 at (89.3, 186.0)
- removed C706: 100nF/50V, Capacitor_SMD:C_0805_2012Metric_Pad1.18x1.45mm_HandSolder
- removed C715: 100u/10V, Capacitor_SMD:CP_Elec_6.3x5.8
- removed the C902 at (43.9, 42.6)
- removed the C908 at (37.0, 44.5)
- removed the C912 at (61.2, 75.5)
- removed the C916 at (37.0, 51.3)
- removed the D902 at (48.7, 52.7)
- removed the FB903 at (53.4, 55.3)
- removed the R707 at (84.5, 168.3)
- removed the R708 at (79.7, 186.0)
- removed the R709 at (79.7, 183.1)
- removed the R710 at (79.7, 180.1)
- removed the R904 at (63.3, 97.5)
- removed the TP702 at (46.5, 275.5)
- removed the TP703 at (46.5, 270.4)
- removed TP901, TP904: TestPoint, TestPoint:TestPoint_Keystone_5005-5009_Compact
- removed the TP903 at (73.0, 86.4)
- removed the U701 at (50.1, 71.0)
- removed U702: NE5532, Package_SO:SOIC-8_3.9x4.9mm_P1.27mm
- removed the U901 at (34.6, 56.6)
- removed U904: TLV76701DRVx, Package_SON:WSON-6-1EP_2x2mm_P0.65mm_EP1x1.6mm_ThermalVias
- added C1001: 390pF, Capacitor_SMD:C_0603_1608Metric, F.Cu at (5.00, 11.0)
- added C1002: 22uF, Skrooter_footprints:c_elec_SMD_12.5x13.5, F.Cu at (11.0, 22.0)
- added C1003: 10nF, Capacitor_SMD:C_0603_1608Metric, F.Cu at (14.0, 37.0)
- added C1004: 10nF, Capacitor_SMD:C_0603_1608Metric, F.Cu at (14.0, 34.0)
- added C1005: 10nF, Capacitor_SMD:C_0603_1608Metric, F.Cu at (5.00, 43.0)
- added C1008: 10nF, Capacitor_SMD:C_0603_1608Metric, F.Cu at (15.0, 49.0)
- added C1009: 10nF, Capacitor_SMD:C_0603_1608Metric, F.Cu at (15.0, 52.0)
- added C101: 100nF, Capacitor_SMD:C_0603_1608Metric, F.Cu at (38.0, 92.0)
- added C1011: 10nF, Capacitor_SMD:C_0603_1608Metric, F.Cu at (13.0, 55.0)
- added C102: 100nF, Capacitor_SMD:C_0603_1608Metric, F.Cu at (38.0, 100.0)
- added C1101: 390pF, Capacitor_SMD:C_0603_1608Metric, F.Cu at (30.0, 11.0)
- added C1102: 22uF, Skrooter_footprints:c_elec_SMD_12.5x13.5, F.Cu at (26.0, 22.0)
- added C1103: 10nF, Capacitor_SMD:C_0603_1608Metric, F.Cu at (29.0, 37.0)
- added C1104: 10nF, Capacitor_SMD:C_0603_1608Metric, F.Cu at (29.0, 34.0)
- added C1105: 10nF, Capacitor_SMD:C_0603_1608Metric, F.Cu at (20.0, 43.0)
- added C1108: 10nF, Capacitor_SMD:C_0603_1608Metric, F.Cu at (30.0, 49.0)
- added C1109: 10nF, Capacitor_SMD:C_0603_1608Metric, F.Cu at (30.0, 52.0)
- added C1111: 10nF, Capacitor_SMD:C_0603_1608Metric, F.Cu at (28.0, 55.0)
- added C1201: 390pF, Capacitor_SMD:C_0603_1608Metric, F.Cu at (50.0, 12.0)
- added C1202: 22uF, Skrooter_footprints:c_elec_SMD_12.5x13.5, F.Cu at (56.0, 23.0)
- added C1203: 10nF, Capacitor_SMD:C_0603_1608Metric, F.Cu at (59.0, 38.0)
- added C1204: 10nF, Capacitor_SMD:C_0603_1608Metric, F.Cu at (59.0, 35.0)
- added C1205: 10nF, Capacitor_SMD:C_0603_1608Metric, F.Cu at (50.0, 44.0)
- added C1208: 10nF, Capacitor_SMD:C_0603_1608Metric, F.Cu at (60.0, 50.0)
- added C1209: 10nF, Capacitor_SMD:C_0603_1608Metric, F.Cu at (60.0, 53.0)
- added C1211: 10nF, Capacitor_SMD:C_0603_1608Metric, F.Cu at (59.0, 56.0)
- added C1301: 390pF, Capacitor_SMD:C_0603_1608Metric, F.Cu at (35.0, 12.0)
- added C1302: 22uF, Skrooter_footprints:c_elec_SMD_12.5x13.5, F.Cu at (41.0, 23.0)
- added C1303: 10nF, Capacitor_SMD:C_0603_1608Metric, F.Cu at (44.0, 38.0)
- added C1304: 10nF, Capacitor_SMD:C_0603_1608Metric, F.Cu at (44.0, 35.0)
- added C1305: 10nF, Capacitor_SMD:C_0603_1608Metric, F.Cu at (35.0, 44.0)
- added C1308: 10nF, Capacitor_SMD:C_0603_1608Metric, F.Cu at (45.0, 50.0)
- added C1309: 10nF, Capacitor_SMD:C_0603_1608Metric, F.Cu at (45.0, 53.0)
- added C1311: 10nF, Capacitor_SMD:C_0603_1608Metric, F.Cu at (44.0, 56.0)
- added C1401: 100nF, Capacitor_SMD:C_0603_1608Metric, F.Cu at (40.5, 123.0)
- added C1402: 100nF, Capacitor_SMD:C_0603_1608Metric, F.Cu at (42.0, 123.0)
- added C1403: 100nF, Capacitor_SMD:C_0603_1608Metric, F.Cu at (45.5, 116.0)
- added C1404: 100nF, Capacitor_SMD:C_0603_1608Metric, F.Cu at (51.0, 128.0)
- added C1405: 100nF, Capacitor_SMD:C_0603_1608Metric, F.Cu at (43.0, 117.0)
- added C1406: 4.7uF, Capacitor_SMD:C_1206_3216Metric, F.Cu at (44.0, 114.0)
- added C401: 4.7uF, Capacitor_SMD:C_1206_3216Metric, F.Cu at (82.5, 77.0)
- added C403: 4.7uF, Capacitor_SMD:C_1206_3216Metric, F.Cu at (80.0, 77.0)
- added C404: 4.7uF, Capacitor_SMD:C_1206_3216Metric, F.Cu at (83.0, 66.0)
- added C407: 4.7uF, Capacitor_SMD:C_1206_3216Metric, F.Cu at (85.0, 71.0)
- added C408: 4.7uF, Capacitor_SMD:C_1206_3216Metric, F.Cu at (85.0, 76.0)
- added C411: 100u, Capacitor_SMD:CP_Elec_6.3x7.7, F.Cu at (78.2, 64.0)
- added C412: 100u, Capacitor_SMD:CP_Elec_6.3x7.7, F.Cu at (70.8, 64.0)
- added C413: 100nF, Capacitor_SMD:C_0603_1608Metric, F.Cu at (86.0, 33.0)
- added C415: 100u, Capacitor_SMD:CP_Elec_6.3x7.7, F.Cu at (66.0, 56.0)
- added C419: 1nF, Capacitor_SMD:C_0603_1608Metric, F.Cu at (85.0, 44.0)
- added C421: 390pF, Capacitor_SMD:C_0603_1608Metric, F.Cu at (79.0, 46.0)
- added C422: 390pF, Capacitor_SMD:C_0603_1608Metric, F.Cu at (71.0, 39.0)
- added C423: 390pF, Capacitor_SMD:C_0603_1608Metric, F.Cu at (81.0, 41.0)
- added C424: 2.2nF, Capacitor_SMD:C_0603_1608Metric, F.Cu at (76.0, 34.0)
- added C425: 2.2nF, Capacitor_SMD:C_0603_1608Metric, F.Cu at (86.0, 36.0)
- added C502: 4.7uF, Capacitor_SMD:C_1206_3216Metric, F.Cu at (7.50, 103.0)
- added C504: 4.7uF, Capacitor_SMD:C_1206_3216Metric, F.Cu at (10.0, 103.0)
- added C508: 4.7uF, Capacitor_SMD:C_1206_3216Metric, F.Cu at (8.00, 93.0)
- added C511: 100u, Capacitor_SMD:CP_Elec_6.3x7.7, F.Cu at (14.8, 105.0)
- added C512: 100u, Capacitor_SMD:CP_Elec_6.3x7.7, F.Cu at (22.2, 105.0)
- added C513: 100nF, Capacitor_SMD:C_0603_1608Metric, F.Cu at (7.00, 136.0)
- added C514: 100u, Capacitor_SMD:CP_Elec_6.3x7.7, F.Cu at (10.0, 113.0)
- added C515: 100u, Capacitor_SMD:CP_Elec_6.3x7.7, F.Cu at (27.0, 113.0)
- added C516: 1nF, Capacitor_SMD:C_0603_1608Metric, F.Cu at (20.0, 124.0)
- added C517: 1nF, Capacitor_SMD:C_0603_1608Metric, F.Cu at (22.0, 124.0)
- added C518: 1nF, Capacitor_SMD:C_0603_1608Metric, F.Cu at (11.0, 123.0)
- added C519: 1nF, Capacitor_SMD:C_0603_1608Metric, F.Cu at (8.00, 125.0)
- added C521: 390pF, Capacitor_SMD:C_0603_1608Metric, F.Cu at (14.0, 123.0)
- added C522: 390pF, Capacitor_SMD:C_0603_1608Metric, F.Cu at (22.0, 130.0)
- added C523: 390pF, Capacitor_SMD:C_0603_1608Metric, F.Cu at (12.0, 128.0)
- added C524: 2.2nF, Capacitor_SMD:C_0603_1608Metric, F.Cu at (17.0, 135.0)
- added C525: 2.2nF, Capacitor_SMD:C_0603_1608Metric, F.Cu at (7.00, 133.0)
- added C705: 100u, Capacitor_SMD:CP_Elec_6.3x7.7, F.Cu at (67.0, 18.0)
- added C904: 10uF, Capacitor_SMD:CP_Elec_4x5.8, F.Cu at (34.1, 143.2)
- added C910: 22pF, Capacitor_SMD:C_0603_1608Metric, F.Cu at (38.1, 133.2)
- added C913: 220uF, Capacitor_SMD:CP_Elec_4x5.8, F.Cu at (34.1, 153.2)
- added C914: 220uF, Capacitor_SMD:CP_Elec_4x5.8, F.Cu at (34.1, 136.2)
- added C917: 220uF, Capacitor_SMD:CP_Elec_4x5.8, F.Cu at (70.0, 147.5)
- added FB905: FerriteBead, Inductor_SMD:L_0805_2012Metric, F.Cu at (31.1, 139.7)
- added H101: MountingHole_Pad, MountingHole:MountingHole_3.2mm_M3_Pad_Via, F.Cu at (86.5, 3.50)
- added H102: MountingHole_Pad, MountingHole:MountingHole_3.2mm_M3_Pad_Via, F.Cu at (3.50, 3.50)
- added H103: MountingHole_Pad, MountingHole:MountingHole_3.2mm_M3_Pad_Via, F.Cu at (3.50, 166.5)
- added H104: MountingHole_Pad, MountingHole:MountingHole_3.2mm_M3_Pad_Via, F.Cu at (86.5, 166.5)
- added J102: Conn_02x05_Odd_Even, Connector_PinHeader_2.54mm:PinHeader_2x05_P2.54mm_Horizontal, F.Cu at (20.1, 159.3)
- added J103: Conn_02x05_Odd_Even, Connector_PinHeader_2.54mm:PinHeader_2x05_P2.54mm_Horizontal, F.Cu at (5.00, 280.0)
- added J1401: Conn_01x03_Pin, Connector_PinHeader_2.54mm:PinHeader_1x03_P2.54mm_Vertical, F.Cu at (57.0, 116.5)
- added J1402: Conn_ARM_SWD_TagConnect_TC2030, Connector:Tag-Connect_TC2030-IDC-FP_2x03_P1.27mm_Vertical, F.Cu at (64.0, 119.0)
- added J1403: Conn_01x02_Pin, Connector_PinHeader_2.54mm:PinHeader_1x02_P2.54mm_Vertical, F.Cu at (42.0, 111.0)
- added J1404: Conn_01x02_Pin, Connector_PinHeader_2.54mm:PinHeader_1x02_P2.54mm_Vertical, F.Cu at (38.0, 120.0)
- added JP101: Jumper_3_Bridged12, Jumper:SolderJumper-3_P1.3mm_Bridged12_RoundedPad1.0x1.5mm_NumberLabels, F.Cu at (51.0, 94.0)
- added JP102: Jumper_3_Bridged12, Jumper:SolderJumper-3_P1.3mm_Bridged12_RoundedPad1.0x1.5mm_NumberLabels, F.Cu at (57.0, 94.0)
- added JP103: Jumper_3_Bridged12, Jumper:SolderJumper-3_P1.3mm_Bridged12_RoundedPad1.0x1.5mm_NumberLabels, F.Cu at (54.0, 94.0)
- added JP104: Jumper_3_Bridged12, Jumper:SolderJumper-3_P1.3mm_Bridged12_RoundedPad1.0x1.5mm_NumberLabels, F.Cu at (48.0, 94.0)
- added JP105: Jumper_3_Bridged12, Jumper:SolderJumper-3_P1.3mm_Bridged12_RoundedPad1.0x1.5mm_NumberLabels, F.Cu at (48.0, 102.0)
- added JP106: Jumper_3_Bridged12, Jumper:SolderJumper-3_P1.3mm_Bridged12_RoundedPad1.0x1.5mm_NumberLabels, F.Cu at (51.0, 102.0)
- added JP107: Jumper_3_Bridged12, Jumper:SolderJumper-3_P1.3mm_Bridged12_RoundedPad1.0x1.5mm_NumberLabels, F.Cu at (54.0, 102.0)
- added JP108: Jumper_3_Bridged12, Jumper:SolderJumper-3_P1.3mm_Bridged12_RoundedPad1.0x1.5mm_NumberLabels, F.Cu at (57.0, 102.0)
- added Q701: NMOS, Package_TO_SOT_SMD:SOT-23-3, F.Cu at (81.0, 16.0)
- added Q702: NMOS, Package_TO_SOT_SMD:SOT-23-3, F.Cu at (81.0, 20.5)
- added R1001: 100R, Resistor_SMD:R_0603_1608Metric, F.Cu at (8.00, 12.0)
- added R1004: 100k, Resistor_SMD:R_0603_1608Metric, F.Cu at (5.00, 13.0)
- added R1005: 100k, Resistor_SMD:R_0603_1608Metric, F.Cu at (7.50, 30.5)
- added R1006: 100k, Resistor_SMD:R_0603_1608Metric, F.Cu at (7.50, 32.0)
- added R1007: 392R, Resistor_SMD:R_0603_1608Metric, F.Cu at (10.0, 34.0)
- added R1008: 732R, Resistor_SMD:R_0603_1608Metric, F.Cu at (10.0, 37.0)
- added R1009: 732R, Resistor_SMD:R_0603_1608Metric, F.Cu at (12.0, 37.0)
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- renumbered FB905 to FB903, TP403 to TP402, TP503 to TP502, TP704 to TP702, TP705 to TP703, TP902 to TP903, TP906 to TP905, TP905 to TP906, U1306 to U1401, U403 to U401, U703 to U701, U902 to U901
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Connections:
- net Net-(C714-Pad1) renamed /Line Driver/LINE_OUT_BIASED_L
- net Net-(C715-Pad1) renamed /Line Driver/LINE_OUT_BIASED_R
- C206 pad 1: +3.3VA -> /AudioAdc0/VMID
- C306 pad 1: +3.3VA -> /AudioAdc1/VMID
- C402 pad 1: +5VA -> /AudioDac0/VCOM
- C414 pad 1: /AudioDac0/VCOM -> /AudioDac0/VOUTL-_BIASED
- C414 pad 2: GND -> /AudioDac0/VOUTL-
- C416 pad 1: VDD -> Net-(C416-Pad1)
- C417 pad 1: VDD -> GND
- C417 pad 2: GND -> Net-(C417-Pad2)
- C418 pad 1: +5VA -> Net-(C418-Pad1)
- C420 pad 1: /AudioDac0/VCOM -> Net-(U402B-+)
- C520 pad 1: /AudioDac1/VCOM -> Net-(U502B-+)
- C601 pad 1: /AudioDac0/OUT_L -> /Headphone_driver/AudioInL
- C602 pad 1: /AudioDac0/OUT_R -> /Headphone_driver/AudioInR
- C702 pad 1: Net-(U703A--) -> Net-(U701B--)
- C702 pad 2: Net-(C712-Pad2) -> /Line Driver/LINE_OUT_BUFF_L
- C703 pad 1: Net-(U703B--) -> Net-(U701A--)
- C703 pad 2: Net-(C713-Pad2) -> /Line Driver/LINE_OUT_BUFF_R
- C906 pad 1: Net-(U901-OUT) -> /AudioPower/16V
- C907 pad 1: Net-(U903-EN) -> Net-(U902-VI)
- C908 pad 1: Net-(U903-EN) -> Net-(U903-VI)
- C909 pad 1: +3.3VA -> /AudioPower/5VA_PRE_FERRITE
- C909 pad 2: GND -> Net-(U902-ADJ)
- C911 pad 1: Net-(U904-OUT) -> /AudioPower/5VA_PRE_FERRITE
- C912 pad 1: Net-(U903-OUT) -> /AudioPower/14.5VAA
- D902 pad 2: Net-(D903-A) -> Net-(D902-A)
- D903 pad 2: Net-(D904-A) -> Net-(D903-A)
- D904 pad 2: Net-(D905-A) -> Net-(D904-A)
- FB902 pad 2: Net-(U903-EN) -> Net-(U902-VI)
- FB903 pad 1: Net-(U904-OUT) -> /AudioPower/16V
- FB903 pad 2: +5VA -> Net-(U903-VI)
- FB904 pad 1: Net-(U903-OUT) -> /AudioPower/5VA_PRE_FERRITE
- FB904 pad 2: VAA -> +5VA
- J101 pad 29: /VAA_EN -> /CFG_AUDIO_ENA
- R705 pad 1: GND -> VAA_BIAS_L
- R705 pad 2: Net-(U703A--) -> Net-(U701B--)
- R706 pad 1: GND -> Net-(U701A--)
- R706 pad 2: Net-(U703B--) -> VAA_BIAS_R
- R707 pad 1: Net-(U703A--) -> Net-(U701B--)
- R708 pad 1: Net-(U703B--) -> Net-(U701A--)
- R709 pad 1: Net-(C712-Pad2) -> /Line Driver/LINE_OUT_BUFF_L
- R710 pad 1: Net-(C713-Pad2) -> /Line Driver/LINE_OUT_BUFF_R
- R901 pad 1: VAA -> Net-(D901-A)
- R901 pad 2: Net-(D901-A) -> +5V
- R906 pad 1: Net-(U901-OUT) -> /AudioPower/14.5VAA
- R907 pad 1: /AudioPower/16V -> Net-(U902-ADJ)
- R907 pad 2: Net-(D903-A) -> GND
- R912 pad 1: Net-(U904-OUT) -> /AudioPower/5VA_PRE_FERRITE
- R912 pad 2: Net-(D904-A) -> Net-(U902-ADJ)
- R913 pad 1: Net-(U903-OUT) -> Net-(U902-ADJ)
- R913 pad 2: Net-(D905-A) -> GND
- TP111 pad 1: /MCLK -> /ADC0_MCLK
- TP112 pad 1: /MCLK -> /ADC1_MCLK
- TP113 pad 1: /MCLK -> /DAC0_MCLK
- TP114 pad 1: /MCLK -> /DAC1_MCLK
- TP117 pad 1: /BCLK -> /ADC0_BCLK
- TP118 pad 1: /BCLK -> /ADC1_BCLK
- TP119 pad 1: /BCLK -> /DAC0_BCLK
- TP120 pad 1: /BCLK -> /DAC1_BCLK
- TP905 pad 1: +5VA -> /AudioPower/14.5VAA
- TP906 pad 1: VAA -> GND
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Routing:
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- added copper zone on B.Cu, net SHIELD
- added copper zone on F.Cu, net SHIELD
- added copper zone on In1.Cu, net SHIELD
- added copper zone on In2.Cu, net SHIELD
Other:
- outline, holes or cut-outs redrawn
- copper layers 2 -> 4

Commit message: Start layout and routing of Audio Daugherboard
Also a lot of small changes to everything that became apperant
when the audio daughterboard was designed. Such as the Headphone
PCB, which is now separate from the rest of the audio.
Parts:
- removed the C601 at (73.2, 280.0)
- removed the C602 at (65.0, 280.0)
- removed the C603 at (65.0, 310.0)
- removed the C604 at (50.0, 280.0)
- removed the C605 at (45.0, 314.0)
- removed C606: 100pF, Capacitor_SMD:C_0805_2012Metric_Pad1.18x1.45mm_HandSolder
- removed C607, C608: 220uF, Capacitor_SMD:CP_Elec_4x5.8
- removed C609, C610, C614, C615: 100u, Capacitor_SMD:CP_Elec_6.3x7.7
- removed C611, C613, C616, C617: 100nF, Capacitor_SMD:C_0603_1608Metric
- removed C612: 10uF, Capacitor_SMD:CP_Elec_4x5.8
- removed J103: Conn_02x05_Odd_Even, Connector_PinHeader_2.54mm:PinHeader_2x05_P2.54mm_Horizontal
- removed the J601 at (10.9, 315.5)
- removed the R601 at (19.6, 287.8)
- removed the R602 at (19.6, 284.9)
- removed the R603 at (19.6, 281.9)
- removed the R604 at (19.6, 278.9)
- removed the R605 at (31.9, 287.5)
- removed the R606 at (31.9, 285.0)
- removed the R607 at (20.0, 275.0)
- removed the R608 at (25.0, 275.0)
- removed the R609 at (14.8, 296.1)
- removed the R610 at (9.90, 297.2)
- removed the R611 at (10.0, 305.0)
- removed the R612 at (10.0, 302.1)
- removed R613, R614: 4R7, Resistor_SMD:R_MELF_MMB-0207
- removed RV601: 10k/PTV112-4420A-B103, Skrooter_footprints:Potentiometer_Bourns_PTV09A-1_Dual_Vertical
- removed the TP601 at (20.0, 310.0)
- removed the TP602 at (20.0, 304.9)
- removed the TP603 at (20.0, 299.9)
- removed TP604, TP605: TestPoint, TestPoint:TestPoint_Keystone_5005-5009_Compact
- removed the U601 at (51.6, 312.3)
- removed U602: NE5532, Package_SO:SOIC-8_3.9x4.9mm_P1.27mm
- removed U603: TDA2822D, Package_SO:SOP-8_3.9x4.9mm_P1.27mm
- added C205: 100nF, Capacitor_SMD:C_0603_1608Metric, F.Cu at (20.0, 67.0)
- added C206: 10uF, Capacitor_SMD:CP_Elec_4x5.8, F.Cu at (26.0, 74.5)
- added C305: 100nF, Capacitor_SMD:C_0603_1608Metric, F.Cu at (51.0, 67.0)
- added C306: 10uF, Capacitor_SMD:CP_Elec_4x5.8, F.Cu at (57.0, 74.5)
- added R207: 2k15, Resistor_SMD:R_0603_1608Metric, F.Cu at (16.5, 67.0)
- added R307: 2k15, Resistor_SMD:R_0603_1608Metric, F.Cu at (48.5, 67.0)
- C1002: renamed from C1102; footprint Skrooter_footprints:c_elec_SMD_12.5x13.5 -> Capacitor_SMD:CP_Elec_6.3x5.4
- C1102: renamed from C1202; footprint Skrooter_footprints:c_elec_SMD_12.5x13.5 -> Capacitor_SMD:CP_Elec_6.3x5.4
- C1202: renamed from C1302; footprint Skrooter_footprints:c_elec_SMD_12.5x13.5 -> Capacitor_SMD:CP_Elec_6.3x5.4
- C902: renamed from C1002; footprint Skrooter_footprints:c_elec_SMD_12.5x13.5 -> Capacitor_SMD:CP_Elec_6.3x5.4
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- renumbered C1101 to C1001, C1103 to C1003, C1104 to C1004, C1105 to C1005, C1106 to C1006, C1107 to C1007, C1108 to C1008, C1109 to C1009, C1110 to C1010, C1111 to C1011, C1112 to C1012, C1113 to C1013, C1201 to C1101, C1203 to C1103, C1204 to C1104, C1205 to C1105, C1206 to C1106, C1207 to C1107, C1208 to C1108, C1209 to C1109, C1210 to C1110, C1211 to C1111, C1212 to C1112, C1213 to C1113, C1301 to C1201, C1303 to C1203, C1304 to C1204, C1305 to C1205, C1306 to C1206, C1307 to C1207, C1308 to C1208, C1309 to C1209, C1310 to C1210, C1311 to C1211, C1312 to C1212, C1313 to C1213, C1401 to C1301, C1402 to C1302, C1403 to C1303, C1404 to C1304, C1405 to C1305, C1406 to C1306, C205 to C207, C206 to C208, C207 to C209, C208 to C210, C209 to C211, C305 to C307, C306 to C308, C307 to C309, C308 to C310, C309 to C311, C701 to C601, C702 to C602, C703 to C603, C704 to C604, C705 to C605, C801 to C701, C802 to C702, C901 to C801, C902 to C802, C903 to C803, C917 to C804, C904 to C805, C906 to C806, C907 to C807, C908 to C808, C909 to C809, C910 to C810, C911 to C811, C912 to C812, C913 to C813, C914 to C814, C915 to C815, C916 to C816, C1001 to C901, C1003 to C903, C1004 to C904, C1005 to C905, C1006 to C906, C1007 to C907, C1008 to C908, C1009 to C909, C1010 to C910, C1011 to C911, C1012 to C912, C1013 to C913, D901 to D801, D902 to D802, D903 to D803, D904 to D804, FB901 to FB801, FB902 to FB802, FB903 to FB803, FB904 to FB804, FB905 to FB805, J1401 to J1301, J1402 to J1302, J1403 to J1303, J1404 to J1304, J701 to J601, L901 to L801, Q701 to Q601, Q702 to Q602, R1101 to R1001, R1104 to R1004, R1105 to R1005, R1106 to R1006, R1107 to R1007, R1108 to R1008, R1109 to R1009, R1110 to R1010, R1111 to R1011, R1112 to R1012, R1113 to R1013, R1114 to R1014, R1115 to R1015, R1116 to R1016, R1117 to R1017, R1118 to R1018, R1201 to R1101, R1204 to R1104, R1205 to R1105, R1206 to R1106, R1207 to R1107, R1208 to R1108, R1209 to R1109, R1210 to R1110, R1211 to R1111, R1212 to R1112, R1213 to R1113, R1214 to R1114, R1215 to R1115, R1216 to R1116, R1217 to R1117, R1218 to R1118, R1301 to R1201, R1304 to R1204, R1305 to R1205, R1306 to R1206, R1307 to R1207, R1308 to R1208, R1309 to R1209, R1310 to R1210, R1311 to R1211, R1312 to R1212, R1313 to R1213, R1314 to R1214, R1315 to R1215, R1316 to R1216, R1317 to R1217, R1318 to R1218, R1401 to R1301, R701 to R601, R702 to R602, R703 to R603, R704 to R604, R705 to R605, R706 to R606, R707 to R607, R708 to R608, R709 to R609, R710 to R610, R711 to R611, R712 to R612, R801 to R701, R802 to R702, R901 to R801, R902 to R802, R903 to R803, R904 to R804, R905 to R805, R906 to R806, R907 to R807, R908 to R808, R909 to R809, R910 to R810, R911 to R811, R912 to R812, R913 to R813, R914 to R814, R915 to R815, R916 to R816, R917 to R817, R1001 to R901, R1004 to R904, R1005 to R905, R1006 to R906, R1007 to R907, R1008 to R908, R1009 to R909, R1010 to R910, R1011 to R911, R1012 to R912, R1013 to R913, R1014 to R914, R1015 to R915, R1016 to R916, R1017 to R917, R1018 to R918, TP1101 to TP1001, TP1102 to TP1002, TP1103 to TP1003, TP121 to TP101, TP127 to TP102, TP101 to TP103, TP102 to TP104, TP103 to TP105, TP104 to TP106, TP105 to TP107, TP106 to TP108, TP107 to TP109, TP108 to TP110, TP1201 to TP1101, TP1202 to TP1102, TP1203 to TP1103, TP126 to TP111, TP125 to TP112, TP124 to TP113, TP123 to TP114, TP122 to TP115, TP109 to TP116, TP110 to TP117, TP111 to TP118, TP112 to TP119, TP113 to TP120, TP1301 to TP1201, TP1302 to TP1202, TP1303 to TP1203, TP114 to TP121, TP115 to TP122, TP116 to TP123, TP117 to TP124, TP118 to TP125, TP119 to TP126, TP120 to TP127, TP701 to TP601, TP702 to TP602, TP703 to TP603, TP801 to TP701, TP802 to TP702, TP803 to TP703, TP1 to TP801, TP902 to TP802, TP903 to TP803, TP905 to TP804, TP906 to TP805, TP907 to TP806, TP908 to TP807, TP1001 to TP901, TP1002 to TP902, TP1003 to TP903, U1101 to U1001, U1102 to U1002, U1103 to U1003, U1104 to U1004, U1105 to U1005, U1201 to U1101, U1202 to U1102, U1203 to U1103, U1204 to U1104, U1205 to U1105, U1301 to U1201, U1302 to U1202, U1303 to U1203, U1304 to U1204, U1305 to U1205, U1401 to U1301, U701 to U601, U801 to U701, U901 to U801, U902 to U802, U903 to U803, U1001 to U901, U1002 to U902, U1003 to U903, U1004 to U904, U1005 to U905
Connections:
- C1008 pad 1: Net-(U1103A--) -> Net-(U1003A-+)
- C1008 pad 2: Net-(C1108-Pad2) -> Net-(C1008-Pad2)
- C1009 pad 1: Net-(U1103A-+) -> Net-(U1003B-+)
- C1108 pad 1: Net-(U1203A--) -> Net-(U1103A-+)
- C1108 pad 2: Net-(C1208-Pad2) -> Net-(C1108-Pad2)
- C1109 pad 1: Net-(U1203A-+) -> Net-(U1103B-+)
- C1208 pad 1: Net-(U1303A--) -> Net-(U1203A-+)
- C1208 pad 2: Net-(C1308-Pad2) -> Net-(C1208-Pad2)
- C1209 pad 1: Net-(U1303A-+) -> Net-(U1203B-+)
- C201 pad 1: /AudioAdc0/Input Filtering1/signal_out -> /AudioAdc0/Input Filtering/signal_out
- C202 pad 1: /AudioAdc0/Input Filtering/signal_out -> /AudioAdc0/Input Filtering1/signal_out
- C301 pad 1: /AudioAdc1/Input Filtering1/signal_out -> /AudioAdc1/Input Filtering/signal_out
- C302 pad 1: /AudioAdc1/Input Filtering/signal_out -> /AudioAdc1/Input Filtering1/signal_out
- C420 pad 1: Net-(U402B-+) -> Net-(U402A-+)
- C421 pad 1: Net-(U402A-+) -> Net-(U403B-+)
- C422 pad 1: Net-(U402B--) -> Net-(U402A--)
- C423 pad 1: Net-(U402A--) -> Net-(U403B--)
- C520 pad 1: Net-(U502B-+) -> Net-(U502A-+)
- C521 pad 1: Net-(U502A-+) -> Net-(U503B-+)
- C522 pad 1: Net-(U502B--) -> Net-(U502A--)
- C523 pad 1: Net-(U502A--) -> Net-(U503B--)
- C908 pad 1: Net-(U1003A--) -> Net-(U903A-+)
- C908 pad 2: Net-(C1008-Pad2) -> Net-(C908-Pad2)
- C909 pad 1: Net-(U1003A-+) -> Net-(U903B-+)
- J102 pad 3: /AudioDac0/OUT_L -> /AudioDac1/OUT_L
- J102 pad 5: /AudioDac0/OUT_R -> /AudioDac1/OUT_R
- J201 pad 1: /AudioAdc0/Input Filtering1/signal in -> /AudioAdc0/Input Filtering/signal in
- J201 pad 2: /AudioAdc0/Input Filtering/signal in -> /AudioAdc0/Input Filtering1/signal in
- J301 pad 1: /AudioAdc1/Input Filtering1/signal in -> /AudioAdc1/Input Filtering/signal in
- J301 pad 2: /AudioAdc1/Input Filtering/signal in -> /AudioAdc1/Input Filtering1/signal in
- R1005 pad 2: VAA_BIAS_L -> VAA_BIAS_R
- R1006 pad 2: VAA_BIAS_L -> VAA_BIAS_R
- R101 pad 2: /AudioDac0/MS/ADR0/RSV -> /AudioDac1/MS/ADR0/RSV
- R1012 pad 2: Net-(U1103B--) -> Net-(U1003A--)
- R1013 pad 1: Net-(R1113-Pad1) -> Net-(R1013-Pad1)
- R1013 pad 2: Net-(U1103B--) -> Net-(U1003A--)
- R1014 pad 1: Net-(U1103A--) -> Net-(U1003A-+)
- R1014 pad 2: Net-(R1113-Pad1) -> Net-(R1013-Pad1)
- R1015 pad 1: Net-(U1103A-+) -> Net-(U1003B-+)
- R1015 pad 2: Net-(C1108-Pad2) -> Net-(C1008-Pad2)
- R1016 pad 2: Net-(U1103B--) -> Net-(U1003A--)
- R1017 pad 1: VAA_BIAS_L -> VAA_BIAS_R
- R102 pad 1: /AudioDac0/MS/ADR0/RSV -> /AudioDac1/MS/ADR0/RSV
- R103 pad 2: /AudioDac0/ADR5/ADR1/RSV -> /AudioDac1/ADR5/ADR1/RSV
- R104 pad 1: /AudioDac0/ADR5/ADR1/RSV -> /AudioDac1/ADR5/ADR1/RSV
- R105 pad 2: /AudioDac1/ADR5/ADR1/RSV -> /AudioDac0/ADR5/ADR1/RSV
- R106 pad 1: /AudioDac1/ADR5/ADR1/RSV -> /AudioDac0/ADR5/ADR1/RSV
- R107 pad 2: /AudioDac1/MS/ADR0/RSV -> /AudioDac0/MS/ADR0/RSV
- R108 pad 1: /AudioDac1/MS/ADR0/RSV -> /AudioDac0/MS/ADR0/RSV
- R1105 pad 2: VAA_BIAS_L -> VAA_BIAS_R
- R1106 pad 2: VAA_BIAS_L -> VAA_BIAS_R
- R1112 pad 2: Net-(U1203B--) -> Net-(U1103A--)
- R1113 pad 1: Net-(R1213-Pad1) -> Net-(R1113-Pad1)
- R1113 pad 2: Net-(U1203B--) -> Net-(U1103A--)
- R1114 pad 1: Net-(U1203A--) -> Net-(U1103A-+)
- R1114 pad 2: Net-(R1213-Pad1) -> Net-(R1113-Pad1)
- R1115 pad 1: Net-(U1203A-+) -> Net-(U1103B-+)
- R1115 pad 2: Net-(C1208-Pad2) -> Net-(C1108-Pad2)
- R1116 pad 2: Net-(U1203B--) -> Net-(U1103A--)
- R1117 pad 1: VAA_BIAS_L -> VAA_BIAS_R
- R1205 pad 2: VAA_BIAS_R -> VAA_BIAS_L
- R1206 pad 2: VAA_BIAS_R -> VAA_BIAS_L
- R1212 pad 2: Net-(U1303B--) -> Net-(U1203A--)
- R1213 pad 1: Net-(R1313-Pad1) -> Net-(R1213-Pad1)
- R1213 pad 2: Net-(U1303B--) -> Net-(U1203A--)
- R1214 pad 1: Net-(U1303A--) -> Net-(U1203A-+)
- R1214 pad 2: Net-(R1313-Pad1) -> Net-(R1213-Pad1)
- R1215 pad 1: Net-(U1303A-+) -> Net-(U1203B-+)
- R1215 pad 2: Net-(C1308-Pad2) -> Net-(C1208-Pad2)
- R1216 pad 2: Net-(U1303B--) -> Net-(U1203A--)
- R1217 pad 1: VAA_BIAS_R -> VAA_BIAS_L
- R409 pad 1: Net-(U402B-+) -> Net-(U402A-+)
- R410 pad 1: Net-(U402B--) -> Net-(U402A--)
- R411 pad 1: Net-(U402A-+) -> Net-(U403B-+)
- R412 pad 1: Net-(U402A--) -> Net-(U403B--)
- R509 pad 1: Net-(U502B-+) -> Net-(U502A-+)
- R510 pad 1: Net-(U502B--) -> Net-(U502A--)
- R511 pad 1: Net-(U502A-+) -> Net-(U503B-+)
- R512 pad 1: Net-(U502A--) -> Net-(U503B--)
- R601 pad 1: /AudioDac1/OUT_L -> /AudioDac0/OUT_L
- R602 pad 1: /AudioDac1/OUT_R -> /AudioDac0/OUT_R
- R905 pad 2: VAA_BIAS_R -> VAA_BIAS_L
- R906 pad 2: VAA_BIAS_R -> VAA_BIAS_L
- R912 pad 2: Net-(U1003B--) -> Net-(U903A--)
- R913 pad 1: Net-(R1013-Pad1) -> Net-(R913-Pad1)
- R913 pad 2: Net-(U1003B--) -> Net-(U903A--)
- R914 pad 1: Net-(U1003A--) -> Net-(U903A-+)
- R914 pad 2: Net-(R1013-Pad1) -> Net-(R913-Pad1)
- R915 pad 1: Net-(U1003A-+) -> Net-(U903B-+)
- R915 pad 2: Net-(C1008-Pad2) -> Net-(C908-Pad2)
- R916 pad 2: Net-(U1003B--) -> Net-(U903A--)
- R917 pad 1: VAA_BIAS_R -> VAA_BIAS_L
- TP201 pad 1: /AudioAdc0/Input Filtering1/signal in -> /AudioAdc0/Input Filtering/signal in
- TP202 pad 1: /AudioAdc0/Input Filtering/signal in -> /AudioAdc0/Input Filtering1/signal in
- TP301 pad 1: /AudioAdc1/Input Filtering1/signal in -> /AudioAdc1/Input Filtering/signal in
- TP302 pad 1: /AudioAdc1/Input Filtering/signal in -> /AudioAdc1/Input Filtering1/signal in
- U1003 pad 1: Net-(R1113-Pad1) -> Net-(C1008-Pad2)
- U1003 pad 2: Net-(U1103A--) -> Net-(U1003A--)
- U1003 pad 3: Net-(U1103A-+) -> Net-(U1003A-+)
- U1003 pad 5: Net-(U1103A--) -> Net-(U1003B-+)
- U1003 pad 6: Net-(U1103B--) -> Net-(U1003A-+)
- U1003 pad 7: Net-(C1108-Pad2) -> Net-(R1013-Pad1)
- U1005 pad 1: VAA_BIAS_L -> VAA_BIAS_R
- U1103 pad 1: Net-(R1213-Pad1) -> Net-(C1108-Pad2)
- U1103 pad 2: Net-(U1203A--) -> Net-(U1103A--)
- U1103 pad 3: Net-(U1203A-+) -> Net-(U1103A-+)
- U1103 pad 5: Net-(U1203A--) -> Net-(U1103B-+)
- U1103 pad 6: Net-(U1203B--) -> Net-(U1103A-+)
- U1103 pad 7: Net-(C1208-Pad2) -> Net-(R1113-Pad1)
- U1105 pad 1: VAA_BIAS_L -> VAA_BIAS_R
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Routing:
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- added copper zone on In1.Cu, net GND
- added copper zone on In2.Cu, net GND
- added copper zone on B.Cu, net VAA
Other:
- board size 90 x 320 mm -> 90 x 155 mm
