File: PCB/Magna/audio_daughterboard/input_filtering.kicad_sch (KiCad schematic)
At the start: 43 parts, among them U1001 NE5532, U1002 NE5532, U1003 NE5532, U1004 NE5532, U1005 LM1971M

Commit message: Start layout and routing of Audio Daugherboard
Also a lot of small changes to everything that became apperant
when the audio daughterboard was designed. Such as the Headphone
PCB, which is now separate from the rest of the audio.
Parts:
- C902: renamed from C1002; footprint Skrooter_footprints:c_elec_SMD_12.5x13.5 -> Capacitor_SMD:CP_Elec_6.3x5.4; LCSC C3829328 -> C2164172
- renumbered C1001 to C901, C1003 to C903, C1004 to C904, C1005 to C905, C1006 to C906, C1007 to C907, C1008 to C908, C1009 to C909, C1010 to C910, C1011 to C911, C1012 to C912, C1013 to C913, R1001 to R901, R1002 to R902, R1003 to R903, R1004 to R904, R1005 to R905, R1006 to R906, R1007 to R907, R1008 to R908, R1009 to R909, R1010 to R910, R1011 to R911, R1012 to R912, R1013 to R913, R1014 to R914, R1015 to R915, R1016 to R916, R1017 to R917, R1018 to R918, S1001 to S901, TP1001 to TP901, TP1002 to TP902, TP1003 to TP903, U1001 to U901, U1002 to U902, U1003 to U903, U1004 to U904, U1005 to U905, V1001 to V901, V1002 to V902, V1003 to V903
Connections:
- net at C908.1, R914.1: now also U903.3 (+), U903.6 (-); no longer U903.2 (-), U903.5 (+)
- net at R913.1, R914.2: now also U903.7; no longer U903.1
- net at R912.2, R913.2, R916.2: now also U903.2 (-); no longer U903.6 (-)
- net at C909.1, R915.1: now also U903.5 (+); no longer U903.3 (+)
- net at C908.2, R915.2: now also U903.1; no longer U903.7
Other:
- moved on the sheet: U903A, U903B

Commit message: Finished first round of routing for the Audio Daughterboard
Parts:
- removed TP902, TP903: TestPoint, TestPoint:TestPoint_Keystone_5005-5009_Compact, symbol Connector:TestPoint
- added C914: 100nF, Capacitor_SMD:C_0603_1608Metric, symbol Device:C
- added C915, C916: 10uF, Capacitor_SMD:CP_Elec_4x5.8, symbol Device:C_Polarized
- added C917, C918: 470p, Capacitor_SMD:C_0603_1608Metric, symbol Device:C
- added C919: 2.7n, Capacitor_SMD:C_0603_1608Metric, symbol Device:C
- added R919, R920, R928, R930: 1k, Resistor_SMD:R_0603_1608Metric, symbol Device:R
- added R921, R922, R923, R925: 10k, Resistor_SMD:R_0603_1608Metric, symbol Device:R
- added R924, R926: 680R, Resistor_SMD:R_0603_1608Metric, symbol Device:R
- added R927, R929: 100R, Resistor_SMD:R_0603_1608Metric, symbol Device:R
- added TP902, TP903, TP904: TestPoint, TestPoint:TestPoint_Pad_1.0x1.0mm, symbol Connector:TestPoint_Alt
- added U906: NE5532, Package_SO:SOIC-8_3.9x4.9mm_P1.27mm, symbol Amplifier_Operational:NE5532
- R901, R904, R905, R906, R907, R908, R909, R910, R911, R912, R913, R914, R915, R916, R917, R918: now in the parts list
Connections:
- net Filtered_input: now also U904.6 (-), TP902.1; no longer U904.5 (+)
- net GND: now also C914.2, U906.4 (V-)
- net VAA: now also C914.1, U906.8 (V+)
- net antennuated_input: now also TP903.1
- net at C911.1, R916.1: now also U904.5 (+); no longer U904.6 (-)
- net at C908.1, R914.1, U903.6 (-): now also U903.2 (-); no longer U903.3 (+)
- net at R912.2, R913.2, R916.2: now also U903.3 (+); no longer U903.2 (-)
- net V_bias renamed INV+
- net signal_out: no longer names the net of R918.2, U904.1
- net signal_out: now also C915.1, R919.2, TP904.1
- new net: C918.1, R925.1, R926.2, U906.3 (+)
- new net: C918.2, R929.2, R930.1, U906.1
- new net: C916.2, R922.2, U906.2 (-)
- new net: C917.1, R923.1, R924.2, U906.5 (+)
- new net: C915.2, R921.1, U906.6 (-)
- new net: C917.2, R927.2, R928.1, U906.7
- new net INV-: R919.1, R920.2
- new net INV_OUT: C916.1, R920.1
- new net VQ: R921.2, R922.1
- new net signal_out+: C919.1, R923.2, R924.1, R927.1, R928.2
- new net signal_out-: C919.2, R925.2, R926.1, R929.1, R930.2
Other:
- note added: "634R"
- note added: "91R"
- moved on the sheet: C903, C904, C905, C908, C909, C911, R907, R908, R909, R910, R911, R912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

Commit message: Fix board alignments and mounting holes
Parts:
- C901, C902, C903, C904, C905, C906, C907, C908, C909, C910, C911, C912, C913, C914, C915, C916, U901, U902, U903, U904, U905, U906: now in the parts list
- TP902, TP903, TP904: now left out of the parts list
Changed lines of the file:
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@@
 		(unit 3)
 		(exclude_from_sim no)
-		(in_bom no)
+		(in_bom yes)
 		(on_board yes)
 		(dnp no)
@@
 		(unit 1)
 		(exclude_from_sim no)
-		(in_bom no)
+		(in_bom yes)
 		(on_board yes)
 		(dnp no)
@@
 		(unit 2)
 		(exclude_from_sim no)
-		(in_bom no)
+		(in_bom yes)
 		(on_board yes)
 		(dnp no)
@@
 		(unit 3)
 		(exclude_from_sim no)
-		(in_bom no)
+		(in_bom yes)
 		(on_board yes)
 		(dnp no)
@@
 		(unit 1)
 		(exclude_from_sim no)
-		(in_bom no)
+		(in_bom yes)
 		(on_board yes)
 		(dnp no)
@@
 		(unit 1)
 		(exclude_from_sim no)
-		(in_bom no)
+		(in_bom yes)
 		(on_board yes)
 		(dnp no)
@@
 		(unit 1)
 		(exclude_from_sim no)
-		(in_bom no)
+		(in_bom yes)
 		(on_board yes)
 		(dnp no)
@@
 		(unit 1)
 		(exclude_from_sim no)
-		(in_bom yes)
+		(in_bom no)
 		(on_board yes)
 		(dnp no)
@@
 		(unit 2)
 		(exclude_from_sim no)
-		(in_bom no)
+		(in_bom yes)
 		(on_board yes)
 		(dnp no)
@@
 		(unit 1)
 		(exclude_from_sim no)
-		(in_bom no)
+		(in_bom yes)
 		(on_board yes)
 		(dnp no)
@@
 		(unit 2)
 		(exclude_from_sim no)
-		(in_bom no)
+		(in_bom yes)
 		(on_board yes)
 		(dnp no)
@@
 		(unit 1)
 		(exclude_from_sim no)
-		(in_bom no)
+		(in_bom yes)
 		(on_board yes)
 		(dnp no)
@@
 		(unit 2)
 		(exclude_from_sim no)
-		(in_bom no)
+		(in_bom yes)
 		(on_board yes)
 		(dnp no)
@@
 		(unit 1)
 		(exclude_from_sim no)
-		(in_bom no)
+		(in_bom yes)
 		(on_board yes)
 		(dnp no)
@@
 		(unit 1)
 		(exclude_from_sim no)
-		(in_bom no)
+		(in_bom yes)
 		(on_board yes)
 		(dnp no)
@@
 		(unit 2)
 		(exclude_from_sim no)
-		(in_bom no)
+		(in_bom yes)
 		(on_board yes)
 		(dnp no)
@@
 		(unit 3)
 		(exclude_from_sim no)
-		(in_bom no)
+		(in_bom yes)
 		(on_board yes)
 		(dnp no)
@@
 		(unit 3)
 		(exclude_from_sim no)
-		(in_bom no)
+		(in_bom yes)
 		(on_board yes)
 		(dnp no)
@@
 		(unit 1)
 		(exclude_from_sim no)
-		(in_bom no)
+		(in_bom yes)
 		(on_board yes)
 		(dnp no)
@@
 		(unit 1)
 		(exclude_from_sim no)
-		(in_bom no)
+		(in_bom yes)
 		(on_board yes)
 		(dnp no)
@@
 		(unit 1)
 		(exclude_from_sim no)
-		(in_bom no)
+		(in_bom yes)
 		(on_board yes)
 		(dnp no)
@@
 		(unit 1)
 		(exclude_from_sim no)
-		(in_bom yes)
+		(in_bom no)
 		(on_board yes)
 		(dnp no)
@@
 		(unit 1)
 		(exclude_from_sim no)
-		(in_bom no)
+		(in_bom yes)
 		(on_board yes)
 		(dnp no)
@@
 		(unit 1)
 		(exclude_from_sim no)
-		(in_bom no)
+		(in_bom yes)
 		(on_board yes)
 		(dnp no)
@@
 		(unit 1)
 		(exclude_from_sim no)
-		(in_bom no)
+		(in_bom yes)
 		(on_board yes)
 		(dnp no)
@@
 		(unit 1)
 		(exclude_from_sim no)
-		(in_bom no)
+		(in_bom yes)
 		(on_board yes)
 		(dnp no)
@@
 		(unit 1)
 		(exclude_from_sim no)
-		(in_bom no)
+		(in_bom yes)
 		(on_board yes)
 		(dnp no)
@@
 		(unit 1)
 		(exclude_from_sim yes)
-		(in_bom no)
+		(in_bom yes)
 		(on_board yes)
 		(dnp no)
@@
 		(unit 1)
 		(exclude_from_sim no)
-		(in_bom no)
+		(in_bom yes)
 		(on_board yes)
 		(dnp no)
@@
 		(unit 3)
 		(exclude_from_sim no)
-		(in_bom no)
+		(in_bom yes)
 		(on_board yes)
 		(dnp no)
@@
 		(unit 1)
 		(exclude_from_sim no)
-		(in_bom no)
+		(in_bom yes)
 		(on_board yes)
 		(dnp no)
@@
 		(unit 1)
 		(exclude_from_sim no)
-		(in_bom yes)
+		(in_bom no)
 		(on_board yes)
 		(dnp no)
@@
 		(unit 1)
 		(exclude_from_sim no)
-		(in_bom no)
+		(in_bom yes)
 		(on_board yes)
 		(dnp no)
@@
 		(unit 1)
 		(exclude_from_sim no)
-		(in_bom no)
+		(in_bom yes)
 		(on_board yes)
 		(dnp no)
@@
 		(unit 1)
 		(exclude_from_sim no)
-		(in_bom no)
+		(in_bom yes)
 		(on_board yes)
 		(dnp no)
